File: Kicad Files/Input control.kicad_sch (KiCad schematic)
At the start: 37 parts, among them SW2 SW_DIP_x08, SW3 SW_DIP_x08, SW4 PROG/Man, SW5 WRITE, SW6 RESET, U44 74LS157, U45 74LS157, U46 74LS595, U47 74LS595, U48 74LS157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

Commit message: solving errors
Connections:
- no-connect marks 19 -> 21
Changed lines of the file:
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@@
   (no_connect (at 187.96 52.07))
   (no_connect (at 250.19 99.06))
+  (no_connect (at 224.79 68.58))
+  (no_connect (at 224.79 66.04))
   (no_connect (at 187.96 87.63))
   (no_connect (at 250.19 86.36))
