File: Kicad Files/clock.kicad_sch (KiCad schematic)
At the start: 34 parts, among them SW7 SW_Push, SW8 SW_SPDT, U60 LM555, U61 LM555, U62 LM555

Commit message: solving errors
Parts:
- gave numbers to parts that had none: 5
Changed lines of the file:
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@@
   (symbol (lib_id "74xx:74HC00") (at 147.32 109.22 0) (unit 1)
     (in_bom yes) (on_board yes)
-    (property "Reference" "U?" (id 0) (at 147.32 109.22 0))
+    (property "Reference" "U63" (id 0) (at 147.32 109.22 0))
     (property "Value" "74HC00" (id 1) (at 147.32 104.14 0))
     (property "Footprint" "" (id 2) (at 147.32 109.22 0)
@@
   (symbol (lib_id "74xx:74HC00") (at 147.32 121.92 0) (unit 2)
     (in_bom yes) (on_board yes)
-    (property "Reference" "U?" (id 0) (at 147.32 121.92 0))
+    (property "Reference" "U63" (id 0) (at 147.32 121.92 0))
     (property "Value" "74HC00" (id 1) (at 147.32 116.84 0))
     (property "Footprint" "" (id 2) (at 147.32 121.92 0)
@@
   (symbol (lib_id "74xx:74HC00") (at 162.56 115.57 0) (unit 3)
     (in_bom yes) (on_board yes)
-    (property "Reference" "U?" (id 0) (at 162.56 115.57 0))
+    (property "Reference" "U63" (id 0) (at 162.56 115.57 0))
     (property "Value" "74HC00" (id 1) (at 162.56 110.49 0))
     (property "Footprint" "" (id 2) (at 162.56 115.57 0)
@@
   (symbol (lib_id "74xx:74HC00") (at 177.8 118.11 0) (unit 4)
     (in_bom yes) (on_board yes)
-    (property "Reference" "U?" (id 0) (at 177.8 118.11 0))
+    (property "Reference" "U63" (id 0) (at 177.8 118.11 0))
     (property "Value" "74HC00" (id 1) (at 177.8 113.03 0))
     (property "Footprint" "" (id 2) (at 177.8 118.11 0)
@@
   (symbol (lib_id "74xx:74HC04") (at 132.08 119.38 0) (unit 1)
     (in_bom yes) (on_board yes)
-    (property "Reference" "U?" (id 0) (at 130.81 119.38 0))
+    (property "Reference" "U54" (id 0) (at 130.81 119.38 0))
     (property "Value" "74HC04" (id 1) (at 132.08 114.3 0))
     (property "Footprint" "" (id 2) (at 132.08 119.38 0)
@@
   (symbol (lib_id "74xx:74HC04") (at 162.56 129.54 0) (unit 2)
     (in_bom yes) (on_board yes)
-    (property "Reference" "U?" (id 0) (at 161.29 129.54 0))
+    (property "Reference" "U54" (id 0) (at 161.29 129.54 0))
     (property "Value" "74HC04" (id 1) (at 162.56 124.46 0))
     (property "Footprint" "" (id 2) (at 162.56 129.54 0)
@@
   (symbol (lib_id "74xx:74HC04") (at 193.04 118.11 0) (unit 3)
     (in_bom yes) (on_board yes)
-    (property "Reference" "U?" (id 0) (at 193.04 110.0582 0))
+    (property "Reference" "U54" (id 0) (at 193.04 110.0582 0))
     (property "Value" "74HC04" (id 1) (at 193.04 112.3696 0))
     (property "Footprint" "" (id 2) (at 193.04 118.11 0)
@@
   (symbol (lib_id "Device:LED") (at 200.66 121.92 90) (unit 1)
     (in_bom yes) (on_board yes)
-    (property "Reference" "D?" (id 0) (at 198.12 121.92 0))
+    (property "Reference" "D107" (id 0) (at 198.12 121.92 0))
     (property "Value" "BLUE" (id 1) (at 203.2 121.92 0))
     (property "Footprint" "LED_THT:LED_D5.0mm" (id 2) (at 200.66 121.92 0)
@@
   (symbol (lib_id "Device:R") (at 200.66 129.54 0) (unit 1)
     (in_bom yes) (on_board yes)
-    (property "Reference" "R?" (id 0) (at 202.692 129.54 90))
+    (property "Reference" "R143" (id 0) (at 202.692 129.54 90))
     (property "Value" "220" (id 1) (at 200.66 129.54 90))
     (property "Footprint" "Resistor_THT:R_Axial_DIN0207_L6.3mm_D2.5mm_P7.62mm_Horizontal" (id 2) (at 198.882 129.54 90)
@@
   (symbol (lib_id "Device:R") (at 72.39 63.5 0) (unit 1)
     (in_bom yes) (on_board yes)
-    (property "Reference" "R?" (id 0) (at 77.47 63.5 90))
+    (property "Reference" "R142" (id 0) (at 77.47 63.5 90))
     (property "Value" "220" (id 1) (at 74.93 63.5 90))
     (property "Footprint" "Resistor_THT:R_Axial_DIN0207_L6.3mm_D2.5mm_P7.62mm_Horizontal" (id 2) (at 70.612 63.5 90)
