File: Kicad Files/clock.kicad_sch (KiCad schematic)
At the start: 28 parts, among them SW1 SW_Push, SW2 SW_SPDT, U4 LM555, U5 LM555, U6 74HC04, U7 74HC00, U8 LM555

Commit message: updated library
Parts:
- removed C4: 100µF, Capacitor_THT:CP_Radial_D5.0mm_P2.00mm, symbol 8bit-computer-rescue:CP1-Device
- removed D33, D34, D36: RED, LED_THT:LED_D5.0mm, symbol 8bit-computer-rescue:LED_ALT-Device
- removed D35: BLUE, LED_THT:LED_D5.0mm, symbol 8bit-computer-rescue:LED_ALT-Device
- removed RV1: 10k, 8bit-custom-footprints:Potentiometer-5.5mm, symbol 8bit-computer-rescue:POT-8bit-computer-rescue
- removed SW1: SW_Push, Button_Switch_THT:SW_PUSH_6mm_H5mm, symbol 8bit-computer-rescue:SW_Push-8bit-computer-rescue
- removed SW2: SW_SPDT, 8bit-custom-footprints:DPDT-pushbutton, symbol 8bit-computer-rescue:SW_SPDT-8bit-computer-rescue
- removed U4, U5, U8: LM555, Package_DIP:DIP-8_W7.62mm, symbol 8bit-computer-rescue:LM555-8bit-computer-rescue
- added C4: C_Polarized, symbol Device:C_Polarized
- added D41, D42, D43, D44: LED, symbol Device:LED
- added RV1: R_Potentiometer, symbol Device:R_Potentiometer
- added SW1: SW_Push, symbol Switch:SW_Push
- added SW2: SW_SPDT, symbol Switch:SW_SPDT
- added U4, U5, U8: NE555P, Package_DIP:DIP-8_W7.62mm, symbol Timer:NE555P
- renumbered R33 to R41, R34 to R42, R35 to R43, R36 to R44, R37 to R45, R38 to R46, R39 to R47, R40 to R48, R41 to R49
Connections:
- net CLK: now also D43.2 (A)
- net GND: now also C4.2, SW1.1, SW2.2 (B), U4.1 (GND), U5.1 (GND), U8.1 (GND), U8.6 (THR)
- net VCC: now also U4.4 (R), U4.8 (VCC), U5.4 (R), U5.8 (VCC), U8.8 (VCC)
- net at U7.2: now also D41.2 (A), U4.3 (Q)
- net at C3.1: now also U4.5 (CV)
- net at R41.2: now also RV1.2, U4.7 (DIS)
- net at R43.2: now also SW1.2, U5.2 (TR)
- net at R47.2: now also SW2.3 (C), U8.4 (R)
- net at R46.2: now also SW2.1 (A), U8.2 (TR)
- net at C6.1, R44.2: now also U5.6 (THR), U5.7 (DIS)
- net at C5.1: now also U5.5 (CV)
- net at C7.1: now also U8.5 (CV)
- net at U6.1, U7.1: now also D44.2 (A), U8.3 (Q)
- net at U7.5: now also D42.2 (A), U5.3 (Q)
- net at R42.1: now also D41.1 (K)
- net at R45.1: now also D42.1 (K)
- net at R49.1: now also D44.1 (K)
- net at R48.1: now also D43.1 (K)
- new net: C4.1, RV1.1, U4.2 (TR), U4.6 (THR)

Commit message: work on clk
Parts:
- removed D41, D42, D44: LED, symbol Device:LED
- removed R42, R45, R49: R, Resistor_THT:R_Axial_DIN0207_L6.3mm_D2.5mm_P7.62mm_Horizontal, symbol Device:R
- added D? (x3): LED, symbol Device:LED
- added R? (x3): R_Small, symbol Device:R_Small
- RV1: value R_Potentiometer -> RV1
Connections:
- net GND: now also C3.1, C5.1, U4.6 (THR), R?.1, R?.1, R?.1; no longer C3.2, C5.2
- net VCC: now also R41.2; no longer R41.1
- net at U4.5 (CV): now also C3.2; no longer C3.1
- net at U5.5 (CV): now also C5.2; no longer C5.1
- net at U6.1, U7.1, U8.3 (Q): now also D?.2 (A)
- net at U4.3 (Q), U7.2: now also D?.2 (A)
- net at U5.3 (Q), U7.5: now also D?.2 (A)
- net at C4.1, U4.2 (TR): now also RV1.2; no longer RV1.1, U4.6 (THR)
- new net: R41.1, RV1.1, U4.7 (DIS)
- new net: D?.1 (K), R?.2 (x3)
Other:
- moved on the sheet: C3, C4, C5, C6, R41, R43, RV1, SW1

Commit message: im sooo stupiiid
Parts:
- gave numbers to parts that had none: 6
Other:
- moved on the sheet: C3, C4, C5, C6, C7, C8, C9, D41, D42, D43, D44, R41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
