File: Kicad Files/ram.kicad_sch (KiCad schematic)
At the start: 30 parts, among them U51 HM62256BLP, U52 74LS245, U53 74LS245, U55 74LS157

Commit message: solving errors
Parts:
- gave numbers to parts that had none: 2
Changed lines of the file:
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@@
   (symbol (lib_id "74xx:74HC00") (at 72.39 218.44 90) (unit 1)
     (in_bom yes) (on_board yes)
-    (property "Reference" "U?" (id 0) (at 72.39 218.44 0))
+    (property "Reference" "U64" (id 0) (at 72.39 218.44 0))
     (property "Value" "74HC00" (id 1) (at 67.31 218.44 0))
     (property "Footprint" "" (id 2) (at 72.39 218.44 0)
@@
   (symbol (lib_id "74xx:74HC00") (at 82.55 218.44 90) (unit 2)
     (in_bom yes) (on_board yes)
-    (property "Reference" "U?" (id 0) (at 82.55 218.44 0))
+    (property "Reference" "U65" (id 0) (at 82.55 218.44 0))
     (property "Value" "74HC00" (id 1) (at 77.47 218.44 0))
     (property "Footprint" "" (id 2) (at 82.55 218.44 0)
@@
   (symbol (lib_id "74xx:74HC00") (at 92.71 218.44 90) (unit 3)
     (in_bom yes) (on_board yes)
-    (property "Reference" "U?" (id 0) (at 92.71 218.44 0))
+    (property "Reference" "U64" (id 0) (at 92.71 218.44 0))
     (property "Value" "74HC00" (id 1) (at 87.63 218.44 0))
     (property "Footprint" "" (id 2) (at 92.71 218.44 0)
@@
   (symbol (lib_id "74xx:74HC00") (at 87.63 232.41 0) (unit 4)
     (in_bom yes) (on_board yes)
-    (property "Reference" "U?" (id 0) (at 87.63 232.41 0))
+    (property "Reference" "U64" (id 0) (at 87.63 232.41 0))
     (property "Value" "74HC00" (id 1) (at 87.63 227.33 0))
     (property "Footprint" "" (id 2) (at 87.63 232.41 0)
@@
   (symbol (lib_id "74xx:74HC00") (at 72.39 234.95 0) (unit 1)
     (in_bom yes) (on_board yes)
-    (property "Reference" "U?" (id 0) (at 72.39 234.95 0))
+    (property "Reference" "U65" (id 0) (at 72.39 234.95 0))
     (property "Value" "74HC00" (id 1) (at 72.39 229.87 0))
     (property "Footprint" "" (id 2) (at 72.39 234.95 0)
@@
   (symbol (lib_id "74xx:74HC00") (at 54.61 229.87 0) (unit 2)
     (in_bom yes) (on_board yes)
-    (property "Reference" "U?" (id 0) (at 54.61 221.615 0))
+    (property "Reference" "U64" (id 0) (at 54.61 221.615 0))
     (property "Value" "74HC00" (id 1) (at 54.61 223.9264 0))
     (property "Footprint" "" (id 2) (at 54.61 229.87 0)
