File: Kicad Files/ram.kicad_sch (KiCad schematic)
At the start: 20 parts, among them U20 HM62256BLP, U22 74LS245

Commit message: fixed erc
Parts:
- gave numbers to parts that had none: 16
- renumbered C12 to C11, C13 to C12, U20 to U13, U22 to U14
Changed lines of the file:
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@@
   (symbol (lib_id "Device:C") (at 175.895 29.21 0) (unit 1)
     (in_bom yes) (on_board yes)
-    (property "Reference" "C13" (id 0) (at 176.53 26.67 0)
+    (property "Reference" "C12" (id 0) (at 176.53 26.67 0)
       (effects (font (size 1.27 1.27)) (justify left))
     )
@@
   (symbol (lib_id "power:GND") (at 172.085 38.1 0) (unit 1)
     (in_bom yes) (on_board yes)
-    (property "Reference" "#PWR088" (id 0) (at 172.085 44.45 0)
+    (property "Reference" "#PWR040" (id 0) (at 172.085 44.45 0)
       (effects (font (size 1.27 1.27)) hide)
     )
@@
   (symbol (lib_id "power:VCC") (at 172.085 20.32 0) (unit 1)
     (in_bom yes) (on_board yes)
-    (property "Reference" "#PWR087" (id 0) (at 172.085 24.13 0)
+    (property "Reference" "#PWR039" (id 0) (at 172.085 24.13 0)
       (effects (font (size 1.27 1.27)) hide)
     )
@@
   (symbol (lib_id "Device:C") (at 168.275 29.21 0) (unit 1)
     (in_bom yes) (on_board yes)
-    (property "Reference" "C12" (id 0) (at 168.91 26.67 0)
+    (property "Reference" "C11" (id 0) (at 168.91 26.67 0)
       (effects (font (size 1.27 1.27)) (justify left))
     )
@@
   (symbol (lib_id "Memory_RAM:HM62256BLP") (at 69.215 66.04 0) (unit 1)
     (in_bom yes) (on_board yes)
-    (property "Reference" "U20" (id 0) (at 67.945 68.58 90)
+    (property "Reference" "U13" (id 0) (at 67.945 68.58 90)
       (effects (font (size 1.27 1.27)) (justify left))
     )
@@
   (symbol (lib_id "74xx:74LS245") (at 140.97 60.96 0) (unit 1)
     (in_bom yes) (on_board yes)
-    (property "Reference" "U22" (id 0) (at 146.05 41.91 0))
+    (property "Reference" "U14" (id 0) (at 146.05 41.91 0))
     (property "Value" "74LS245" (id 1) (at 146.05 44.45 0))
     (property "Footprint" "" (id 2) (at 140.97 60.96 0)
@@
   (symbol (lib_id "power:GND") (at 69.215 88.9 90) (unit 1)
     (in_bom yes) (on_board yes)
-    (property "Reference" "#PWR073" (id 0) (at 75.565 88.9 0)
+    (property "Reference" "#PWR033" (id 0) (at 75.565 88.9 0)
       (effects (font (size 1.27 1.27)) hide)
     )
@@
   (symbol (lib_id "power:VCC") (at 69.215 43.18 90) (unit 1)
     (in_bom yes) (on_board yes)
-    (property "Reference" "#PWR083" (id 0) (at 73.025 43.18 0)
+    (property "Reference" "#PWR032" (id 0) (at 73.025 43.18 0)
       (effects (font (size 1.27 1.27)) hide)
     )
@@
   (symbol (lib_id "power:GND") (at 140.97 81.28 90) (unit 1)
     (in_bom yes) (on_board yes)
-    (property "Reference" "#PWR086" (id 0) (at 147.32 81.28 0)
+    (property "Reference" "#PWR038" (id 0) (at 147.32 81.28 0)
       (effects (font (size 1.27 1.27)) hide)
     )
@@
   (symbol (lib_id "power:VCC") (at 140.97 40.64 0) (unit 1)
     (in_bom yes) (on_board yes)
-    (property "Reference" "#PWR085" (id 0) (at 140.97 44.45 0)
+    (property "Reference" "#PWR037" (id 0) (at 140.97 44.45 0)
       (effects (font (size 1.27 1.27)) hide)
     )
@@
   (symbol (lib_id "power:GND") (at 81.915 71.12 90) (unit 1)
     (in_bom yes) (on_board yes)
-    (property "Reference" "#PWR079" (id 0) (at 88.265 71.12 0)
+    (property "Reference" "#PWR034" (id 0) (at 88.265 71.12 0)
       (effects (font (size 1.27 1.27)) hide)
     )
@@
   (symbol (lib_id "Device:R_Small") (at 120.015 36.195 180) (unit 1)
     (in_bom yes) (on_board yes)
-    (property "Reference" "R?" (id 0) (at 120.015 36.195 90))
+    (property "Reference" "R64" (id 0) (at 120.015 36.195 90))
     (property "Value" "R_Small" (id 1) (at 118.745 28.575 90))
     (property "Footprint" "" (id 2) (at 120.015 36.195 0)
@@
   (symbol (lib_id "Device:R_Small") (at 114.935 36.195 180) (unit 1)
     (in_bom yes) (on_board yes)
-    (property "Reference" "R?" (id 0) (at 114.935 36.195 90))
+    (property "Reference" "R62" (id 0) (at 114.935 36.195 90))
     (property "Value" "R_Small" (id 1) (at 118.745 28.575 90))
     (property "Footprint" "" (id 2) (at 114.935 36.195 0)
@@
   (symbol (lib_id "Device:LED") (at 112.395 42.545 270) (unit 1)
     (in_bom yes) (on_board yes)
-    (property "Reference" "D?" (id 0) (at 112.395 42.545 0))
+    (property "Reference" "D56" (id 0) (at 112.395 42.545 0))
     (property "Value" "LED" (id 1) (at 108.585 48.895 0))
     (property "Footprint" "" (id 2) (at 112.395 42.545 0)
@@
   (symbol (lib_id "Device:R_Small") (at 104.775 36.195 180) (unit 1)
     (in_bom yes) (on_board yes)
-    (property "Reference" "R?" (id 0) (at 104.775 36.195 90))
+    (property "Reference" "R58" (id 0) (at 104.775 36.195 90))
     (property "Value" "R_Small" (id 1) (at 108.585 28.575 90))
     (property "Footprint" "" (id 2) (at 104.775 36.195 0)
@@
   (symbol (lib_id "Device:LED") (at 122.555 42.545 270) (unit 1)
     (in_bom yes) (on_board yes)
-    (property "Reference" "D?" (id 0) (at 122.555 42.545 0))
+    (property "Reference" "D60" (id 0) (at 122.555 42.545 0))
     (property "Value" "LED" (id 1) (at 118.745 48.895 0))
     (property "Footprint" "" (id 2) (at 122.555 42.545 0)
@@
   (symbol (lib_id "Device:LED") (at 104.775 42.545 270) (unit 1)
     (in_bom yes) (on_board yes)
-    (property "Reference" "D?" (id 0) (at 104.775 42.545 0))
+    (property "Reference" "D53" (id 0) (at 104.775 42.545 0))
     (property "Value" "LED" (id 1) (at 108.585 48.895 0))
     (property "Footprint" "" (id 2) (at 104.775 42.545 0)
@@
   (symbol (lib_id "Device:LED") (at 120.015 42.545 270) (unit 1)
     (in_bom yes) (on_board yes)
-    (property "Reference" "D?" (id 0) (at 120.015 42.545 0))
+    (property "Reference" "D59" (id 0) (at 120.015 42.545 0))
     (property "Value" "LED" (id 1) (at 118.745 48.895 0))
     (property "Footprint" "" (id 2) (at 120.015 42.545 0)
@@
   (symbol (lib_id "Device:R_Small") (at 109.855 36.195 180) (unit 1)
     (in_bom yes) (on_board yes)
-    (property "Reference" "R?" (id 0) (at 109.855 36.195 90))
+    (property "Reference" "R60" (id 0) (at 109.855 36.195 90))
     (property "Value" "R_Small" (id 1) (at 108.585 28.575 90))
     (property "Footprint" "" (id 2) (at 109.855 36.195 0)
@@
   (symbol (lib_id "Device:R_Small") (at 117.475 36.195 180) (unit 1)
     (in_bom yes) (on_board yes)
-    (property "Reference" "R?" (id 0) (at 117.475 36.195 90))
+    (property "Reference" "R63" (id 0) (at 117.475 36.195 90))
     (property "Value" "R_Small" (id 1) (at 118.745 28.575 90))
     (property "Footprint" "" (id 2) (at 117.475 36.195 0)
@@
   (symbol (lib_id "Device:R_Small") (at 107.315 36.195 180) (unit 1)
     (in_bom yes) (on_board yes)
-    (property "Reference" "R?" (id 0) (at 107.315 36.195 90))
+    (property "Reference" "R59" (id 0) (at 107.315 36.195 90))
     (property "Value" "R_Small" (id 1) (at 108.585 28.575 90))
     (property "Footprint" "" (id 2) (at 107.315 36.195 0)
@@
   (symbol (lib_id "Device:LED") (at 109.855 42.545 270) (unit 1)
     (in_bom yes) (on_board yes)
-    (property "Reference" "D?" (id 0) (at 109.855 42.545 0))
+    (property "Reference" "D55" (id 0) (at 109.855 42.545 0))
     (property "Value" "LED" (id 1) (at 108.585 48.895 0))
     (property "Footprint" "" (id 2) (at 109.855 42.545 0)
@@
   (symbol (lib_id "Device:LED") (at 117.475 42.545 270) (unit 1)
     (in_bom yes) (on_board yes)
-    (property "Reference" "D?" (id 0) (at 117.475 42.545 0))
+    (property "Reference" "D58" (id 0) (at 117.475 42.545 0))
     (property "Value" "LED" (id 1) (at 118.745 48.895 0))
     (property "Footprint" "" (id 2) (at 117.475 42.545 0)
@@
   (symbol (lib_id "power:GND") (at 102.235 33.655 270) (unit 1)
     (in_bom yes) (on_board yes) (fields_autoplaced)
-    (property "Reference" "#PWR?" (id 0) (at 95.885 33.655 0)
+    (property "Reference" "#PWR036" (id 0) (at 95.885 33.655 0)
       (effects (font (size 1.27 1.27)) hide)
     )
@@
   (symbol (lib_id "Device:LED") (at 107.315 42.545 270) (unit 1)
     (in_bom yes) (on_board yes)
-    (property "Reference" "D?" (id 0) (at 107.315 42.545 0))
+    (property "Reference" "D54" (id 0) (at 107.315 42.545 0))
     (property "Value" "LED" (id 1) (at 108.585 48.895 0))
     (property "Footprint" "" (id 2) (at 107.315 42.545 0)
@@
   (symbol (lib_id "power:GND") (at 81.915 76.2 90) (unit 1)
     (in_bom yes) (on_board yes)
-    (property "Reference" "#PWR?" (id 0) (at 88.265 76.2 0)
+    (property "Reference" "#PWR035" (id 0) (at 88.265 76.2 0)
       (effects (font (size 1.27 1.27)) hide)
     )
@@
   (symbol (lib_id "Device:LED") (at 114.935 42.545 270) (unit 1)
     (in_bom yes) (on_board yes)
-    (property "Reference" "D?" (id 0) (at 114.935 42.545 0))
+    (property "Reference" "D57" (id 0) (at 114.935 42.545 0))
     (property "Value" "LED" (id 1) (at 118.745 48.895 0))
     (property "Footprint" "" (id 2) (at 114.935 42.545 0)
@@
   (symbol (lib_id "Device:R_Small") (at 112.395 36.195 180) (unit 1)
     (in_bom yes) (on_board yes)
-    (property "Reference" "R?" (id 0) (at 112.395 36.195 90))
+    (property "Reference" "R61" (id 0) (at 112.395 36.195 90))
     (property "Value" "R_Small" (id 1) (at 108.585 28.575 90))
     (property "Footprint" "" (id 2) (at 112.395 36.195 0)
@@
   (symbol (lib_id "Device:R_Small") (at 122.555 36.195 180) (unit 1)
     (in_bom yes) (on_board yes)
-    (property "Reference" "R?" (id 0) (at 122.555 36.195 90))
+    (property "Reference" "R65" (id 0) (at 122.555 36.195 90))
     (property "Value" "R_Small" (id 1) (at 118.745 28.575 90))
     (property "Footprint" "" (id 2) (at 122.555 36.195 0)

Commit message: np2
Other:
- moved on the sheet: C11, C12, D53, D54, D55, D56, D57, D58, D59, D60, R58, R59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

Commit message: updated library
Parts:
- renumbered D53 to D61, D54 to D62, D55 to D63, D56 to D64, D57 to D65, D58 to D66, D59 to D67, D60 to D68, R58 to R66, R59 to R67, R60 to R68, R61 to R69, R62 to R70, R63 to R71, R64 to R72, R65 to R73
Changed lines of the file:
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@@
   (symbol (lib_id "power:GND") (at 198.12 80.645 0) (unit 1)
     (in_bom yes) (on_board yes)
-    (property "Reference" "#PWR040" (id 0) (at 198.12 86.995 0)
+    (property "Reference" "#PWR048" (id 0) (at 198.12 86.995 0)
       (effects (font (size 1.27 1.27)) hide)
     )
@@
   (symbol (lib_id "power:VCC") (at 198.12 62.865 0) (unit 1)
     (in_bom yes) (on_board yes)
-    (property "Reference" "#PWR039" (id 0) (at 198.12 66.675 0)
+    (property "Reference" "#PWR047" (id 0) (at 198.12 66.675 0)
       (effects (font (size 1.27 1.27)) hide)
     )
@@
   (symbol (lib_id "power:GND") (at 95.25 131.445 90) (unit 1)
     (in_bom yes) (on_board yes)
-    (property "Reference" "#PWR033" (id 0) (at 101.6 131.445 0)
+    (property "Reference" "#PWR041" (id 0) (at 101.6 131.445 0)
       (effects (font (size 1.27 1.27)) hide)
     )
@@
   (symbol (lib_id "power:VCC") (at 95.25 85.725 90) (unit 1)
     (in_bom yes) (on_board yes)
-    (property "Reference" "#PWR032" (id 0) (at 99.06 85.725 0)
+    (property "Reference" "#PWR040" (id 0) (at 99.06 85.725 0)
       (effects (font (size 1.27 1.27)) hide)
     )
@@
   (symbol (lib_id "power:GND") (at 167.005 123.825 90) (unit 1)
     (in_bom yes) (on_board yes)
-    (property "Reference" "#PWR038" (id 0) (at 173.355 123.825 0)
+    (property "Reference" "#PWR046" (id 0) (at 173.355 123.825 0)
       (effects (font (size 1.27 1.27)) hide)
     )
@@
   (symbol (lib_id "power:VCC") (at 167.005 83.185 0) (unit 1)
     (in_bom yes) (on_board yes)
-    (property "Reference" "#PWR037" (id 0) (at 167.005 86.995 0)
+    (property "Reference" "#PWR045" (id 0) (at 167.005 86.995 0)
       (effects (font (size 1.27 1.27)) hide)
     )
@@
   (symbol (lib_id "power:GND") (at 107.95 113.665 90) (unit 1)
     (in_bom yes) (on_board yes)
-    (property "Reference" "#PWR034" (id 0) (at 114.3 113.665 0)
+    (property "Reference" "#PWR042" (id 0) (at 114.3 113.665 0)
       (effects (font (size 1.27 1.27)) hide)
     )
@@
   (symbol (lib_id "Device:R_Small") (at 146.05 78.74 180) (unit 1)
     (in_bom yes) (on_board yes)
-    (property "Reference" "R64" (id 0) (at 146.05 78.74 90))
+    (property "Reference" "R72" (id 0) (at 146.05 78.74 90))
     (property "Value" "R_Small" (id 1) (at 144.78 71.12 90))
     (property "Footprint" "" (id 2) (at 146.05 78.74 0)
@@
   (symbol (lib_id "Device:R_Small") (at 140.97 78.74 180) (unit 1)
     (in_bom yes) (on_board yes)
-    (property "Reference" "R62" (id 0) (at 140.97 78.74 90))
+    (property "Reference" "R70" (id 0) (at 140.97 78.74 90))
     (property "Value" "R_Small" (id 1) (at 144.78 71.12 90))
     (property "Footprint" "" (id 2) (at 140.97 78.74 0)
@@
   (symbol (lib_id "Device:LED") (at 138.43 85.09 270) (unit 1)
     (in_bom yes) (on_board yes)
-    (property "Reference" "D56" (id 0) (at 138.43 85.09 0))
+    (property "Reference" "D64" (id 0) (at 138.43 85.09 0))
     (property "Value" "LED" (id 1) (at 134.62 91.44 0))
     (property "Footprint" "" (id 2) (at 138.43 85.09 0)
@@
   (symbol (lib_id "Device:R_Small") (at 130.81 78.74 180) (unit 1)
     (in_bom yes) (on_board yes)
-    (property "Reference" "R58" (id 0) (at 130.81 78.74 90))
+    (property "Reference" "R66" (id 0) (at 130.81 78.74 90))
     (property "Value" "R_Small" (id 1) (at 134.62 71.12 90))
     (property "Footprint" "" (id 2) (at 130.81 78.74 0)
@@
   (symbol (lib_id "Device:LED") (at 148.59 85.09 270) (unit 1)
     (in_bom yes) (on_board yes)
-    (property "Reference" "D60" (id 0) (at 148.59 85.09 0))
+    (property "Reference" "D68" (id 0) (at 148.59 85.09 0))
     (property "Value" "LED" (id 1) (at 144.78 91.44 0))
     (property "Footprint" "" (id 2) (at 148.59 85.09 0)
@@
   (symbol (lib_id "Device:LED") (at 130.81 85.09 270) (unit 1)
     (in_bom yes) (on_board yes)
-    (property "Reference" "D53" (id 0) (at 130.81 85.09 0))
+    (property "Reference" "D61" (id 0) (at 130.81 85.09 0))
     (property "Value" "LED" (id 1) (at 134.62 91.44 0))
     (property "Footprint" "" (id 2) (at 130.81 85.09 0)
@@
   (symbol (lib_id "Device:LED") (at 146.05 85.09 270) (unit 1)
     (in_bom yes) (on_board yes)
-    (property "Reference" "D59" (id 0) (at 146.05 85.09 0))
+    (property "Reference" "D67" (id 0) (at 146.05 85.09 0))
     (property "Value" "LED" (id 1) (at 144.78 91.44 0))
     (property "Footprint" "" (id 2) (at 146.05 85.09 0)
@@
   (symbol (lib_id "Device:R_Small") (at 135.89 78.74 180) (unit 1)
     (in_bom yes) (on_board yes)
-    (property "Reference" "R60" (id 0) (at 135.89 78.74 90))
+    (property "Reference" "R68" (id 0) (at 135.89 78.74 90))
     (property "Value" "R_Small" (id 1) (at 134.62 71.12 90))
     (property "Footprint" "" (id 2) (at 135.89 78.74 0)
@@
   (symbol (lib_id "Device:R_Small") (at 143.51 78.74 180) (unit 1)
     (in_bom yes) (on_board yes)
-    (property "Reference" "R63" (id 0) (at 143.51 78.74 90))
+    (property "Reference" "R71" (id 0) (at 143.51 78.74 90))
     (property "Value" "R_Small" (id 1) (at 144.78 71.12 90))
     (property "Footprint" "" (id 2) (at 143.51 78.74 0)
@@
   (symbol (lib_id "Device:R_Small") (at 133.35 78.74 180) (unit 1)
     (in_bom yes) (on_board yes)
-    (property "Reference" "R59" (id 0) (at 133.35 78.74 90))
+    (property "Reference" "R67" (id 0) (at 133.35 78.74 90))
     (property "Value" "R_Small" (id 1) (at 134.62 71.12 90))
     (property "Footprint" "" (id 2) (at 133.35 78.74 0)
@@
   (symbol (lib_id "Device:LED") (at 135.89 85.09 270) (unit 1)
     (in_bom yes) (on_board yes)
-    (property "Reference" "D55" (id 0) (at 135.89 85.09 0))
+    (property "Reference" "D63" (id 0) (at 135.89 85.09 0))
     (property "Value" "LED" (id 1) (at 134.62 91.44 0))
     (property "Footprint" "" (id 2) (at 135.89 85.09 0)
@@
   (symbol (lib_id "Device:LED") (at 143.51 85.09 270) (unit 1)
     (in_bom yes) (on_board yes)
-    (property "Reference" "D58" (id 0) (at 143.51 85.09 0))
+    (property "Reference" "D66" (id 0) (at 143.51 85.09 0))
     (property "Value" "LED" (id 1) (at 144.78 91.44 0))
     (property "Footprint" "" (id 2) (at 143.51 85.09 0)
@@
   (symbol (lib_id "power:GND") (at 128.27 76.2 270) (unit 1)
     (in_bom yes) (on_board yes) (fields_autoplaced)
-    (property "Reference" "#PWR036" (id 0) (at 121.92 76.2 0)
+    (property "Reference" "#PWR044" (id 0) (at 121.92 76.2 0)
       (effects (font (size 1.27 1.27)) hide)
     )
@@
   (symbol (lib_id "Device:LED") (at 133.35 85.09 270) (unit 1)
     (in_bom yes) (on_board yes)
-    (property "Reference" "D54" (id 0) (at 133.35 85.09 0))
+    (property "Reference" "D62" (id 0) (at 133.35 85.09 0))
     (property "Value" "LED" (id 1) (at 134.62 91.44 0))
     (property "Footprint" "" (id 2) (at 133.35 85.09 0)
@@
   (symbol (lib_id "power:GND") (at 107.95 118.745 90) (unit 1)
     (in_bom yes) (on_board yes)
-    (property "Reference" "#PWR035" (id 0) (at 114.3 118.745 0)
+    (property "Reference" "#PWR043" (id 0) (at 114.3 118.745 0)
       (effects (font (size 1.27 1.27)) hide)
     )
@@
   (symbol (lib_id "Device:LED") (at 140.97 85.09 270) (unit 1)
     (in_bom yes) (on_board yes)
-    (property "Reference" "D57" (id 0) (at 140.97 85.09 0))
+    (property "Reference" "D65" (id 0) (at 140.97 85.09 0))
     (property "Value" "LED" (id 1) (at 144.78 91.44 0))
     (property "Footprint" "" (id 2) (at 140.97 85.09 0)
@@
   (symbol (lib_id "Device:R_Small") (at 138.43 78.74 180) (unit 1)
     (in_bom yes) (on_board yes)
-    (property "Reference" "R61" (id 0) (at 138.43 78.74 90))
+    (property "Reference" "R69" (id 0) (at 138.43 78.74 90))
     (property "Value" "R_Small" (id 1) (at 134.62 71.12 90))
     (property "Footprint" "" (id 2) (at 138.43 78.74 0)
@@
   (symbol (lib_id "Device:R_Small") (at 148.59 78.74 180) (unit 1)
     (in_bom yes) (on_board yes)
-    (property "Reference" "R65" (id 0) (at 148.59 78.74 90))
+    (property "Reference" "R73" (id 0) (at 148.59 78.74 90))
     (property "Value" "R_Small" (id 1) (at 144.78 71.12 90))
     (property "Footprint" "" (id 2) (at 148.59 78.74 0)
