File: Kicad Files/ram.kicad_sch (KiCad schematic)
At the start: 20 parts, among them U13 HM62256BLP, U14 74LS245

Commit message: im sooo stupiiid
Connections:
- net ~{RI} renamed ~{W}
- net ~{RO} renamed ~{R}
Other:
- moved on the sheet: C11, C12, D61, D62, D63, D64, D65, D66, D67, D68, R66, R67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
