File: Kicad Files/8bit-computer.kicad_sch (KiCad schematic)
At the start: 2 parts, among them J1 USB_A

Commit message: work on pc2
Parts:
- added D? (x16): LED, symbol Device:LED
- added R? (x16): R_Small, symbol Device:R_Small
Connections:
- net GND: now also R?.2, R?.2, R?.2, R?.2, R?.2, R?.2, R?.2, R?.2, R?.2, R?.2, R?.2, R?.2, R?.2, R?.2, R?.2, R?.2
- new net: D?.1 (K), R?.1 (x16)
Other:
- sheet MAR ports: added ~{MO}; removed MO
- note added: "TODO: redraw ic possibly 32Bit sigs connect mar,xreg control sigs rework pc to 16bit addr Bus +(control sigs) rework to central lowHigh sigs (PC, MAR,) rework ram"
- note added: "upgrade"
- note removed: "TODO: redraw ic connect mar,xreg control sigs rework pc to 16bit(control sigs)"
