File: Kicad Files/8bit-computer.kicad_sch (KiCad schematic)
At the start: 74 parts, among them J1 USB_A, J2 Conn_01x05_Female, J3 Conn_01x05_Male, J4 Conn_01x08_Male, J5 Conn_01x08_Female, J6 Conn_01x17_Female, J7 Conn_01x17_Male, J8 Conn_01x32_Female, J9 Conn_01x32_Male

Commit message: work on clk
Other:
- sheet IO ports: added ~{CLK}; removed none

Commit message: im sooo stupiiid
Parts:
- renumbered D25 to D17, D26 to D18, D27 to D19, D28 to D20, D29 to D21, D30 to D22, D31 to D23, D32 to D24, D17 to D25, D18 to D26, D19 to D27, D20 to D28, D21 to D29, D22 to D30, D23 to D31, D24 to D32, R25 to R17, R26 to R18, R27 to R19, R28 to R20, R29 to R21, R30 to R22, R31 to R23, R32 to R24, R17 to R25, R18 to R26, R19 to R27, R20 to R28, R21 to R29, R22 to R30, R23 to R31, R24 to R32
Connections:
- no-connect marks 11 -> 10
Other:
- sheet ALU ports: added BF, ~{FO}; removed OF
- sheet Control logic ports: added BF, MS0, ~{FO}, ~{HI}, ~{LI}, ~{R}, ~{W}, ~{ZO}; removed -7, OF, ZMS, ~{MIhb}, ~{MIlb}, ~{RI}, ~{RO}
- sheet MAR ports: added ~{HI}, ~{LI}; removed ~{MIhb}, ~{MIlb}
- sheet RAM ports: added ~{R}, ~{W}; removed ~{RI}, ~{RO}
- sheet Z register ports: added ~{ZO}; removed none
- moved on the sheet: C1, D1, D10, D11, D12, D13, D14, D15, D16, D17, D18, D19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

Commit message: complete redraw to bus system
Parts:
- removed J2: Conn_01x05_Female, symbol Connector:Conn_01x05_Female
- removed J3: Conn_01x05_Male, symbol Connector:Conn_01x05_Male
- removed J4: Conn_01x08_Male, symbol Connector:Conn_01x08_Male
- removed J5: Conn_01x08_Female, symbol Connector:Conn_01x08_Female
- removed J6: Conn_01x17_Female, symbol Connector:Conn_01x17_Female
- removed J7: Conn_01x17_Male, symbol Connector:Conn_01x17_Male
- removed J8: Conn_01x32_Female, symbol Connector:Conn_01x32_Female
- removed J9: Conn_01x32_Male, symbol Connector:Conn_01x32_Male
Connections:
- no-connect marks 10 -> 2
Other:
- added sheet AddrDecoder (addrDecoder.kicad_sch)
- added sheet Data Bus Buffer (dataBusBuffer.kicad_sch)
- added sheet Program Counter (programCounter.kicad_sch)
- added sheet ROM (rom.kicad_sch)
- sheet A register ports: added D0, D1, D2, D3, D4, D5, D6, D7; removed BUS_0, BUS_1, BUS_2, BUS_3, BUS_4, BUS_5, BUS_6, BUS_7
- sheet ALU ports: added D0, D1, D2, D3, D4, D5, D6, D7; removed BUS_0, BUS_1, BUS_2, BUS_3, BUS_4, BUS_5, BUS_6, BUS_7
- sheet B register ports: added D0, D1, D2, D3, D4, D5, D6, D7; removed BUS_0, BUS_1, BUS_2, BUS_3, BUS_4, BUS_5, BUS_6, BUS_7
- sheet IO ports: added R/~{W}, a00, a01, a02, a03, a04, a05, a06, a07, a08, a09, a10, a11, a12, a13, a14, a15, d0, d1, d2, d3, d4, d5, d6, d7; removed ABUS_00, ABUS_01, ABUS_02, ABUS_03, ABUS_04, ABUS_05, ABUS_06, ABUS_07, ABUS_08, ABUS_09, ABUS_10, ABUS_11, ABUS_12, ABUS_13, ABUS_14, ABUS_15, BUS_0, BUS_1, BUS_2, BUS_3, BUS_4, BUS_5, BUS_6, BUS_7, ~{RI}, ~{RO}
- sheet Instruction register ports: added d0, d1, d2, d3, d4, d5, d6, d7; removed BUS_0, BUS_1, BUS_2, BUS_3, BUS_4, BUS_5, BUS_6, BUS_7
- sheet MAR ports: added D0, D1, D2, D3, D4, D5, D6, D7, a00, a01, a02, a03, a04, a05, a06, a07, a08, a09, a10, a11, a12, a13, a14, a15, ~{MIhb}, ~{MIlb}; removed ABUS_00, ABUS_01, ABUS_02, ABUS_03, ABUS_04, ABUS_05, ABUS_06, ABUS_07, ABUS_08, ABUS_09, ABUS_10, ABUS_11, ABUS_12, ABUS_13, ABUS_14, ABUS_15, BUS_0, BUS_1, BUS_2, BUS_3, BUS_4, BUS_5, BUS_6, BUS_7, ~{HI}, ~{LI}
- sheet RAM ports: added R/~{W}, a00, a01, a02, a03, a04, a05, a06, a07, a08, a09, a10, a11, a12, a13, a14, a15, d0, d1, d2, d3, d4, d5, d6, d7, ~{CS}_{RAM}; removed ABUS_00, ABUS_01, ABUS_02, ABUS_03, ABUS_04, ABUS_05, ABUS_06, ABUS_07, ABUS_08, ABUS_09, ABUS_10, ABUS_11, ABUS_12, ABUS_13, ABUS_14, ABUS_15, BUS_0, BUS_1, BUS_2, BUS_3, BUS_4, BUS_5, BUS_6, BUS_7, ~{R}, ~{W}
- sheet X register ports: added D0, D1, D2, D3, D4, D5, D6, D7; removed BUS_0, BUS_1, BUS_2, BUS_3, BUS_4, BUS_5, BUS_6, BUS_7
- sheet Y register ports: added D0, D1, D2, D3, D4, D5, D6, D7; removed BUS_0, BUS_1, BUS_2, BUS_3, BUS_4, BUS_5, BUS_6, BUS_7
- sheet Z register ports: added D0, D1, D2, D3, D4, D5, D6, D7; removed BUS_0, BUS_1, BUS_2, BUS_3, BUS_4, BUS_5, BUS_6, BUS_7
- note added: "Address Section"
- note added: "Control Section"
- note added: "Memory Section"
- note added: "Register Section"
- note added: "TODO: R/W ALU rethink"
- note removed: "TODO: BOM"
- moved on the sheet: C1, D1, D10, D11, D12, D13, D14, D15, D16, D17, D18, D19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

Commit message: update
Parts:
- removed C1: C_Polarized, symbol Device:C_Polarized
- removed D1, D10, D11, D12, D13, D14, D15, D16, D17, D18, D19, D2, D20, D21, D22, D23, D24, D25, D26, D27, D28, D29, D3, D30, D31, D32, D4, D5, D6, D7, D8, D9: LED, symbol Device:LED
- removed J1: USB_A, symbol Connector:USB_A
- removed R24, R25, R26, R27, R28, R29, R30, R31, R32: R_Small, symbol Device:R_Small
- added C8: C_Polarized, symbol Device:C_Polarized
- added D1, D10, D11, D12, D13, D14, D15, D16, D17, D18, D19, D2, D20, D21, D22, D23, D3, D4, D5, D6, D7, D8, D9: LED_Small, symbol Device:LED_Small
Connections:
- net GND: now also C8.2; no longer R16.2, R17.2, R18.2, R19.2, R20.2, R21.2, R22.2, R23.2
- net VCC: now also C8.1
- net at R21.1: now also D21.1 (K)
- net at R16.1: now also D16.1 (K)
- net at R10.1: now also D10.1 (K)
- net at R13.1: now also D13.1 (K)
- net at R23.1: now also D23.1 (K)
- net at R1.1: now also D1.1 (K)
- net at R7.1: now also D7.1 (K)
- net at R3.1: now also D3.1 (K)
- net at R20.1: now also D20.1 (K)
- net at R6.1: now also D6.1 (K)
- net at R9.1: now also D9.1 (K)
- net at R14.1: now also D14.1 (K)
- net at R12.1: now also D12.1 (K)
- net at R19.1: now also D19.1 (K)
- net at R15.1: now also D15.1 (K)
- net at R4.1: now also D4.1 (K)
- net at R8.1: now also D8.1 (K)
- net at R2.1: now also D2.1 (K)
- net at R17.1: now also D17.1 (K)
- net at R5.1: now also D5.1 (K)
- net at R11.1: now also D11.1 (K)
- net at R22.1: now also D22.1 (K)
- net at R18.1: now also D18.1 (K)
- new net: D1.2 (A), D2.2 (A), D3.2 (A), D4.2 (A), D5.2 (A), D6.2 (A), D7.2 (A), D8.2 (A)
- new net: D10.2 (A), D11.2 (A), D12.2 (A), D13.2 (A), D14.2 (A), D15.2 (A), D9.2 (A)
- new net: D16.2 (A), D17.2 (A), D18.2 (A), D19.2 (A), D20.2 (A), D21.2 (A), D22.2 (A), D23.2 (A)
- new net: R16.2, R17.2, R18.2, R19.2, R20.2, R21.2, R22.2, R23.2
- no-connect marks 2 -> 0
Other:
- sheet Control logic renamed Instruction Decode
- sheet IO renamed DEBUG
- removed sheet B register
- added sheet Interrupt Logic (il.kicad_sch)
- added sheet Processor Status Register (preg.kicad_sch)
- added sheet StackPointer (sp.kicad_sch)
- added sheet VIA (via.kicad_sch)
- sheet A register: file a-register.kicad_sch -> areg.kicad_sch
- sheet A register ports: added d_{i}0, d_{i}1, d_{i}2, d_{i}3, d_{i}4, d_{i}5, d_{i}6, d_{i}7, ~{A}_{I}, ~{A}_{O}; removed D0, D1, D2, D3, D4, D5, D6, D7, ~{AI}, ~{AO}
- sheet ALU ports: added F_C, F_N, F_V, F_Z, d_{i}0, d_{i}1, d_{i}2, d_{i}3, d_{i}4, d_{i}5, d_{i}6, d_{i}7, ~{F}, ~{Σ}_{O}; removed BF, B_0, B_1, B_2, B_3, B_4, B_5, B_6, B_7, CF, D0, D1, D2, D3, D4, D5, D6, D7, NF, ZF, ~{FI}, ~{FO}, ~{ΣO}
- sheet AddrDecoder: file addrDecoder.kicad_sch -> addrdec.kicad_sch
- sheet AddrDecoder ports: added R/~{W}, ~{CS}_{VIA}, ~{R}/W; removed ~{CS}_{2}
- sheet Clock: file clock.kicad_sch -> clk.kicad_sch
- sheet Clock ports: added none; removed ~{CLK}
- sheet DEBUG: file IO.kicad_sch -> debug.kicad_sch
- sheet DEBUG ports: added d_{e}0, d_{e}1, d_{e}2, d_{e}3, d_{e}4, d_{e}5, d_{e}6, d_{e}7; removed CLR, HLT, OVRD, d0, d1, d2, d3, d4, d5, d6, d7, ~{CLK}
- sheet Data Bus Buffer: file dataBusBuffer.kicad_sch -> dbb.kicad_sch
- sheet Data Bus Buffer ports: added R/~{W}, d_{e}0, d_{e}1, d_{e}2, d_{e}3, d_{e}4, d_{e}5, d_{e}6, d_{e}7, d_{i}0, d_{i}1, d_{i}2, d_{i}3, d_{i}4, d_{i}5, d_{i}6, d_{i}7, ~{D_{O}}; removed D0, D1, D2, D3, D4, D5, D6, D7
- sheet Instruction Decode: file control.kicad_sch -> id.kicad_sch
- sheet Instruction Decode ports: added CLK, F_4, F_5, F_6, F_7, F_C, F_N, F_V, F_Z, H/~{L}, I_0, I_1, I_2, I_3, I_4, I_5, I_6, I_7, R/~{W}, Z_{I}, ~{A}_{I}, ~{A}_{O}, ~{D_{O}}, ~{F}, ~{I}_{I}, ~{I}_{O}, ~{M_{I}}, ~{M_{O}}, ~{PC_{I}}, ~{PC_{Oa}}, ~{PC_{Od}}, ~{P}_{I}, ~{P}_{O}, ~{R}/W, ~{SP_{I}}, ~{SP_{Oa}}, ~{SP_{Od}}, ~{X_{I}}, ~{X_{Oa}}, ~{X_{Od}}, ~{Y_{I}}, ~{Y_{Oa}}, ~{Y_{Od}}, ~{Z}_{O}, ~{Σ}_{O}; removed -0, -1, -2, -3, -4, -5, -6, BF, CF, IR_0, IR_1, IR_2, IR_3, IR_4, IR_5, IR_6, IR_7, MS0, NF, OVRD, ZF, ZI, ~{AI}, ~{AO}, ~{BI}, ~{BO}, ~{CLK}, ~{FI}, ~{FO}, ~{HI}, ~{II}, ~{IO}, ~{LI}, ~{MO}, ~{R}, ~{W}, ~{XI}, ~{XO}, ~{YI}, ~{YO}, ~{ZO}, ~{ΣO}
- sheet Instruction register: file inst-register.kicad_sch -> ireg.kicad_sch
- sheet Instruction register ports: added I_0, I_1, I_2, I_3, I_4, I_5, I_6, I_7, d_{e}0, d_{e}1, d_{e}2, d_{e}3, d_{e}4, d_{e}5, d_{e}6, d_{e}7, ~{I}_{I}, ~{I}_{O}; removed IR_0, IR_1, IR_2, IR_3, IR_4, IR_5, IR_6, IR_7, d0, d1, d2, d3, d4, d5, d6, d7, ~{II}, ~{IO}
- sheet MAR ports: added H/~{L}, d_{i}0, d_{i}1, d_{i}2, d_{i}3, d_{i}4, d_{i}5, d_{i}6, d_{i}7, ~{M_{I}}, ~{M_{O}}; removed D0, D1, D2, D3, D4, D5, D6, D7, ~{MIhb}, ~{MIlb}, ~{MO}
- sheet Program Counter: file programCounter.kicad_sch -> pc.kicad_sch
- sheet Program Counter ports: added CLK, CLR, H/~{L}, PC_{INC}, PC_{I}, PC_{Od}, d_{i}0, d_{i}1, d_{i}2, d_{i}3, d_{i}4, d_{i}5, d_{i}6, d_{i}7, ~{PC_{Oa}}; removed D0, D1, D2, D3, D4, D5, D6, D7
- sheet RAM ports: added d_{e}0, d_{e}1, d_{e}2, d_{e}3, d_{e}4, d_{e}5, d_{e}6, d_{e}7; removed d0, d1, d2, d3, d4, d5, d6, d7
- sheet ROM ports: added d_{e}0, d_{e}1, d_{e}2, d_{e}3, d_{e}4, d_{e}5, d_{e}6, d_{e}7, ~{R}/W; removed R/~{W}, d0, d1, d2, d3, d4, d5, d6, d7
- sheet X register: file x-register.kicad_sch -> xreg.kicad_sch
- sheet X register ports: added a00, a01, a02, a03, a04, a05, a06, a07, d_{i}0, d_{i}1, d_{i}2, d_{i}3, d_{i}4, d_{i}5, d_{i}6, d_{i}7, ~{X_{I}}, ~{X_{Oa}}, ~{X_{Od}}; removed D0, D1, D2, D3, D4, D5, D6, D7, ~{XI}, ~{XO}
- sheet Y register: file y-register.kicad_sch -> yreg.kicad_sch
- sheet Y register ports: added a08, a09, a10, a11, a12, a13, a14, a15, d_{i}0, d_{i}1, d_{i}2, d_{i}3, d_{i}4, d_{i}5, d_{i}6, d_{i}7, ~{Y_{I}}, ~{Y_{Oa}}, ~{Y_{Od}}; removed D0, D1, D2, D3, D4, D5, D6, D7, ~{YI}, ~{YO}
- sheet Z register: file Z register.kicad_sch -> zreg.kicad_sch
- sheet Z register ports: added Z_{I}, d_{i}0, d_{i}1, d_{i}2, d_{i}3, d_{i}4, d_{i}5, d_{i}6, d_{i}7, ~{Z}_{O}; removed D0, D1, D2, D3, D4, D5, D6, D7, ZI, ~{ZO}
- note added: "ADDRESS BUS"
- note added: "Color Conventions: red = data orange = internal data tx yellow = control green = interal data rx blue = external data bus purple = address bus white = clk"
- note added: "EXT DATA BUS"
- note added: "INT DATA BUS"
- note added: "TODO: PC draw ALU rethink CL rethink interrupts instruction layout timing control?"
- note added: "done"
- note removed: "TODO: R/W ALU rethink"

Commit message: rethink alu
Other:
- note added: "eTODO: color coding LED PC draw ALU rethink CL rethink interrupts instruction layout timing control?"
- note removed: "TODO: PC draw ALU rethink CL rethink interrupts instruction layout timing control?"
Changed lines of the file:
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@@
     (stroke (width 0) (type default))
+  )
+  (text "done" (at 220.345 242.57 0)
+    (effects (font (size 1.524 1.524)) (justify left bottom))
   )
   (text "Control Section\n" (at 50.8 74.93 0)
@@
     (effects (font (size 1.524 1.524)) (justify left bottom))
   )
-  (text "TODO:\nPC draw\nALU rethink\nCL rethink\n	interrupts\n	instruction layout\n	timing control?\n"
+  (text "eTODO:\ncolor coding LED\nPC draw\nALU rethink\nCL rethink\n	interrupts\n	instruction layout\n	timing control?\n"
     (at 27.94 31.75 0)
     (effects (font (size 1.524 1.524)) (justify left bottom))
@@
     (effects (font (size 1.524 1.524)) (justify left bottom))
   )
+  (text "done" (at 167.005 165.1 0)
+    (effects (font (size 1.524 1.524)) (justify left bottom))
+  )
