File: Kicad Files/Flags register.kicad_sch (KiCad schematic)
At the start: 20 parts

Commit message: started tidy up in control
Parts:
- gave numbers to parts that had none: 20
Changed lines of the file:
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@@
   (symbol (lib_id "74xx:74LS173") (at 203.2 73.66 0) (unit 1)
     (in_bom yes) (on_board yes)
-    (property "Reference" "" (id 0) (at 203.2 46.2026 0))
+    (property "Reference" "U8" (id 0) (at 203.2 46.2026 0))
     (property "Value" "74LS173" (id 1) (at 203.2 48.514 0))
     (property "Footprint" "" (id 2) (at 203.2 73.66 0)
@@
   (symbol (lib_id "Device:LED") (at 240.03 44.45 270) (unit 1)
     (in_bom yes) (on_board yes)
-    (property "Reference" "" (id 0) (at 242.062 43.1038 0)
+    (property "Reference" "D40" (id 0) (at 242.062 43.1038 0)
       (effects (font (size 1.27 1.27)) (justify top) hide)
     )
@@
   (symbol (lib_id "Device:LED") (at 233.68 44.45 270) (unit 1)
     (in_bom yes) (on_board yes)
-    (property "Reference" "" (id 0) (at 235.712 43.1038 0)
+    (property "Reference" "D39" (id 0) (at 235.712 43.1038 0)
       (effects (font (size 1.27 1.27)) (justify top) hide)
     )
@@
   (symbol (lib_id "Device:LED") (at 227.33 44.45 270) (unit 1)
     (in_bom yes) (on_board yes)
-    (property "Reference" "" (id 0) (at 229.362 43.1038 0)
+    (property "Reference" "D38" (id 0) (at 229.362 43.1038 0)
       (effects (font (size 1.27 1.27)) (justify top) hide)
     )
@@
   (symbol (lib_id "Device:LED") (at 220.98 44.45 270) (unit 1)
     (in_bom yes) (on_board yes)
-    (property "Reference" "" (id 0) (at 223.012 43.1038 0)
+    (property "Reference" "D37" (id 0) (at 223.012 43.1038 0)
       (effects (font (size 1.27 1.27)) (justify top) hide)
     )
@@
   (symbol (lib_id "Device:R") (at 220.98 36.83 0) (unit 1)
     (in_bom yes) (on_board yes)
-    (property "Reference" "" (id 0) (at 217.8304 37.1856 90)
+    (property "Reference" "R45" (id 0) (at 217.8304 37.1856 90)
       (effects (font (size 1.27 1.27)) (justify top))
     )
@@
   (symbol (lib_id "Device:R") (at 240.03 36.83 0) (unit 1)
     (in_bom yes) (on_board yes)
-    (property "Reference" "" (id 0) (at 236.8804 37.1856 90)
+    (property "Reference" "R48" (id 0) (at 236.8804 37.1856 90)
       (effects (font (size 1.27 1.27)) (justify top))
     )
@@
   (symbol (lib_id "Device:R") (at 233.68 36.83 0) (unit 1)
     (in_bom yes) (on_board yes)
-    (property "Reference" "" (id 0) (at 230.5304 37.1856 90)
+    (property "Reference" "R47" (id 0) (at 230.5304 37.1856 90)
       (effects (font (size 1.27 1.27)) (justify top))
     )
@@
   (symbol (lib_id "Device:R") (at 227.33 36.83 0) (unit 1)
     (in_bom yes) (on_board yes)
-    (property "Reference" "" (id 0) (at 224.1804 37.1856 90)
+    (property "Reference" "R46" (id 0) (at 224.1804 37.1856 90)
       (effects (font (size 1.27 1.27)) (justify top))
     )
@@
   (symbol (lib_id "74xx:74LS00") (at 119.38 69.85 0) (unit 1)
     (in_bom yes) (on_board yes)
-    (property "Reference" "" (id 0) (at 119.38 61.595 0))
+    (property "Reference" "U6" (id 0) (at 119.38 61.595 0))
     (property "Value" "74LS00" (id 1) (at 119.38 63.9064 0))
     (property "Footprint" "" (id 2) (at 119.38 69.85 0)
@@
   (symbol (lib_id "74xx:74LS00") (at 134.62 76.2 0) (unit 1)
     (in_bom yes) (on_board yes)
-    (property "Reference" "" (id 0) (at 134.62 67.945 0))
+    (property "Reference" "U9" (id 0) (at 134.62 67.945 0))
     (property "Value" "74LS00" (id 1) (at 134.62 70.2564 0))
     (property "Footprint" "" (id 2) (at 134.62 76.2 0)
@@
   (symbol (lib_id "74xx:74LS00") (at 134.62 63.5 0) (unit 1)
     (in_bom yes) (on_board yes)
-    (property "Reference" "" (id 0) (at 134.62 55.245 0))
+    (property "Reference" "U5" (id 0) (at 134.62 55.245 0))
     (property "Value" "74LS00" (id 1) (at 134.62 57.5564 0))
     (property "Footprint" "" (id 2) (at 134.62 63.5 0)
@@
   (symbol (lib_id "74xx:74LS00") (at 149.86 69.85 0) (unit 1)
     (in_bom yes) (on_board yes)
-    (property "Reference" "" (id 0) (at 149.86 61.595 0))
+    (property "Reference" "U7" (id 0) (at 149.86 61.595 0))
     (property "Value" "74LS00" (id 1) (at 149.86 63.9064 0))
     (property "Footprint" "" (id 2) (at 149.86 69.85 0)
@@
   (symbol (lib_id "74xx:74LS02") (at 124.46 85.09 0) (unit 1)
     (in_bom yes) (on_board yes)
-    (property "Reference" "" (id 0) (at 124.46 76.835 0))
+    (property "Reference" "U10" (id 0) (at 124.46 76.835 0))
     (property "Value" "74LS02" (id 1) (at 124.46 79.1464 0))
     (property "Footprint" "" (id 2) (at 124.46 85.09 0)
@@
   (symbol (lib_id "74xx:74LS08") (at 154.94 100.33 0) (unit 1)
     (in_bom yes) (on_board yes)
-    (property "Reference" "" (id 0) (at 154.94 92.075 0))
+    (property "Reference" "U13" (id 0) (at 154.94 92.075 0))
     (property "Value" "74LS08" (id 1) (at 154.94 94.3864 0))
     (property "Footprint" "" (id 2) (at 154.94 100.33 0)
@@
   (symbol (lib_id "74xx:74LS08") (at 139.7 87.63 0) (unit 1)
     (in_bom yes) (on_board yes)
-    (property "Reference" "" (id 0) (at 139.7 79.375 0))
+    (property "Reference" "U11" (id 0) (at 139.7 79.375 0))
     (property "Value" "74LS08" (id 1) (at 139.7 81.6864 0))
     (property "Footprint" "" (id 2) (at 139.7 87.63 0)
@@
   (symbol (lib_id "74xx:74LS08") (at 139.7 113.03 0) (unit 1)
     (in_bom yes) (on_board yes)
-    (property "Reference" "" (id 0) (at 139.7 104.775 0))
+    (property "Reference" "U15" (id 0) (at 139.7 104.775 0))
     (property "Value" "74LS08" (id 1) (at 139.7 107.0864 0))
     (property "Footprint" "" (id 2) (at 139.7 113.03 0)
@@
   (symbol (lib_id "74xx:74LS02") (at 124.46 95.25 0) (unit 1)
     (in_bom yes) (on_board yes)
-    (property "Reference" "" (id 0) (at 124.46 86.995 0))
+    (property "Reference" "U12" (id 0) (at 124.46 86.995 0))
     (property "Value" "74LS02" (id 1) (at 124.46 89.3064 0))
     (property "Footprint" "" (id 2) (at 124.46 95.25 0)
@@
   (symbol (lib_id "74xx:74LS02") (at 124.46 105.41 0) (unit 1)
     (in_bom yes) (on_board yes)
-    (property "Reference" "" (id 0) (at 124.46 97.155 0))
+    (property "Reference" "U14" (id 0) (at 124.46 97.155 0))
     (property "Value" "74LS02" (id 1) (at 124.46 99.4664 0))
     (property "Footprint" "" (id 2) (at 124.46 105.41 0)
@@
   (symbol (lib_id "74xx:74LS02") (at 124.46 115.57 0) (unit 1)
     (in_bom yes) (on_board yes)
-    (property "Reference" "" (id 0) (at 124.46 107.315 0))
+    (property "Reference" "U16" (id 0) (at 124.46 107.315 0))
     (property "Value" "74LS02" (id 1) (at 124.46 109.6264 0))
     (property "Footprint" "" (id 2) (at 124.46 115.57 0)

Commit message: work on cl
Parts:
- D104: renamed from D37; value GREEN -> LED
- D105: renamed from D38; value GREEN -> LED
- D106: renamed from D39; value GREEN -> LED
- D107: renamed from D40; value GREEN -> LED
- R139: renamed from R45; value 220 -> R
- R140: renamed from R46; value 220 -> R
- R141: renamed from R47; value 220 -> R
- R142: renamed from R48; value 220 -> R
- renumbered U6 to U53, U10 to U54, U12 to U55, U14 to U56, U16 to U57, U5 to U58, U9 to U59, U11 to U60, U15 to U61, U7 to U62, U13 to U63, U8 to U64
Changed lines of the file:
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@@
   (symbol (lib_id "74xx:74LS173") (at 203.2 73.66 0) (unit 1)
     (in_bom yes) (on_board yes)
-    (property "Reference" "U8" (id 0) (at 203.2 46.2026 0))
+    (property "Reference" "U64" (id 0) (at 203.2 46.2026 0))
     (property "Value" "74LS173" (id 1) (at 203.2 48.514 0))
     (property "Footprint" "" (id 2) (at 203.2 73.66 0)
@@
   (symbol (lib_id "Device:LED") (at 240.03 44.45 270) (unit 1)
     (in_bom yes) (on_board yes)
-    (property "Reference" "D40" (id 0) (at 242.062 43.1038 0)
+    (property "Reference" "D107" (id 0) (at 242.062 43.1038 0)
       (effects (font (size 1.27 1.27)) (justify top) hide)
     )
-    (property "Value" "GREEN" (id 1) (at 242.062 45.4152 0)
+    (property "Value" "LED" (id 1) (at 242.062 45.4152 0)
       (effects (font (size 1.27 1.27)) (justify bottom))
     )
@@
   (symbol (lib_id "Device:LED") (at 233.68 44.45 270) (unit 1)
     (in_bom yes) (on_board yes)
-    (property "Reference" "D39" (id 0) (at 235.712 43.1038 0)
+    (property "Reference" "D106" (id 0) (at 235.712 43.1038 0)
       (effects (font (size 1.27 1.27)) (justify top) hide)
     )
-    (property "Value" "GREEN" (id 1) (at 235.712 45.4152 0)
+    (property "Value" "LED" (id 1) (at 235.712 45.4152 0)
       (effects (font (size 1.27 1.27)) (justify bottom))
     )
@@
   (symbol (lib_id "Device:LED") (at 227.33 44.45 270) (unit 1)
     (in_bom yes) (on_board yes)
-    (property "Reference" "D38" (id 0) (at 229.362 43.1038 0)
+    (property "Reference" "D105" (id 0) (at 229.362 43.1038 0)
       (effects (font (size 1.27 1.27)) (justify top) hide)
     )
-    (property "Value" "GREEN" (id 1) (at 229.362 45.4152 0)
+    (property "Value" "LED" (id 1) (at 229.362 45.4152 0)
       (effects (font (size 1.27 1.27)) (justify bottom))
     )
@@
   (symbol (lib_id "Device:LED") (at 220.98 44.45 270) (unit 1)
     (in_bom yes) (on_board yes)
-    (property "Reference" "D37" (id 0) (at 223.012 43.1038 0)
+    (property "Reference" "D104" (id 0) (at 223.012 43.1038 0)
       (effects (font (size 1.27 1.27)) (justify top) hide)
     )
-    (property "Value" "GREEN" (id 1) (at 223.012 45.4152 0)
+    (property "Value" "LED" (id 1) (at 223.012 45.4152 0)
       (effects (font (size 1.27 1.27)) (justify bottom))
     )
@@
   (symbol (lib_id "Device:R") (at 220.98 36.83 0) (unit 1)
     (in_bom yes) (on_board yes)
-    (property "Reference" "R45" (id 0) (at 217.8304 37.1856 90)
+    (property "Reference" "R139" (id 0) (at 217.8304 37.1856 90)
       (effects (font (size 1.27 1.27)) (justify top))
     )
-    (property "Value" "220" (id 1) (at 223.3168 37.1856 90))
+    (property "Value" "R" (id 1) (at 223.3168 37.1856 90))
     (property "Footprint" "" (id 2) (at 219.202 36.83 90)
       (effects (font (size 1.27 1.27)) hide)
@@
   (symbol (lib_id "Device:R") (at 240.03 36.83 0) (unit 1)
     (in_bom yes) (on_board yes)
-    (property "Reference" "R48" (id 0) (at 236.8804 37.1856 90)
+    (property "Reference" "R142" (id 0) (at 236.8804 37.1856 90)
       (effects (font (size 1.27 1.27)) (justify top))
     )
-    (property "Value" "220" (id 1) (at 242.3668 37.1856 90))
+    (property "Value" "R" (id 1) (at 242.3668 37.1856 90))
     (property "Footprint" "" (id 2) (at 238.252 36.83 90)
       (effects (font (size 1.27 1.27)) hide)
@@
   (symbol (lib_id "Device:R") (at 233.68 36.83 0) (unit 1)
     (in_bom yes) (on_board yes)
-    (property "Reference" "R47" (id 0) (at 230.5304 37.1856 90)
+    (property "Reference" "R141" (id 0) (at 230.5304 37.1856 90)
       (effects (font (size 1.27 1.27)) (justify top))
     )
-    (property "Value" "220" (id 1) (at 236.0168 37.1856 90))
+    (property "Value" "R" (id 1) (at 236.0168 37.1856 90))
     (property "Footprint" "" (id 2) (at 231.902 36.83 90)
       (effects (font (size 1.27 1.27)) hide)
@@
   (symbol (lib_id "Device:R") (at 227.33 36.83 0) (unit 1)
     (in_bom yes) (on_board yes)
-    (property "Reference" "R46" (id 0) (at 224.1804 37.1856 90)
+    (property "Reference" "R140" (id 0) (at 224.1804 37.1856 90)
       (effects (font (size 1.27 1.27)) (justify top))
     )
-    (property "Value" "220" (id 1) (at 229.6668 37.1856 90))
+    (property "Value" "R" (id 1) (at 229.6668 37.1856 90))
     (property "Footprint" "" (id 2) (at 225.552 36.83 90)
       (effects (font (size 1.27 1.27)) hide)
@@
   (symbol (lib_id "power:GND") (at 247.65 29.21 0) (unit 1)
     (in_bom yes) (on_board yes)
-    (property "Reference" "#PWR031" (id 0) (at 247.65 35.56 0)
+    (property "Reference" "#PWR0140" (id 0) (at 247.65 35.56 0)
       (effects (font (size 1.27 1.27)) hide)
     )
@@
   (symbol (lib_id "power:GND") (at 203.2 96.52 0) (unit 1)
     (in_bom yes) (on_board yes)
-    (property "Reference" "#PWR034" (id 0) (at 203.2 102.87 0)
+    (property "Reference" "#PWR0138" (id 0) (at 203.2 102.87 0)
       (effects (font (size 1.27 1.27)) hide)
     )
@@
   (symbol (lib_id "power:VCC") (at 210.82 50.8 0) (unit 1)
     (in_bom yes) (on_board yes)
-    (property "Reference" "#PWR032" (id 0) (at 210.82 54.61 0)
+    (property "Reference" "#PWR0139" (id 0) (at 210.82 54.61 0)
       (effects (font (size 1.27 1.27)) hide)
     )
@@
   (symbol (lib_id "power:GND") (at 185.42 73.66 0) (unit 1)
     (in_bom yes) (on_board yes)
-    (property "Reference" "#PWR033" (id 0) (at 185.42 80.01 0)
+    (property "Reference" "#PWR0137" (id 0) (at 185.42 80.01 0)
       (effects (font (size 1.27 1.27)) hide)
     )
@@
   (symbol (lib_id "74xx:74LS00") (at 119.38 69.85 0) (unit 1)
     (in_bom yes) (on_board yes)
-    (property "Reference" "U6" (id 0) (at 119.38 61.595 0))
+    (property "Reference" "U53" (id 0) (at 119.38 61.595 0))
     (property "Value" "74LS00" (id 1) (at 119.38 63.9064 0))
     (property "Footprint" "" (id 2) (at 119.38 69.85 0)
@@
   (symbol (lib_id "74xx:74LS00") (at 134.62 76.2 0) (unit 1)
     (in_bom yes) (on_board yes)
-    (property "Reference" "U9" (id 0) (at 134.62 67.945 0))
+    (property "Reference" "U59" (id 0) (at 134.62 67.945 0))
     (property "Value" "74LS00" (id 1) (at 134.62 70.2564 0))
     (property "Footprint" "" (id 2) (at 134.62 76.2 0)
@@
   (symbol (lib_id "74xx:74LS00") (at 134.62 63.5 0) (unit 1)
     (in_bom yes) (on_board yes)
-    (property "Reference" "U5" (id 0) (at 134.62 55.245 0))
+    (property "Reference" "U58" (id 0) (at 134.62 55.245 0))
     (property "Value" "74LS00" (id 1) (at 134.62 57.5564 0))
     (property "Footprint" "" (id 2) (at 134.62 63.5 0)
@@
   (symbol (lib_id "74xx:74LS00") (at 149.86 69.85 0) (unit 1)
     (in_bom yes) (on_board yes)
-    (property "Reference" "U7" (id 0) (at 149.86 61.595 0))
+    (property "Reference" "U62" (id 0) (at 149.86 61.595 0))
     (property "Value" "74LS00" (id 1) (at 149.86 63.9064 0))
     (property "Footprint" "" (id 2) (at 149.86 69.85 0)
@@
   (symbol (lib_id "74xx:74LS02") (at 124.46 85.09 0) (unit 1)
     (in_bom yes) (on_board yes)
-    (property "Reference" "U10" (id 0) (at 124.46 76.835 0))
+    (property "Reference" "U54" (id 0) (at 124.46 76.835 0))
     (property "Value" "74LS02" (id 1) (at 124.46 79.1464 0))
     (property "Footprint" "" (id 2) (at 124.46 85.09 0)
@@
   (symbol (lib_id "74xx:74LS08") (at 154.94 100.33 0) (unit 1)
     (in_bom yes) (on_board yes)
-    (property "Reference" "U13" (id 0) (at 154.94 92.075 0))
+    (property "Reference" "U63" (id 0) (at 154.94 92.075 0))
     (property "Value" "74LS08" (id 1) (at 154.94 94.3864 0))
     (property "Footprint" "" (id 2) (at 154.94 100.33 0)
@@
   (symbol (lib_id "74xx:74LS08") (at 139.7 87.63 0) (unit 1)
     (in_bom yes) (on_board yes)
-    (property "Reference" "U11" (id 0) (at 139.7 79.375 0))
+    (property "Reference" "U60" (id 0) (at 139.7 79.375 0))
     (property "Value" "74LS08" (id 1) (at 139.7 81.6864 0))
     (property "Footprint" "" (id 2) (at 139.7 87.63 0)
@@
   (symbol (lib_id "74xx:74LS08") (at 139.7 113.03 0) (unit 1)
     (in_bom yes) (on_board yes)
-    (property "Reference" "U15" (id 0) (at 139.7 104.775 0))
+    (property "Reference" "U61" (id 0) (at 139.7 104.775 0))
     (property "Value" "74LS08" (id 1) (at 139.7 107.0864 0))
     (property "Footprint" "" (id 2) (at 139.7 113.03 0)
@@
   (symbol (lib_id "74xx:74LS02") (at 124.46 95.25 0) (unit 1)
     (in_bom yes) (on_board yes)
-    (property "Reference" "U12" (id 0) (at 124.46 86.995 0))
+    (property "Reference" "U55" (id 0) (at 124.46 86.995 0))
     (property "Value" "74LS02" (id 1) (at 124.46 89.3064 0))
     (property "Footprint" "" (id 2) (at 124.46 95.25 0)
@@
   (symbol (lib_id "74xx:74LS02") (at 124.46 105.41 0) (unit 1)
     (in_bom yes) (on_board yes)
-    (property "Reference" "U14" (id 0) (at 124.46 97.155 0))
+    (property "Reference" "U56" (id 0) (at 124.46 97.155 0))
     (property "Value" "74LS02" (id 1) (at 124.46 99.4664 0))
     (property "Footprint" "" (id 2) (at 124.46 105.41 0)
@@
   (symbol (lib_id "74xx:74LS02") (at 124.46 115.57 0) (unit 1)
     (in_bom yes) (on_board yes)
-    (property "Reference" "U16" (id 0) (at 124.46 107.315 0))
+    (property "Reference" "U57" (id 0) (at 124.46 107.315 0))
     (property "Value" "74LS02" (id 1) (at 124.46 109.6264 0))
     (property "Footprint" "" (id 2) (at 124.46 115.57 0)

Commit message: fixed ecc problems
Parts:
- renumbered U53 to U56, U54 to U57, U55 to U58, U56 to U59, U57 to U60, U58 to U61, U59 to U62, U60 to U63, U61 to U64, U62 to U65, U63 to U66, U64 to U67
Changed lines of the file:
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@@
   (symbol (lib_id "74xx:74LS173") (at 203.2 73.66 0) (unit 1)
     (in_bom yes) (on_board yes)
-    (property "Reference" "U64" (id 0) (at 203.2 46.2026 0))
+    (property "Reference" "U67" (id 0) (at 203.2 46.2026 0))
     (property "Value" "74LS173" (id 1) (at 203.2 48.514 0))
     (property "Footprint" "" (id 2) (at 203.2 73.66 0)
@@
   (symbol (lib_id "power:GND") (at 247.65 29.21 0) (unit 1)
     (in_bom yes) (on_board yes)
-    (property "Reference" "#PWR0140" (id 0) (at 247.65 35.56 0)
+    (property "Reference" "#PWR0162" (id 0) (at 247.65 35.56 0)
       (effects (font (size 1.27 1.27)) hide)
     )
@@
   (symbol (lib_id "power:GND") (at 203.2 96.52 0) (unit 1)
     (in_bom yes) (on_board yes)
-    (property "Reference" "#PWR0138" (id 0) (at 203.2 102.87 0)
+    (property "Reference" "#PWR0160" (id 0) (at 203.2 102.87 0)
       (effects (font (size 1.27 1.27)) hide)
     )
@@
   (symbol (lib_id "power:VCC") (at 210.82 50.8 0) (unit 1)
     (in_bom yes) (on_board yes)
-    (property "Reference" "#PWR0139" (id 0) (at 210.82 54.61 0)
+    (property "Reference" "#PWR0161" (id 0) (at 210.82 54.61 0)
       (effects (font (size 1.27 1.27)) hide)
     )
@@
   (symbol (lib_id "power:GND") (at 185.42 73.66 0) (unit 1)
     (in_bom yes) (on_board yes)
-    (property "Reference" "#PWR0137" (id 0) (at 185.42 80.01 0)
+    (property "Reference" "#PWR0159" (id 0) (at 185.42 80.01 0)
       (effects (font (size 1.27 1.27)) hide)
     )
@@
   (symbol (lib_id "74xx:74LS00") (at 119.38 69.85 0) (unit 1)
     (in_bom yes) (on_board yes)
-    (property "Reference" "U53" (id 0) (at 119.38 61.595 0))
+    (property "Reference" "U56" (id 0) (at 119.38 61.595 0))
     (property "Value" "74LS00" (id 1) (at 119.38 63.9064 0))
     (property "Footprint" "" (id 2) (at 119.38 69.85 0)
@@
   (symbol (lib_id "74xx:74LS00") (at 134.62 76.2 0) (unit 1)
     (in_bom yes) (on_board yes)
-    (property "Reference" "U59" (id 0) (at 134.62 67.945 0))
+    (property "Reference" "U62" (id 0) (at 134.62 67.945 0))
     (property "Value" "74LS00" (id 1) (at 134.62 70.2564 0))
     (property "Footprint" "" (id 2) (at 134.62 76.2 0)
@@
   (symbol (lib_id "74xx:74LS00") (at 134.62 63.5 0) (unit 1)
     (in_bom yes) (on_board yes)
-    (property "Reference" "U58" (id 0) (at 134.62 55.245 0))
+    (property "Reference" "U61" (id 0) (at 134.62 55.245 0))
     (property "Value" "74LS00" (id 1) (at 134.62 57.5564 0))
     (property "Footprint" "" (id 2) (at 134.62 63.5 0)
@@
   (symbol (lib_id "74xx:74LS00") (at 149.86 69.85 0) (unit 1)
     (in_bom yes) (on_board yes)
-    (property "Reference" "U62" (id 0) (at 149.86 61.595 0))
+    (property "Reference" "U65" (id 0) (at 149.86 61.595 0))
     (property "Value" "74LS00" (id 1) (at 149.86 63.9064 0))
     (property "Footprint" "" (id 2) (at 149.86 69.85 0)
@@
   (symbol (lib_id "74xx:74LS02") (at 124.46 85.09 0) (unit 1)
     (in_bom yes) (on_board yes)
-    (property "Reference" "U54" (id 0) (at 124.46 76.835 0))
+    (property "Reference" "U57" (id 0) (at 124.46 76.835 0))
     (property "Value" "74LS02" (id 1) (at 124.46 79.1464 0))
     (property "Footprint" "" (id 2) (at 124.46 85.09 0)
@@
   (symbol (lib_id "74xx:74LS08") (at 154.94 100.33 0) (unit 1)
     (in_bom yes) (on_board yes)
-    (property "Reference" "U63" (id 0) (at 154.94 92.075 0))
+    (property "Reference" "U66" (id 0) (at 154.94 92.075 0))
     (property "Value" "74LS08" (id 1) (at 154.94 94.3864 0))
     (property "Footprint" "" (id 2) (at 154.94 100.33 0)
@@
   (symbol (lib_id "74xx:74LS08") (at 139.7 87.63 0) (unit 1)
     (in_bom yes) (on_board yes)
-    (property "Reference" "U60" (id 0) (at 139.7 79.375 0))
+    (property "Reference" "U63" (id 0) (at 139.7 79.375 0))
     (property "Value" "74LS08" (id 1) (at 139.7 81.6864 0))
     (property "Footprint" "" (id 2) (at 139.7 87.63 0)
@@
   (symbol (lib_id "74xx:74LS08") (at 139.7 113.03 0) (unit 1)
     (in_bom yes) (on_board yes)
-    (property "Reference" "U61" (id 0) (at 139.7 104.775 0))
+    (property "Reference" "U64" (id 0) (at 139.7 104.775 0))
     (property "Value" "74LS08" (id 1) (at 139.7 107.0864 0))
     (property "Footprint" "" (id 2) (at 139.7 113.03 0)
@@
   (symbol (lib_id "74xx:74LS02") (at 124.46 95.25 0) (unit 1)
     (in_bom yes) (on_board yes)
-    (property "Reference" "U55" (id 0) (at 124.46 86.995 0))
+    (property "Reference" "U58" (id 0) (at 124.46 86.995 0))
     (property "Value" "74LS02" (id 1) (at 124.46 89.3064 0))
     (property "Footprint" "" (id 2) (at 124.46 95.25 0)
@@
   (symbol (lib_id "74xx:74LS02") (at 124.46 105.41 0) (unit 1)
     (in_bom yes) (on_board yes)
-    (property "Reference" "U56" (id 0) (at 124.46 97.155 0))
+    (property "Reference" "U59" (id 0) (at 124.46 97.155 0))
     (property "Value" "74LS02" (id 1) (at 124.46 99.4664 0))
     (property "Footprint" "" (id 2) (at 124.46 105.41 0)
@@
   (symbol (lib_id "74xx:74LS02") (at 124.46 115.57 0) (unit 1)
     (in_bom yes) (on_board yes)
-    (property "Reference" "U57" (id 0) (at 124.46 107.315 0))
+    (property "Reference" "U60" (id 0) (at 124.46 107.315 0))
     (property "Value" "74LS02" (id 1) (at 124.46 109.6264 0))
     (property "Footprint" "" (id 2) (at 124.46 115.57 0)
