File: Kicad Files/Flags register.kicad_sch (KiCad schematic)
At the start: 20 parts, among them U56 74LS00, U57 74LS02, U58 74LS02, U59 74LS02, U60 74LS02, U61 74LS00, U62 74LS00, U63 74LS08, U64 74LS08, U65 74LS00, U66 74LS08, U67 74LS173

Commit message: put it allll together
Changed lines of the file:
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@@
   (junction (at 233.68 63.5) (diameter 0) (color 0 0 0 0)
   )
+  (junction (at 190.5 71.12) (diameter 0) (color 0 0 0 0)
+  )
   (junction (at 227.33 60.96) (diameter 0) (color 0 0 0 0)
   )
   (junction (at 227.33 29.21) (diameter 0) (color 0 0 0 0)
   )
-  (junction (at 190.5 73.66) (diameter 0) (color 0 0 0 0)
-  )
   (junction (at 109.22 72.39) (diameter 0) (color 0 0 0 0)
   )
@@
   (junction (at 127 69.85) (diameter 0) (color 0 0 0 0)
   )
-  (wire (pts (xy 185.42 73.66) (xy 190.5 73.66))
-    (stroke (width 0) (type default) (color 0 0 0 0))
-  )
   (wire (pts (xy 190.5 81.28) (xy 185.42 81.28))
     (stroke (width 0) (type default) (color 0 0 0 0))
@@
   )
   (wire (pts (xy 92.71 106.68) (xy 111.76 106.68))
-    (stroke (width 0) (type default) (color 0 0 0 0))
-  )
-  (wire (pts (xy 203.2 50.8) (xy 210.82 50.8))
     (stroke (width 0) (type default) (color 0 0 0 0))
   )
@@
   (symbol (lib_id "74xx:74LS173") (at 203.2 73.66 0) (unit 1)
     (in_bom yes) (on_board yes)
-    (property "Reference" "U67" (id 0) (at 203.2 46.2026 0))
-    (property "Value" "74LS173" (id 1) (at 203.2 48.514 0))
+    (property "Reference" "U67" (id 0) (at 205.74 52.705 0))
+    (property "Value" "74LS173" (id 1) (at 208.28 54.61 0))
     (property "Footprint" "" (id 2) (at 203.2 73.66 0)
       (effects (font (size 1.27 1.27)) hide)
@@
     (pin "1")
   )
-  (symbol (lib_id "power:VCC") (at 210.82 50.8 0) (unit 1)
-    (in_bom yes) (on_board yes)
-    (property "Reference" "#PWR0161" (id 0) (at 210.82 54.61 0)
-      (effects (font (size 1.27 1.27)) hide)
-    )
-    (property "Value" "VCC" (id 1) (at 211.201 46.4058 0))
-    (property "Footprint" "" (id 2) (at 210.82 50.8 0)
-      (effects (font (size 1.27 1.27)) hide)
-    )
-    (property "Datasheet" "" (id 3) (at 210.82 50.8 0)
-      (effects (font (size 1.27 1.27)) hide)
-    )
-    (pin "1")
-  )
-  (symbol (lib_id "power:GND") (at 185.42 73.66 0) (unit 1)
-    (in_bom yes) (on_board yes)
-    (property "Reference" "#PWR0159" (id 0) (at 185.42 80.01 0)
-      (effects (font (size 1.27 1.27)) hide)
-    )
-    (property "Value" "GND" (id 1) (at 185.547 78.0542 0))
-    (property "Footprint" "" (id 2) (at 185.42 73.66 0)
-      (effects (font (size 1.27 1.27)) hide)
-    )
-    (property "Datasheet" "" (id 3) (at 185.42 73.66 0)
-      (effects (font (size 1.27 1.27)) hide)
-    )
+  (symbol (lib_id "power:VCC") (at 203.2 50.8 0) (unit 1)
+    (in_bom yes) (on_board yes)
+    (property "Reference" "#PWR0161" (id 0) (at 203.2 54.61 0)
+      (effects (font (size 1.27 1.27)) hide)
+    )
+    (property "Value" "VCC" (id 1) (at 203.581 46.4058 0))
+    (property "Footprint" "" (id 2) (at 203.2 50.8 0)
+      (effects (font (size 1.27 1.27)) hide)
+    )
+    (property "Datasheet" "" (id 3) (at 203.2 50.8 0)
+      (effects (font (size 1.27 1.27)) hide)
+    )
+    (pin "1")
+  )
+  (symbol (lib_id "power:GND") (at 190.5 71.12 270) (unit 1)
+    (in_bom yes) (on_board yes)
+    (property "Reference" "#PWR0159" (id 0) (at 184.15 71.12 0)
+      (effects (font (size 1.27 1.27)) hide)
+    )
+    (property "Value" "GND" (id 1) (at 186.1058 71.247 0))
+    (property "Footprint" "" (id 2) (at 190.5 71.12 0)
+      (effects (font (size 1.27 1.27)) hide)
+    )
+    (property "Datasheet" "" (id 3) (at 190.5 71.12 0)
+      (effects (font (size 1.27 1.27)) hide)
+    )

Commit message: fixed erc
Parts:
- renumbered D104 to D149, D105 to D150, D106 to D151, D107 to D152, R139 to R158, R140 to R159, R141 to R160, R142 to R161, U56 to U52, U57 to U53, U58 to U54, U59 to U55, U60 to U56, U61 to U57, U62 to U58, U63 to U59, U64 to U60, U65 to U61, U66 to U62, U67 to U63
Changed lines of the file:
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@@
   (symbol (lib_id "74xx:74LS173") (at 203.2 73.66 0) (unit 1)
     (in_bom yes) (on_board yes)
-    (property "Reference" "U67" (id 0) (at 205.74 52.705 0))
+    (property "Reference" "U63" (id 0) (at 205.74 52.705 0))
     (property "Value" "74LS173" (id 1) (at 208.28 54.61 0))
     (property "Footprint" "" (id 2) (at 203.2 73.66 0)
@@
   (symbol (lib_id "Device:LED") (at 240.03 44.45 270) (unit 1)
     (in_bom yes) (on_board yes)
-    (property "Reference" "D107" (id 0) (at 242.062 43.1038 0)
+    (property "Reference" "D152" (id 0) (at 242.062 43.1038 0)
       (effects (font (size 1.27 1.27)) (justify top) hide)
     )
@@
   (symbol (lib_id "Device:LED") (at 233.68 44.45 270) (unit 1)
     (in_bom yes) (on_board yes)
-    (property "Reference" "D106" (id 0) (at 235.712 43.1038 0)
+    (property "Reference" "D151" (id 0) (at 235.712 43.1038 0)
       (effects (font (size 1.27 1.27)) (justify top) hide)
     )
@@
   (symbol (lib_id "Device:LED") (at 227.33 44.45 270) (unit 1)
     (in_bom yes) (on_board yes)
-    (property "Reference" "D105" (id 0) (at 229.362 43.1038 0)
+    (property "Reference" "D150" (id 0) (at 229.362 43.1038 0)
       (effects (font (size 1.27 1.27)) (justify top) hide)
     )
@@
   (symbol (lib_id "Device:LED") (at 220.98 44.45 270) (unit 1)
     (in_bom yes) (on_board yes)
-    (property "Reference" "D104" (id 0) (at 223.012 43.1038 0)
+    (property "Reference" "D149" (id 0) (at 223.012 43.1038 0)
       (effects (font (size 1.27 1.27)) (justify top) hide)
     )
@@
   (symbol (lib_id "Device:R") (at 220.98 36.83 0) (unit 1)
     (in_bom yes) (on_board yes)
-    (property "Reference" "R139" (id 0) (at 217.8304 37.1856 90)
+    (property "Reference" "R158" (id 0) (at 217.8304 37.1856 90)
       (effects (font (size 1.27 1.27)) (justify top))
     )
@@
   (symbol (lib_id "Device:R") (at 240.03 36.83 0) (unit 1)
     (in_bom yes) (on_board yes)
-    (property "Reference" "R142" (id 0) (at 236.8804 37.1856 90)
+    (property "Reference" "R161" (id 0) (at 236.8804 37.1856 90)
       (effects (font (size 1.27 1.27)) (justify top))
     )
@@
   (symbol (lib_id "Device:R") (at 233.68 36.83 0) (unit 1)
     (in_bom yes) (on_board yes)
-    (property "Reference" "R141" (id 0) (at 230.5304 37.1856 90)
+    (property "Reference" "R160" (id 0) (at 230.5304 37.1856 90)
       (effects (font (size 1.27 1.27)) (justify top))
     )
@@
   (symbol (lib_id "Device:R") (at 227.33 36.83 0) (unit 1)
     (in_bom yes) (on_board yes)
-    (property "Reference" "R140" (id 0) (at 224.1804 37.1856 90)
+    (property "Reference" "R159" (id 0) (at 224.1804 37.1856 90)
       (effects (font (size 1.27 1.27)) (justify top))
     )
@@
   (symbol (lib_id "power:GND") (at 247.65 29.21 0) (unit 1)
     (in_bom yes) (on_board yes)
-    (property "Reference" "#PWR0162" (id 0) (at 247.65 35.56 0)
+    (property "Reference" "#PWR0126" (id 0) (at 247.65 35.56 0)
       (effects (font (size 1.27 1.27)) hide)
     )
@@
   (symbol (lib_id "power:GND") (at 203.2 96.52 0) (unit 1)
     (in_bom yes) (on_board yes)
-    (property "Reference" "#PWR0160" (id 0) (at 203.2 102.87 0)
+    (property "Reference" "#PWR0125" (id 0) (at 203.2 102.87 0)
       (effects (font (size 1.27 1.27)) hide)
     )
@@
   (symbol (lib_id "power:VCC") (at 203.2 50.8 0) (unit 1)
     (in_bom yes) (on_board yes)
-    (property "Reference" "#PWR0161" (id 0) (at 203.2 54.61 0)
+    (property "Reference" "#PWR0124" (id 0) (at 203.2 54.61 0)
       (effects (font (size 1.27 1.27)) hide)
     )
@@
   (symbol (lib_id "power:GND") (at 190.5 71.12 270) (unit 1)
     (in_bom yes) (on_board yes)
-    (property "Reference" "#PWR0159" (id 0) (at 184.15 71.12 0)
+    (property "Reference" "#PWR0123" (id 0) (at 184.15 71.12 0)
       (effects (font (size 1.27 1.27)) hide)
     )
@@
   (symbol (lib_id "74xx:74LS00") (at 119.38 69.85 0) (unit 1)
     (in_bom yes) (on_board yes)
-    (property "Reference" "U56" (id 0) (at 119.38 61.595 0))
+    (property "Reference" "U52" (id 0) (at 119.38 61.595 0))
     (property "Value" "74LS00" (id 1) (at 119.38 63.9064 0))
     (property "Footprint" "" (id 2) (at 119.38 69.85 0)
@@
   (symbol (lib_id "74xx:74LS00") (at 134.62 76.2 0) (unit 1)
     (in_bom yes) (on_board yes)
-    (property "Reference" "U62" (id 0) (at 134.62 67.945 0))
+    (property "Reference" "U58" (id 0) (at 134.62 67.945 0))
     (property "Value" "74LS00" (id 1) (at 134.62 70.2564 0))
     (property "Footprint" "" (id 2) (at 134.62 76.2 0)
@@
   (symbol (lib_id "74xx:74LS00") (at 134.62 63.5 0) (unit 1)
     (in_bom yes) (on_board yes)
-    (property "Reference" "U61" (id 0) (at 134.62 55.245 0))
+    (property "Reference" "U57" (id 0) (at 134.62 55.245 0))
     (property "Value" "74LS00" (id 1) (at 134.62 57.5564 0))
     (property "Footprint" "" (id 2) (at 134.62 63.5 0)
@@
   (symbol (lib_id "74xx:74LS00") (at 149.86 69.85 0) (unit 1)
     (in_bom yes) (on_board yes)
-    (property "Reference" "U65" (id 0) (at 149.86 61.595 0))
+    (property "Reference" "U61" (id 0) (at 149.86 61.595 0))
     (property "Value" "74LS00" (id 1) (at 149.86 63.9064 0))
     (property "Footprint" "" (id 2) (at 149.86 69.85 0)
@@
   (symbol (lib_id "74xx:74LS02") (at 124.46 85.09 0) (unit 1)
     (in_bom yes) (on_board yes)
-    (property "Reference" "U57" (id 0) (at 124.46 76.835 0))
+    (property "Reference" "U53" (id 0) (at 124.46 76.835 0))
     (property "Value" "74LS02" (id 1) (at 124.46 79.1464 0))
     (property "Footprint" "" (id 2) (at 124.46 85.09 0)
@@
   (symbol (lib_id "74xx:74LS08") (at 154.94 100.33 0) (unit 1)
     (in_bom yes) (on_board yes)
-    (property "Reference" "U66" (id 0) (at 154.94 92.075 0))
+    (property "Reference" "U62" (id 0) (at 154.94 92.075 0))
     (property "Value" "74LS08" (id 1) (at 154.94 94.3864 0))
     (property "Footprint" "" (id 2) (at 154.94 100.33 0)
@@
   (symbol (lib_id "74xx:74LS08") (at 139.7 87.63 0) (unit 1)
     (in_bom yes) (on_board yes)
-    (property "Reference" "U63" (id 0) (at 139.7 79.375 0))
+    (property "Reference" "U59" (id 0) (at 139.7 79.375 0))
     (property "Value" "74LS08" (id 1) (at 139.7 81.6864 0))
     (property "Footprint" "" (id 2) (at 139.7 87.63 0)
@@
   (symbol (lib_id "74xx:74LS08") (at 139.7 113.03 0) (unit 1)
     (in_bom yes) (on_board yes)
-    (property "Reference" "U64" (id 0) (at 139.7 104.775 0))
+    (property "Reference" "U60" (id 0) (at 139.7 104.775 0))
     (property "Value" "74LS08" (id 1) (at 139.7 107.0864 0))
     (property "Footprint" "" (id 2) (at 139.7 113.03 0)
@@
   (symbol (lib_id "74xx:74LS02") (at 124.46 95.25 0) (unit 1)
     (in_bom yes) (on_board yes)
-    (property "Reference" "U58" (id 0) (at 124.46 86.995 0))
+    (property "Reference" "U54" (id 0) (at 124.46 86.995 0))
     (property "Value" "74LS02" (id 1) (at 124.46 89.3064 0))
     (property "Footprint" "" (id 2) (at 124.46 95.25 0)
@@
   (symbol (lib_id "74xx:74LS02") (at 124.46 105.41 0) (unit 1)
     (in_bom yes) (on_board yes)
-    (property "Reference" "U59" (id 0) (at 124.46 97.155 0))
+    (property "Reference" "U55" (id 0) (at 124.46 97.155 0))
     (property "Value" "74LS02" (id 1) (at 124.46 99.4664 0))
     (property "Footprint" "" (id 2) (at 124.46 105.41 0)
@@
   (symbol (lib_id "74xx:74LS02") (at 124.46 115.57 0) (unit 1)
     (in_bom yes) (on_board yes)
-    (property "Reference" "U60" (id 0) (at 124.46 107.315 0))
+    (property "Reference" "U56" (id 0) (at 124.46 107.315 0))
     (property "Value" "74LS02" (id 1) (at 124.46 109.6264 0))
     (property "Footprint" "" (id 2) (at 124.46 115.57 0)
