File: Kicad Files/IO.kicad_sch (KiCad schematic)
At the start: 0 parts

Commit message: finished todo list
Parts:
- added U?: RP2040, Package_DFN_QFN:QFN-56-1EP_7x7mm_P0.4mm_EP3.2x3.2mm, symbol MCU_RaspberryPi:RP2040
Connections:
- net ABUS_00: now also U?.37 (GPIO25)
- net ABUS_01: now also U?.36 (GPIO24)
- net ABUS_02: now also U?.35 (GPIO23)
- net ABUS_03: now also U?.34 (GPIO22)
- net ABUS_04: now also U?.32 (GPIO21)
- net ABUS_05: now also U?.31 (GPIO20)
- net ABUS_06: now also U?.30 (GPIO19)
- net ABUS_07: now also U?.29 (GPIO18)
- net ABUS_08: now also U?.28 (GPIO17)
- net ABUS_09: now also U?.27 (GPIO16)
- net ABUS_10: now also U?.18 (GPIO15)
- net ABUS_11: now also U?.17 (GPIO14)
- net ABUS_12: now also U?.16 (GPIO13)
- net ABUS_13: now also U?.15 (GPIO12)
- net ABUS_14: now also U?.14 (GPIO11)
- net ABUS_15: now also U?.13 (GPIO10)
- net BUS_0: now also U?.4 (GPIO2)
- net BUS_1: now also U?.5 (GPIO3)
- net BUS_2: now also U?.6 (GPIO4)
- net BUS_3: now also U?.7 (GPIO5)
- net BUS_4: now also U?.8 (GPIO6)
- net BUS_5: now also U?.9 (GPIO7)
- net BUS_6: now also U?.11 (GPIO8)
- net BUS_7: now also U?.12 (GPIO9)
- new net: U?.1 (IOVDD), U?.10 (IOVDD), U?.22 (IOVDD), U?.33 (IOVDD), U?.42 (IOVDD), U?.49 (IOVDD)
- new net: U?.23 (DVDD), U?.50 (DVDD)
- new net CLR: U?.41 (GPIO29_ADC3)
- new net GND: U?.57 (GND)
- new net OVRD: U?.40 (GPIO28_ADC2)
- new net VCC: U?.44 (VREG_IN)
- new net ~{RI}: U?.3 (GPIO1)
- new net ~{RO}: U?.2 (GPIO0)
- no-connect marks 0 -> 20

Commit message: fixed erc
Parts:
- gave numbers to parts that had none: 1
Connections:
- no-connect marks 20 -> 21
Changed lines of the file:
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@@
 (kicad_sch (version 20211123) (generator eeschema)
   (paper "A4")
+  (no_connect (at 103.505 97.155))
   (no_connect (at 149.225 97.155))
   (no_connect (at 126.365 97.155))
@@
   (symbol (lib_id "MCU_RaspberryPi:RP2040") (at 131.445 71.755 90) (unit 1)
     (in_bom yes) (on_board yes) (fields_autoplaced)
-    (property "Reference" "U?" (id 0) (at 179.07 68.1736 90))
+    (property "Reference" "U67" (id 0) (at 179.07 68.1736 90))
     (property "Value" "RP2040" (id 1) (at 179.07 70.7136 90))
     (property "Footprint" "Package_DFN_QFN:QFN-56-1EP_7x7mm_P0.4mm_EP3.2x3.2mm" (id 2) (at 131.445 71.755 0)
@@
   (symbol (lib_id "power:VCC") (at 85.725 61.595 0) (unit 1)
     (in_bom yes) (on_board yes) (fields_autoplaced)
-    (property "Reference" "#PWR?" (id 0) (at 85.725 65.405 0)
+    (property "Reference" "#PWR0132" (id 0) (at 85.725 65.405 0)
       (effects (font (size 1.27 1.27)) hide)
     )
@@
   (symbol (lib_id "power:GND") (at 177.165 71.755 0) (unit 1)
     (in_bom yes) (on_board yes) (fields_autoplaced)
-    (property "Reference" "#PWR?" (id 0) (at 177.165 78.105 0)
+    (property "Reference" "#PWR0133" (id 0) (at 177.165 78.105 0)
       (effects (font (size 1.27 1.27)) hide)
     )
