File: Kicad Files/a-register.kicad_sch (KiCad schematic)
At the start: 20 parts, among them U37 74LS245, U38 74LS173, U39 74LS173

Commit message: finished todo list
Changed lines of the file:
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@@
-    (stroke (width 0) (type default) (color 0 0 0 0))
-  )
-  (wire (pts (xy 195.58 43.18) (xy 195.58 38.1))
     (stroke (width 0) (type default) (color 0 0 0 0))
   )
@@
     (stroke (width 0) (type default) (color 0 0 0 0))
   )
+  (wire (pts (xy 199.39 48.26) (xy 208.28 48.26))
+    (stroke (width 0) (type default) (color 0 0 0 0))
+  )
   (wire (pts (xy 231.14 71.12) (xy 231.14 73.66))
     (stroke (width 0) (type default) (color 0 0 0 0))
@@
     (stroke (width 0) (type default) (color 0 0 0 0))
   )
-  (wire (pts (xy 195.58 38.1) (xy 208.28 38.1))
+  (wire (pts (xy 160.02 43.18) (xy 208.28 43.18))
     (stroke (width 0) (type default) (color 0 0 0 0))
   )
@@
     (stroke (width 0) (type default) (color 0 0 0 0))
   )
-  (wire (pts (xy 104.14 93.98) (xy 208.28 93.98))
+  (wire (pts (xy 199.39 93.98) (xy 199.39 48.26))
+    (stroke (width 0) (type default) (color 0 0 0 0))
+  )
+  (wire (pts (xy 104.14 93.98) (xy 199.39 93.98))
     (stroke (width 0) (type default) (color 0 0 0 0))
   )
@@
     (stroke (width 0) (type default) (color 0 0 0 0))
   )
-  (wire (pts (xy 160.02 43.18) (xy 195.58 43.18))
-    (stroke (width 0) (type default) (color 0 0 0 0))
-  )
   (wire (pts (xy 137.16 146.05) (xy 137.16 149.86))
     (stroke (width 0) (type default) (color 0 0 0 0))
@@
     (effects (font (size 1.524 1.524)) (justify right))
   )
-  (hierarchical_label "CLR" (shape input) (at 208.28 38.1 0)
+  (hierarchical_label "CLR" (shape input) (at 208.28 43.18 0)
     (effects (font (size 1.524 1.524)) (justify left))
   )
@@
     (effects (font (size 1.524 1.524)) (justify right))
   )
-  (hierarchical_label "~{AO}" (shape input) (at 208.28 93.98 0)
-    (effects (font (size 1.524 1.524)) (justify left))
-  )
+  (hierarchical_label "~{AO}" (shape input) (at 208.28 48.26 0)
+    (effects (font (size 1.524 1.524)) (justify left))
+  )

Commit message: fixed erc
Parts:
- renumbered C19 to C18, D42 to D79, D43 to D80, D44 to D81, D45 to D82, D46 to D83, D47 to D84, D48 to D85, D49 to D86, R77 to R88, R78 to R89, R79 to R90, R80 to R91, R81 to R92, R82 to R93, R83 to R94, R84 to R95, U37 to U32, U38 to U33, U39 to U34
Changed lines of the file:
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@@
   (symbol (lib_id "8bit-computer-rescue:74LS173-8bit-computer-rescue") (at 133.35 68.58 270) (unit 1)
     (in_bom yes) (on_board yes)
-    (property "Reference" "U38" (id 0) (at 135.89 71.12 0))
+    (property "Reference" "U33" (id 0) (at 135.89 71.12 0))
     (property "Value" "74LS173" (id 1) (at 132.08 71.12 0))
     (property "Footprint" "Package_DIP:DIP-16_W7.62mm" (id 2) (at 133.35 68.58 0)
@@
   (symbol (lib_id "8bit-computer-rescue:LED_ALT-Device") (at 114.3 142.24 90) (unit 1)
     (in_bom yes) (on_board yes)
-    (property "Reference" "D44" (id 0) (at 111.76 142.24 0))
+    (property "Reference" "D81" (id 0) (at 111.76 142.24 0))
     (property "Value" "RED" (id 1) (at 116.84 142.24 0))
     (property "Footprint" "LED_THT:LED_D5.0mm" (id 2) (at 114.3 142.24 0)
@@
   (symbol (lib_id "8bit-computer-rescue:LED_ALT-Device") (at 144.78 142.24 90) (unit 1)
     (in_bom yes) (on_board yes)
-    (property "Reference" "D48" (id 0) (at 142.24 142.24 0))
+    (property "Reference" "D85" (id 0) (at 142.24 142.24 0))
     (property "Value" "RED" (id 1) (at 147.32 142.24 0))
     (property "Footprint" "LED_THT:LED_D5.0mm" (id 2) (at 144.78 142.24 0)
@@
   (symbol (lib_id "8bit-computer-rescue:LED_ALT-Device") (at 152.4 142.24 90) (unit 1)
     (in_bom yes) (on_board yes)
-    (property "Reference" "D49" (id 0) (at 149.86 142.24 0))
+    (property "Reference" "D86" (id 0) (at 149.86 142.24 0))
     (property "Value" "RED" (id 1) (at 154.94 142.24 0))
     (property "Footprint" "LED_THT:LED_D5.0mm" (id 2) (at 152.4 142.24 0)
@@
   (symbol (lib_id "Device:R") (at 114.3 153.67 0) (unit 1)
     (in_bom yes) (on_board yes)
-    (property "Reference" "R79" (id 0) (at 116.332 153.67 90))
+    (property "Reference" "R90" (id 0) (at 116.332 153.67 90))
     (property "Value" "R" (id 1) (at 114.3 153.67 90))
     (property "Footprint" "Resistor_THT:R_Axial_DIN0207_L6.3mm_D2.5mm_P7.62mm_Horizontal" (id 2) (at 112.522 153.67 90)
@@
   (symbol (lib_id "Device:R") (at 121.92 153.67 0) (unit 1)
     (in_bom yes) (on_board yes)
-    (property "Reference" "R80" (id 0) (at 123.952 153.67 90))
+    (property "Reference" "R91" (id 0) (at 123.952 153.67 90))
     (property "Value" "R" (id 1) (at 121.92 153.67 90))
     (property "Footprint" "Resistor_THT:R_Axial_DIN0207_L6.3mm_D2.5mm_P7.62mm_Horizontal" (id 2) (at 120.142 153.67 90)
@@
   (symbol (lib_id "Device:R") (at 137.16 153.67 0) (unit 1)
     (in_bom yes) (on_board yes)
-    (property "Reference" "R82" (id 0) (at 139.192 153.67 90))
+    (property "Reference" "R93" (id 0) (at 139.192 153.67 90))
     (property "Value" "R" (id 1) (at 137.16 153.67 90))
     (property "Footprint" "Resistor_THT:R_Axial_DIN0207_L6.3mm_D2.5mm_P7.62mm_Horizontal" (id 2) (at 135.382 153.67 90)
@@
   (symbol (lib_id "Device:R") (at 152.4 153.67 0) (unit 1)
     (in_bom yes) (on_board yes)
-    (property "Reference" "R84" (id 0) (at 154.432 153.67 90))
+    (property "Reference" "R95" (id 0) (at 154.432 153.67 90))
     (property "Value" "R" (id 1) (at 152.4 153.67 90))
     (property "Footprint" "Resistor_THT:R_Axial_DIN0207_L6.3mm_D2.5mm_P7.62mm_Horizontal" (id 2) (at 150.622 153.67 90)
@@
   (symbol (lib_id "power:VCC") (at 101.6 86.36 180) (unit 1)
     (in_bom yes) (on_board yes)
-    (property "Reference" "#PWR0116" (id 0) (at 101.6 82.55 0)
+    (property "Reference" "#PWR075" (id 0) (at 101.6 82.55 0)
       (effects (font (size 1.27 1.27)) hide)
     )
@@
   (symbol (lib_id "8bit-computer-rescue:74LS173-8bit-computer-rescue") (at 173.99 68.58 270) (unit 1)
     (in_bom yes) (on_board yes)
-    (property "Reference" "U39" (id 0) (at 176.53 71.12 0))
+    (property "Reference" "U34" (id 0) (at 176.53 71.12 0))
     (property "Value" "74LS173" (id 1) (at 172.72 71.12 0))
     (property "Footprint" "Package_DIP:DIP-16_W7.62mm" (id 2) (at 173.99 68.58 0)
@@
   (symbol (lib_id "8bit-computer-rescue:74LS245-8bit-computer-rescue") (at 91.44 68.58 90) (unit 1)
     (in_bom yes) (on_board yes)
-    (property "Reference" "U37" (id 0) (at 76.835 66.04 0)
+    (property "Reference" "U32" (id 0) (at 76.835 66.04 0)
       (effects (font (size 1.27 1.27)) (justify left bottom))
     )
@@
   (symbol (lib_id "8bit-computer-rescue:LED_ALT-Device") (at 99.06 142.24 90) (unit 1)
     (in_bom yes) (on_board yes)
-    (property "Reference" "D42" (id 0) (at 96.52 142.24 0))
+    (property "Reference" "D79" (id 0) (at 96.52 142.24 0))
     (property "Value" "RED" (id 1) (at 101.6 142.24 0))
     (property "Footprint" "LED_THT:LED_D5.0mm" (id 2) (at 99.06 142.24 0)
@@
   (symbol (lib_id "8bit-computer-rescue:LED_ALT-Device") (at 106.68 142.24 90) (unit 1)
     (in_bom yes) (on_board yes)
-    (property "Reference" "D43" (id 0) (at 104.14 142.24 0))
+    (property "Reference" "D80" (id 0) (at 104.14 142.24 0))
     (property "Value" "RED" (id 1) (at 109.22 142.24 0))
     (property "Footprint" "LED_THT:LED_D5.0mm" (id 2) (at 106.68 142.24 0)
@@
   (symbol (lib_id "8bit-computer-rescue:LED_ALT-Device") (at 121.92 142.24 90) (unit 1)
     (in_bom yes) (on_board yes)
-    (property "Reference" "D45" (id 0) (at 119.38 142.24 0))
+    (property "Reference" "D82" (id 0) (at 119.38 142.24 0))
     (property "Value" "RED" (id 1) (at 124.46 142.24 0))
     (property "Footprint" "LED_THT:LED_D5.0mm" (id 2) (at 121.92 142.24 0)
@@
   (symbol (lib_id "8bit-computer-rescue:LED_ALT-Device") (at 129.54 142.24 90) (unit 1)
     (in_bom yes) (on_board yes)
-    (property "Reference" "D46" (id 0) (at 127 142.24 0))
+    (property "Reference" "D83" (id 0) (at 127 142.24 0))
     (property "Value" "RED" (id 1) (at 132.08 142.24 0))
     (property "Footprint" "LED_THT:LED_D5.0mm" (id 2) (at 129.54 142.24 0)
@@
   (symbol (lib_id "8bit-computer-rescue:LED_ALT-Device") (at 137.16 142.24 90) (unit 1)
     (in_bom yes) (on_board yes)
-    (property "Reference" "D47" (id 0) (at 134.62 142.24 0))
+    (property "Reference" "D84" (id 0) (at 134.62 142.24 0))
     (property "Value" "RED" (id 1) (at 139.7 142.24 0))
     (property "Footprint" "LED_THT:LED_D5.0mm" (id 2) (at 137.16 142.24 0)
@@
   (symbol (lib_id "Device:R") (at 99.06 153.67 0) (unit 1)
     (in_bom yes) (on_board yes)
-    (property "Reference" "R77" (id 0) (at 101.092 153.67 90))
+    (property "Reference" "R88" (id 0) (at 101.092 153.67 90))
     (property "Value" "R" (id 1) (at 99.06 153.67 90))
     (property "Footprint" "Resistor_THT:R_Axial_DIN0207_L6.3mm_D2.5mm_P7.62mm_Horizontal" (id 2) (at 97.282 153.67 90)
@@
   (symbol (lib_id "Device:R") (at 106.68 153.67 0) (unit 1)
     (in_bom yes) (on_board yes)
-    (property "Reference" "R78" (id 0) (at 108.712 153.67 90))
+    (property "Reference" "R89" (id 0) (at 108.712 153.67 90))
     (property "Value" "R" (id 1) (at 106.68 153.67 90))
     (property "Footprint" "Resistor_THT:R_Axial_DIN0207_L6.3mm_D2.5mm_P7.62mm_Horizontal" (id 2) (at 104.902 153.67 90)
@@
   (symbol (lib_id "Device:R") (at 129.54 153.67 0) (unit 1)
     (in_bom yes) (on_board yes)
-    (property "Reference" "R81" (id 0) (at 131.572 153.67 90))
+    (property "Reference" "R92" (id 0) (at 131.572 153.67 90))
     (property "Value" "R" (id 1) (at 129.54 153.67 90))
     (property "Footprint" "Resistor_THT:R_Axial_DIN0207_L6.3mm_D2.5mm_P7.62mm_Horizontal" (id 2) (at 127.762 153.67 90)
@@
   (symbol (lib_id "Device:R") (at 144.78 153.67 0) (unit 1)
     (in_bom yes) (on_board yes)
-    (property "Reference" "R83" (id 0) (at 146.812 153.67 90))
+    (property "Reference" "R94" (id 0) (at 146.812 153.67 90))
     (property "Value" "R" (id 1) (at 144.78 153.67 90))
     (property "Footprint" "Resistor_THT:R_Axial_DIN0207_L6.3mm_D2.5mm_P7.62mm_Horizontal" (id 2) (at 143.002 153.67 90)
@@
   (symbol (lib_id "power:GND") (at 125.73 166.37 0) (unit 1)
     (in_bom yes) (on_board yes)
-    (property "Reference" "#PWR0117" (id 0) (at 125.73 172.72 0)
+    (property "Reference" "#PWR076" (id 0) (at 125.73 172.72 0)
       (effects (font (size 1.27 1.27)) hide)
     )
@@
   (symbol (lib_id "power:GND") (at 195.58 55.88 0) (unit 1)
     (in_bom yes) (on_board yes)
-    (property "Reference" "#PWR0118" (id 0) (at 195.58 62.23 0)
+    (property "Reference" "#PWR077" (id 0) (at 195.58 62.23 0)
       (effects (font (size 1.27 1.27)) hide)
     )
@@
   (symbol (lib_id "Device:C") (at 231.14 67.31 0) (unit 1)
     (in_bom yes) (on_board yes)
-    (property "Reference" "C19" (id 0) (at 231.775 64.77 0)
+    (property "Reference" "C18" (id 0) (at 231.775 64.77 0)
       (effects (font (size 1.27 1.27)) (justify left))
     )
@@
   (symbol (lib_id "power:GND") (at 231.14 73.66 0) (unit 1)
     (in_bom yes) (on_board yes)
-    (property "Reference" "#PWR0120" (id 0) (at 231.14 80.01 0)
+    (property "Reference" "#PWR079" (id 0) (at 231.14 80.01 0)
       (effects (font (size 1.27 1.27)) hide)
     )
@@
   (symbol (lib_id "power:VCC") (at 231.14 60.96 0) (unit 1)
     (in_bom yes) (on_board yes)
-    (property "Reference" "#PWR0119" (id 0) (at 231.14 64.77 0)
-      (effects (font (size 1.27 1.27)) hide)
-    )
+    (property "Reference" "#PWR078" (id 0) (at 231.14 64.77 0)
+      (effects (font (size 1.27 1.27)) hide)
+    )
