File: Kicad Files/alu.kicad_sch (KiCad schematic)
At the start: 33 parts

Commit message: started tidy up in control
Parts:
- gave numbers to parts that had none: 27

Commit message: work on cl
Parts:
- C22: renamed from C2; value 0.1µF -> C
- C23: renamed from C3; value 0.1µF -> C
- R129: renamed from R49; value 220 -> R
- R130: renamed from R50; value 220 -> R
- R131: renamed from R51; value 220 -> R
- R132: renamed from R52; value 220 -> R
- R133: renamed from R53; value 220 -> R
- R134: renamed from R54; value 220 -> R
- R135: renamed from R55; value 220 -> R
- R136: renamed from R56; value 220 -> R
- R137: renamed from R57; value 220 -> R
- R138: renamed from R58; value 220 -> R
- renumbered D47 to D100, D48 to D101, D49 to D102, D50 to D103, D41 to D94, D42 to D95, D43 to D96, D44 to D97, D45 to D98, D46 to D99, U18 to U48, U20 to U49, U21 to U50, U17 to U51, U19 to U52

Commit message: fixed ecc problems
Parts:
- renumbered U48 to U51, U49 to U52, U50 to U53, U51 to U54, U52 to U55
Connections:
- no-connect marks 1 -> 0
Changed lines of the file:
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@@
   (junction (at 107.95 96.52) (diameter 0) (color 0 0 0 0)
   )
-  (no_connect (at 13.97 187.96))
   (wire (pts (xy 259.08 34.29) (xy 259.08 88.9))
     (stroke (width 0) (type default) (color 0 0 0 0))
@@
     (stroke (width 0) (type default) (color 0 0 0 0))
   )
-  (wire (pts (xy 13.97 161.29) (xy 13.97 142.24))
-    (stroke (width 0) (type default) (color 0 0 0 0))
-  )
   (wire (pts (xy 97.79 22.86) (xy 120.65 22.86))
     (stroke (width 0) (type default) (color 0 0 0 0))
@@
   (symbol (lib_id "8bit-computer-rescue:74LS245-8bit-computer-rescue") (at 118.11 58.42 90) (unit 1)
     (in_bom yes) (on_board yes)
-    (property "Reference" "U48" (id 0) (at 103.505 55.88 0)
+    (property "Reference" "U51" (id 0) (at 103.505 55.88 0)
       (effects (font (size 1.27 1.27)) (justify left bottom))
     )
@@
   (symbol (lib_id "8bit-computer-rescue:74LS283-8bit-computer-rescue") (at 153.67 93.98 180) (unit 1)
     (in_bom yes) (on_board yes)
-    (property "Reference" "U49" (id 0) (at 153.67 93.98 0))
+    (property "Reference" "U52" (id 0) (at 153.67 93.98 0))
     (property "Value" "74LS283" (id 1) (at 152.4 85.09 0))
     (property "Footprint" "Package_DIP:DIP-16_W7.62mm" (id 2) (at 153.67 93.98 0)
@@
   (symbol (lib_id "8bit-computer-rescue:74LS283-8bit-computer-rescue") (at 153.67 124.46 180) (unit 1)
     (in_bom yes) (on_board yes)
-    (property "Reference" "U50" (id 0) (at 153.67 124.46 0))
+    (property "Reference" "U53" (id 0) (at 153.67 124.46 0))
     (property "Value" "74LS283" (id 1) (at 152.4 115.57 0))
     (property "Footprint" "Package_DIP:DIP-16_W7.62mm" (id 2) (at 153.67 124.46 0)
@@
   (symbol (lib_id "8bit-computer-rescue:74LS86-8bit-computer-rescue") (at 227.33 107.95 180) (unit 3)
     (in_bom yes) (on_board yes)
-    (property "Reference" "U52" (id 0) (at 226.06 109.22 0))
+    (property "Reference" "U55" (id 0) (at 226.06 109.22 0))
     (property "Value" "74LS86" (id 1) (at 226.06 106.68 0))
     (property "Footprint" "Package_DIP:DIP-14_W7.62mm" (id 2) (at 227.33 107.95 0)
@@
   (symbol (lib_id "8bit-computer-rescue:74LS86-8bit-computer-rescue") (at 227.33 120.65 180) (unit 4)
     (in_bom yes) (on_board yes)
-    (property "Reference" "U52" (id 0) (at 226.06 121.92 0))
+    (property "Reference" "U55" (id 0) (at 226.06 121.92 0))
     (property "Value" "74LS86" (id 1) (at 226.06 119.38 0))
     (property "Footprint" "Package_DIP:DIP-14_W7.62mm" (id 2) (at 227.33 120.65 0)
@@
   (symbol (lib_id "8bit-computer-rescue:74LS86-8bit-computer-rescue") (at 227.33 82.55 180) (unit 1)
     (in_bom yes) (on_board yes)
-    (property "Reference" "U52" (id 0) (at 226.06 83.82 0))
+    (property "Reference" "U55" (id 0) (at 226.06 83.82 0))
     (property "Value" "74LS86" (id 1) (at 226.06 81.28 0))
     (property "Footprint" "Package_DIP:DIP-14_W7.62mm" (id 2) (at 227.33 82.55 0)
@@
   (symbol (lib_id "8bit-computer-rescue:74LS86-8bit-computer-rescue") (at 227.33 95.25 180) (unit 2)
     (in_bom yes) (on_board yes)
-    (property "Reference" "U52" (id 0) (at 226.06 96.52 0))
+    (property "Reference" "U55" (id 0) (at 226.06 96.52 0))
     (property "Value" "74LS86" (id 1) (at 226.06 93.98 0))
     (property "Footprint" "Package_DIP:DIP-14_W7.62mm" (id 2) (at 227.33 95.25 0)
@@
   (symbol (lib_id "8bit-computer-rescue:74LS86-8bit-computer-rescue") (at 227.33 57.15 180) (unit 3)
     (in_bom yes) (on_board yes)
-    (property "Reference" "U51" (id 0) (at 226.06 58.42 0))
+    (property "Reference" "U54" (id 0) (at 226.06 58.42 0))
     (property "Value" "74LS86" (id 1) (at 226.06 55.88 0))
     (property "Footprint" "Package_DIP:DIP-14_W7.62mm" (id 2) (at 227.33 57.15 0)
@@
   (symbol (lib_id "8bit-computer-rescue:74LS86-8bit-computer-rescue") (at 227.33 69.85 180) (unit 4)
     (in_bom yes) (on_board yes)
-    (property "Reference" "U51" (id 0) (at 226.06 71.12 0))
+    (property "Reference" "U54" (id 0) (at 226.06 71.12 0))
     (property "Value" "74LS86" (id 1) (at 226.06 68.58 0))
     (property "Footprint" "Package_DIP:DIP-14_W7.62mm" (id 2) (at 227.33 69.85 0)
@@
   (symbol (lib_id "8bit-computer-rescue:74LS86-8bit-computer-rescue") (at 227.33 31.75 180) (unit 1)
     (in_bom yes) (on_board yes)
-    (property "Reference" "U51" (id 0) (at 226.06 33.02 0))
+    (property "Reference" "U54" (id 0) (at 226.06 33.02 0))
     (property "Value" "74LS86" (id 1) (at 226.06 30.48 0))
     (property "Footprint" "Package_DIP:DIP-14_W7.62mm" (id 2) (at 227.33 31.75 0)
@@
   (symbol (lib_id "8bit-computer-rescue:74LS86-8bit-computer-rescue") (at 227.33 44.45 180) (unit 2)
     (in_bom yes) (on_board yes)
-    (property "Reference" "U51" (id 0) (at 226.06 45.72 0))
+    (property "Reference" "U54" (id 0) (at 226.06 45.72 0))
     (property "Value" "74LS86" (id 1) (at 226.06 43.18 0))
     (property "Footprint" "Package_DIP:DIP-14_W7.62mm" (id 2) (at 227.33 44.45 0)
@@
   (symbol (lib_id "power:VCC") (at 135.89 68.58 0) (unit 1)
     (in_bom yes) (on_board yes)
-    (property "Reference" "#PWR0134" (id 0) (at 135.89 72.39 0)
+    (property "Reference" "#PWR0156" (id 0) (at 135.89 72.39 0)
       (effects (font (size 1.27 1.27)) hide)
     )
@@
   (symbol (lib_id "power:VCC") (at 149.86 154.94 0) (unit 1)
     (in_bom yes) (on_board yes)
-    (property "Reference" "#PWR0135" (id 0) (at 149.86 158.75 0)
+    (property "Reference" "#PWR0157" (id 0) (at 149.86 158.75 0)
       (effects (font (size 1.27 1.27)) hide)
     )
@@
   (symbol (lib_id "power:GND") (at 149.86 172.72 0) (unit 1)
     (in_bom yes) (on_board yes)
-    (property "Reference" "#PWR0136" (id 0) (at 149.86 179.07 0)
+    (property "Reference" "#PWR0158" (id 0) (at 149.86 179.07 0)
       (effects (font (size 1.27 1.27)) hide)
     )
@@
   (symbol (lib_id "power:GND") (at 71.12 116.84 270) (unit 1)
     (in_bom yes) (on_board yes)
-    (property "Reference" "#PWR0133" (id 0) (at 64.77 116.84 0)
-      (effects (font (size 1.27 1.27)) hide)
-    )
+    (property "Reference" "#PWR0155" (id 0) (at 64.77 116.84 0)
+      (effects (font (size 1.27 1.27)) hide)
+    )

Commit message: work on pc2
Parts:
- removed D100, D101, D94, D95, D96, D97, D98, D99: RED, LED_THT:LED_D5.0mm, symbol 8bit-computer-rescue:LED_ALT-Device
- removed D102, D103: BLUE, LED_THT:LED_D5.0mm, symbol 8bit-computer-rescue:LED_ALT-Device
- removed R129, R130, R131, R132, R133, R134, R135, R136, R137, R138: R, Resistor_THT:R_Axial_DIN0207_L6.3mm_D2.5mm_P7.62mm_Horizontal, symbol Device:R
- added D? (x10): LED, symbol Device:LED
- added R? (x10): R_Small, symbol Device:R_Small
Connections:
- net Cin: now also D?.2 (A)
- net Cout: now also D?.2 (A)
- net E_0: now also D?.2 (A)
- net E_1: now also D?.2 (A)
- net E_2: now also D?.2 (A)
- net E_3: now also D?.2 (A)
- net E_4: now also D?.2 (A)
- net E_5: now also D?.2 (A)
- net E_6: now also D?.2 (A)
- net E_7: now also D?.2 (A)
- net GND: now also R?.2, R?.2, R?.2, R?.2, R?.2, R?.2, R?.2, R?.2, R?.2, R?.2
- new net: D?.1 (K), R?.1 (x10)

Commit message: finished todo list
Connections:
- net ~{EO} renamed ~{ΣO}
Changed lines of the file:
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@@
     (effects (font (size 1.524 1.524)) (justify left))
   )
-  (hierarchical_label "~{EO}" (shape input) (at 260.35 22.86 0)
+  (hierarchical_label "~{ΣO}" (shape input) (at 260.35 22.86 0)
     (effects (font (size 1.524 1.524)) (justify left))
   )

Commit message: fixed erc
Parts:
- gave numbers to parts that had none: 20
- renumbered C22 to C21, C23 to C22, U51 to U47, U52 to U48, U53 to U49, U54 to U50, U55 to U51
