File: Kicad Files/alu.kicad_sch (KiCad schematic)
At the start: 29 parts, among them U40 SST39SF040, U41 SST39SF040, U42 74LS173, U43 74HC245, U44 74HC245

Commit message: update
Parts:
- removed D131, D132, D133, D134, D135, D136, D137, D138, D139, D140, D141, D142: LED, symbol Device:LED
- removed R140, R141, R142, R143, R144, R145, R146, R147, R148, R149, R150, R151: R_Small, symbol Device:R_Small
- removed U42: 74LS173, symbol 74xx:74LS173
- removed U44: 74HC245, symbol 74xx:74HC245
- added D1, D106, D2, D3, D4, D49, D5, D6, D7, D8: LED_Small, symbol Device:LED_Small
- added R1, R115, R2, R3, R4, R5, R54, R6, R7, R8: R_Small, symbol Device:R_Small
- added U44: 74LS173, symbol 74xx:74LS173
- renumbered U40 to U65, U41 to U66, U43 to U68
Connections:
- net B_0 is gone; now on net GND: U65.27 (A8), U66.27 (A8)
- net B_1 is gone; now on net GND: U65.26 (A9), U66.26 (A9)
- net B_2 is gone; now on net GND: U65.23 (A10), U66.23 (A10)
- net B_3 is gone; now on net GND: U65.25 (A11), U66.25 (A11)
- net B_4 is gone; now on net GND: U65.4 (A12), U66.4 (A12)
- net B_5 is gone; now on net GND: U65.28 (A13), U66.28 (A13)
- net B_6 is gone; now on net GND: U65.29 (A14), U66.29 (A14)
- net B_7 is gone; now on net GND: U65.3 (A15), U66.3 (A15)
- net CLK: now also U44.7 (Cp)
- net CLR: now also U44.15 (Mr)
- net GND: now also R1.2, R2.2, R3.2, R4.2, R5.2, R6.2, R7.2, R8.2, U44.1 (Oe1), U44.2 (Oe2), U44.8 (GND)
- net VCC: now also R115.2, R54.2, U44.16 (VCC)
- net at U65.15 (D2), U68.4 (A2): now also D6.2 (A)
- net at U65.19 (D5), U68.7 (A5): now also D3.2 (A)
- net at U65.13 (D0), U68.2 (A0): now also D8.2 (A)
- net at U65.17 (D3), U68.5 (A3): now also D5.2 (A)
- net at U66.17 (D3): now also U44.11 (D3)
- net at U66.15 (D2): now also U44.12 (D2)
- net at U66.14 (D1): now also U44.13 (D1)
- net at U66.13 (D0): now also U44.14 (D0)
- net at U65.21 (D7), U68.9 (A7): now also D1.2 (A)
- net at U65.14 (D1), U68.3 (A1): now also D7.2 (A)
- net at U65.18 (D4), U68.6 (A4): now also D4.2 (A)
- net at U65.20 (D6), U68.8 (A6): now also D2.2 (A)
- net D0 renamed d_{i}0
- net D1 renamed d_{i}1
- net D2 renamed d_{i}2
- net D3 renamed d_{i}3
- net D4 renamed d_{i}4
- net D5 renamed d_{i}5
- net D6 renamed d_{i}6
- net D7 renamed d_{i}7
- net ~{FO} renamed ~{Σ}_{O}
- net ~{Σ}_{O}: now also D106.1 (K)
- new net: D8.1 (K), R8.1
- new net: D1.1 (K), R2.1
- new net: D4.1 (K), R4.1
- new net: D3.1 (K), R3.1
- new net: D5.1 (K), R5.1
- new net: D2.1 (K), R1.1
- new net: D6.1 (K), R6.1
- new net: D106.2 (A), R115.1
- new net: D49.2 (A), R54.1
- new net: D7.1 (K), R7.1
- new net F_C: U44.3 (Q0)
- new net F_N: U44.5 (Q2)
- new net F_V: U44.6 (Q3)
- new net F_Z: U44.4 (Q1)
- new net ~{F}: D49.1 (K), U44.10 (E2), U44.9 (E1)
Other:
- moved on the sheet: U68

Commit message: rethink alu
Parts:
- removed U65, U66: SST39SF040, symbol Memory_Flash:SST39SF040
- added U44 (x2): 74LS173, symbol 74xx:74LS173
- added U65, U86: 28C256, symbol Memory_EEPROM:28C256
Connections:
- net A_0: now also U65.6 (A4)
- net A_1: now also U65.5 (A5)
- net A_2: now also U65.4 (A6)
- net A_3: now also U65.3 (A7)
- net A_4: now also U86.6 (A4)
- net A_5: now also U86.5 (A5)
- net A_6: now also U86.4 (A6)
- net A_7: now also U86.3 (A7)
- net F_C: now also U65.25 (A8)
- net GND: now also U44.8 (GND), U44.8 (GND), U65.14 (GND), U86.14 (GND)
- net VCC: now also U44.16 (VCC), U44.16 (VCC), U65.28 (VCC), U86.28 (VCC)
- net ~{Σ}_{O}: no longer U68.19 (CE)
- net at D8.2 (A), U68.2 (A0): now also U65.11 (D0)
- net at D1.2 (A), U68.9 (A7): now also U86.15 (D3)
- net at D4.2 (A), U68.6 (A4): now also U86.11 (D0)
- net at D3.2 (A), U68.7 (A5): now also U86.12 (D1)
- net at D7.2 (A), U68.3 (A1): now also U65.12 (D1)
- net at D6.2 (A), U68.4 (A2): now also U65.13 (D2)
- net at D5.2 (A), U68.5 (A3): now also U65.15 (D3)
- net at D2.2 (A), U68.8 (A6): now also U86.13 (D2)
- net at U44.14 (D0): now also U86.16 (D4)
- net at U44.13 (D1): now also U86.17 (D5)
- net at U44.12 (D2): now also U86.18 (D6)
- net at U44.11 (D3): now also U86.19 (D7)
- net ~{F}: no longer names the net of D49.1 (K), U44.10 (E2), U44.9 (E1)
- new net: U44.3 (Q0), U86.10 (A0)
- new net: U44.4 (Q1), U86.9 (A1)
- new net: U44.5 (Q2), U86.8 (A2)
- new net: U44.6 (Q3), U86.7 (A3)
- new net: U44.3 (Q0), U65.10 (A0)
- new net: U44.4 (Q1), U65.9 (A1)
- new net: U44.5 (Q2), U65.8 (A2)
- new net: U44.6 (Q3), U65.7 (A3)
- new net: U65.17 (D5), U86.24 (A9)
- new net: U65.16 (D4), U86.25 (A8)
- no-connect marks 4 -> 2
Other:
- note added: "F_C"
- note added: "F_Z"
- moved on the sheet: D1, D106, D2, D3, D4, D49, D5, D6, D7, D8, R1, R115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

Commit message: c30
Parts:
- removed D106, D49: LED_Small, symbol Device:LED_Small
- removed R115, R54: R_Small, symbol Device:R_Small
- removed U44 (x2): 74LS173, symbol 74xx:74LS173
- removed U68: 74HC245, symbol 74xx:74HC245
- added U32, U42 (x3): 74HC245, symbol 74xx:74HC245
- added U44 (x2), U54: 74LS173, symbol 74xx:74LS173
- added U64: 27C512, Package_DIP:DIP-28_W15.24mm, symbol Memory_EPROM:27C512
Connections:
- net A_0 is gone; now on net F_C: U65.6 (A4)
- net A_1 is gone; now on net GND: U65.5 (A5)
- net A_2 is gone; now on net GND: U65.4 (A6)
- net A_4 is gone; now on an unnamed net: U86.6 (A4)
- net A_5 is gone; now on an unnamed net: U86.5 (A5)
- net A_6 is gone; now on net GND: U86.4 (A6)
- net A_7 is gone; now on an unnamed net: U86.3 (A7)
- net CLK: now also U44.7 (Cp), U44.7 (Cp), U54.7 (Cp)
- net CLR: now also U44.15 (Mr), U44.15 (Mr), U54.15 (Mr)
- net F_C: now also D1.2 (A), U32.18 (B0); no longer U65.25 (A8)
- net F_N: now also D3.2 (A), U32.16 (B2)
- net F_V: now also D4.2 (A), U32.15 (B3)
- net F_Z: now also D2.2 (A), U32.17 (B1)
- net GND: now also U32.1 (A->B), U32.10 (GND), U42.1 (A->B), U42.1 (A->B), U42.10 (GND), U42.10 (GND), U42.10 (GND), U44.1 (Oe1), U44.1 (Oe1), U44.2 (Oe2), U44.2 (Oe2), U44.8 (GND), U44.8 (GND), U54.1 (Oe1), U54.2 (Oe2), U54.8 (GND), U64.14 (GND), U64.20 (~{CE}), U64.22 (~{OE})
- net VCC: now also U32.20 (VCC), U42.1 (A->B), U42.20 (VCC), U42.20 (VCC), U42.20 (VCC), U44.16 (VCC), U44.16 (VCC), U54.16 (VCC), U64.28 (VCC)
- net d_{i}0: now also U65.10 (A0), U32.2 (A0), U42.2 (A0), U42.2 (A0)
- net d_{i}1: now also U65.9 (A1), U32.3 (A1), U42.3 (A1), U42.3 (A1)
- net d_{i}2: now also U65.8 (A2), U32.4 (A2), U42.4 (A2), U42.4 (A2)
- net d_{i}3: now also U65.7 (A3), U32.5 (A3), U42.5 (A3), U42.5 (A3)
- net d_{i}4: now also U86.10 (A0), U32.6 (A4), U42.6 (A4), U42.6 (A4), U44.14 (D0)
- net d_{i}5: now also U86.9 (A1), U32.7 (A5), U42.7 (A5), U42.7 (A5), U44.13 (D1)
- net d_{i}6: now also U86.8 (A2), U32.8 (A6), U42.8 (A6), U42.8 (A6), U44.12 (D2)
- net d_{i}7: now also U86.7 (A3), U32.9 (A7), U42.9 (A7), U42.9 (A7), U44.11 (D3)
- net at U65.11 (D0): now also U42.18 (B0); no longer D8.2 (A)
- net at U86.15 (D3): now also U42.11 (B7); no longer D1.2 (A)
- net at U86.11 (D0): now also U42.14 (B4); no longer D4.2 (A)
- net at U86.12 (D1): now also U42.13 (B5); no longer D3.2 (A)
- net at U86.13 (D2): now also U42.12 (B6); no longer D2.2 (A)
- net at U65.13 (D2): now also U42.16 (B2); no longer D6.2 (A)
- net at U44.10 (E2), U44.9 (E1): now also U44.10 (E2), U44.9 (E1), U64.18 (D6)
- net at U65.12 (D1): now also U42.17 (B1); no longer D7.2 (A)
- net at U86.1 (A14): now also U42.11 (B7), U44.6 (Q3)
- net at U86.2 (A12): now also U42.13 (B5), U44.4 (Q1)
- net at U86.21 (A10): now also U65.21 (A10), U64.15 (D3)
- net at U86.23 (A11): now also U42.14 (B4), U44.3 (Q0)
- net at U86.24 (A9): now also U65.24 (A9), U64.13 (D2); no longer U65.17 (D5)
- net at U86.25 (A8): now also U65.25 (A8), U64.12 (D1); no longer U65.16 (D4)
- net at U86.26 (A13): now also U42.12 (B6), U44.5 (Q2)
- net at U65.15 (D3): now also U42.15 (B3); no longer D5.2 (A)
- net at U65.1 (A14): now also U42.15 (B3), U54.6 (Q3)
- net at U65.2 (A12): now also U42.17 (B1), U54.4 (Q1)
- net at U65.23 (A11): now also U42.18 (B0), U54.3 (Q0)
- net at U65.26 (A13): now also U42.16 (B2), U54.5 (Q2)
- net A_3: no longer names the net of U65.3 (A7)
- net A_3: now also U64.11 (D0)
- new net: U44.10 (E2), U44.9 (E1), U54.10 (E2), U54.9 (E1), U64.16 (D4)
- new net: U42.15 (B3), U42.5 (A3), U54.11 (D3)
- new net: U42.16 (B2), U42.4 (A2), U54.12 (D2)
- new net: U42.17 (B1), U42.3 (A1), U54.13 (D1)
- new net: U42.18 (B0), U42.2 (A0), U54.14 (D0)
- new net: U42.11 (B7), U42.9 (A7), U44.11 (D3)
- new net: U42.12 (B6), U42.8 (A6), U44.12 (D2)
- new net: U42.13 (B5), U42.7 (A5), U44.13 (D1)
- new net: U42.14 (B4), U42.6 (A4), U44.14 (D0)
- new net: U42.19 (CE), U64.17 (D5)
- new net: U32.19 (CE), U64.19 (D7)
- new net: U42.19 (CE), U65.17 (D5)
- new net: U42.19 (CE), U65.16 (D4)
- new net CA_{M}0: U64.10 (A0)
- new net CA_{M}1: U64.9 (A1)
- new net CA_{M}2: U64.8 (A2)
- new net CA_{M}3: U64.7 (A3)
- new net CA_{S}0: U64.6 (A4)
- new net CA_{S}1: U64.5 (A5)
- new net CA_{S}2: U64.4 (A6)
- new net CA_{S}3: U64.3 (A7)
- new net CO_{M}0: U64.25 (A8)
- new net CO_{M}1: U64.24 (A9)
- new net CO_{M}2: U64.21 (A10)
- new net CO_{M}3: U64.23 (A11)
- new net CO_{S}0: U64.2 (A12)
- new net CO_{S}1: U64.26 (A13)
- new net CO_{S}2: U64.27 (A14)
- new net CO_{S}3: U64.1 (A15)
- new net F_4: D5.2 (A), U32.14 (B4), U44.3 (Q0)
- new net F_5: D6.2 (A), U32.13 (B5), U44.4 (Q1)
- new net F_6: D7.2 (A), U32.12 (B6), U44.5 (Q2)
- new net F_7: D8.2 (A), U32.11 (B7), U44.6 (Q3)
- no-connect marks 2 -> 0
Other:
- note added: "CLK"
- note added: "CLR"
- note added: "~{AI}_{ALU}"
- note added: "~{A}_{I}"
- note added: "~{A}_{O}"
- note added: "~{P}_{I}"
- note added: "~{P}_{O}"
- moved on the sheet: U44, U65, U86
