File: Kicad Files/b-register.kicad_sch (KiCad schematic)
At the start: 20 parts, among them U40 74LS245, U41 74LS173, U42 74LS173

Commit message: finished todo list
Changed lines of the file:
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@@
     (stroke (width 0) (type default) (color 0 0 0 0))
   )
-  (wire (pts (xy 104.14 91.44) (xy 208.28 91.44))
+  (wire (pts (xy 104.14 91.44) (xy 198.755 91.44))
     (stroke (width 0) (type default) (color 0 0 0 0))
   )
@@
     (stroke (width 0) (type default) (color 0 0 0 0))
   )
-  (wire (pts (xy 195.58 40.64) (xy 195.58 35.56))
-    (stroke (width 0) (type default) (color 0 0 0 0))
-  )
   (wire (pts (xy 152.4 143.51) (xy 152.4 147.32))
     (stroke (width 0) (type default) (color 0 0 0 0))
@@
     (stroke (width 0) (type default) (color 0 0 0 0))
   )
-  (wire (pts (xy 160.02 40.64) (xy 195.58 40.64))
-    (stroke (width 0) (type default) (color 0 0 0 0))
-  )
   (wire (pts (xy 137.16 154.94) (xy 137.16 158.75))
     (stroke (width 0) (type default) (color 0 0 0 0))
@@
     (stroke (width 0) (type default) (color 0 0 0 0))
   )
+  (wire (pts (xy 208.28 45.72) (xy 198.755 45.72))
+    (stroke (width 0) (type default) (color 0 0 0 0))
+  )
   (wire (pts (xy 119.38 40.64) (xy 160.02 40.64))
     (stroke (width 0) (type default) (color 0 0 0 0))
@@
     (stroke (width 0) (type default) (color 0 0 0 0))
   )
-  (wire (pts (xy 195.58 35.56) (xy 208.28 35.56))
+  (wire (pts (xy 160.02 40.64) (xy 208.28 40.64))
     (stroke (width 0) (type default) (color 0 0 0 0))
   )
@@
   )
   (wire (pts (xy 99.06 158.75) (xy 106.68 158.75))
+    (stroke (width 0) (type default) (color 0 0 0 0))
+  )
+  (wire (pts (xy 198.755 45.72) (xy 198.755 91.44))
     (stroke (width 0) (type default) (color 0 0 0 0))
   )
@@
     (effects (font (size 1.524 1.524)) (justify right))
   )
-  (hierarchical_label "~{BO}" (shape input) (at 208.28 91.44 0)
+  (hierarchical_label "~{BO}" (shape input) (at 208.28 45.72 0)
     (effects (font (size 1.524 1.524)) (justify left))
   )
@@
     (effects (font (size 1.524 1.524)) (justify left))
   )
-  (hierarchical_label "CLR" (shape input) (at 208.28 35.56 0)
-    (effects (font (size 1.524 1.524)) (justify left))
-  )
+  (hierarchical_label "CLR" (shape input) (at 208.28 40.64 0)
+    (effects (font (size 1.524 1.524)) (justify left))
+  )

Commit message: fixed erc
Parts:
- renumbered C20 to C19, D50 to D87, D51 to D88, D52 to D89, D53 to D90, D54 to D91, D55 to D92, D56 to D93, D57 to D94, R89 to R100, R90 to R101, R91 to R102, R92 to R103, R85 to R96, R86 to R97, R87 to R98, R88 to R99, U40 to U35, U41 to U36, U42 to U37
Changed lines of the file:
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@@
   (symbol (lib_id "8bit-computer-rescue:74LS173-8bit-computer-rescue") (at 173.99 66.04 270) (unit 1)
     (in_bom yes) (on_board yes)
-    (property "Reference" "U42" (id 0) (at 176.53 68.58 0))
+    (property "Reference" "U37" (id 0) (at 176.53 68.58 0))
     (property "Value" "74LS173" (id 1) (at 172.72 68.58 0))
     (property "Footprint" "Package_DIP:DIP-16_W7.62mm" (id 2) (at 173.99 66.04 0)
@@
   (symbol (lib_id "8bit-computer-rescue:74LS245-8bit-computer-rescue") (at 91.44 66.04 90) (unit 1)
     (in_bom yes) (on_board yes)
-    (property "Reference" "U40" (id 0) (at 76.835 63.5 0)
+    (property "Reference" "U35" (id 0) (at 76.835 63.5 0)
       (effects (font (size 1.27 1.27)) (justify left bottom))
     )
@@
   (symbol (lib_id "8bit-computer-rescue:LED_ALT-Device") (at 106.68 139.7 90) (unit 1)
     (in_bom yes) (on_board yes)
-    (property "Reference" "D51" (id 0) (at 104.14 139.7 0))
+    (property "Reference" "D88" (id 0) (at 104.14 139.7 0))
     (property "Value" "RED" (id 1) (at 109.22 139.7 0))
     (property "Footprint" "LED_THT:LED_D5.0mm" (id 2) (at 106.68 139.7 0)
@@
   (symbol (lib_id "Device:R") (at 99.06 151.13 0) (unit 1)
     (in_bom yes) (on_board yes)
-    (property "Reference" "R85" (id 0) (at 101.092 151.13 90))
+    (property "Reference" "R96" (id 0) (at 101.092 151.13 90))
     (property "Value" "R" (id 1) (at 99.06 151.13 90))
     (property "Footprint" "Resistor_THT:R_Axial_DIN0207_L6.3mm_D2.5mm_P7.62mm_Horizontal" (id 2) (at 97.282 151.13 90)
@@
   (symbol (lib_id "Device:R") (at 106.68 151.13 0) (unit 1)
     (in_bom yes) (on_board yes)
-    (property "Reference" "R86" (id 0) (at 108.712 151.13 90))
+    (property "Reference" "R97" (id 0) (at 108.712 151.13 90))
     (property "Value" "R" (id 1) (at 106.68 151.13 90))
     (property "Footprint" "Resistor_THT:R_Axial_DIN0207_L6.3mm_D2.5mm_P7.62mm_Horizontal" (id 2) (at 104.902 151.13 90)
@@
   (symbol (lib_id "Device:R") (at 144.78 151.13 0) (unit 1)
     (in_bom yes) (on_board yes)
-    (property "Reference" "R91" (id 0) (at 146.812 151.13 90))
+    (property "Reference" "R102" (id 0) (at 146.812 151.13 90))
     (property "Value" "R" (id 1) (at 144.78 151.13 90))
     (property "Footprint" "Resistor_THT:R_Axial_DIN0207_L6.3mm_D2.5mm_P7.62mm_Horizontal" (id 2) (at 143.002 151.13 90)
@@
   (symbol (lib_id "power:GND") (at 125.73 163.83 0) (unit 1)
     (in_bom yes) (on_board yes)
-    (property "Reference" "#PWR0122" (id 0) (at 125.73 170.18 0)
+    (property "Reference" "#PWR081" (id 0) (at 125.73 170.18 0)
       (effects (font (size 1.27 1.27)) hide)
     )
@@
   (symbol (lib_id "power:GND") (at 195.58 53.34 0) (unit 1)
     (in_bom yes) (on_board yes)
-    (property "Reference" "#PWR0123" (id 0) (at 195.58 59.69 0)
+    (property "Reference" "#PWR082" (id 0) (at 195.58 59.69 0)
       (effects (font (size 1.27 1.27)) hide)
     )
@@
   (symbol (lib_id "8bit-computer-rescue:74LS173-8bit-computer-rescue") (at 133.35 66.04 270) (unit 1)
     (in_bom yes) (on_board yes)
-    (property "Reference" "U41" (id 0) (at 135.89 68.58 0))
+    (property "Reference" "U36" (id 0) (at 135.89 68.58 0))
     (property "Value" "74LS173" (id 1) (at 132.08 68.58 0))
     (property "Footprint" "Package_DIP:DIP-16_W7.62mm" (id 2) (at 133.35 66.04 0)
@@
   (symbol (lib_id "8bit-computer-rescue:LED_ALT-Device") (at 99.06 139.7 90) (unit 1)
     (in_bom yes) (on_board yes)
-    (property "Reference" "D50" (id 0) (at 96.52 139.7 0))
+    (property "Reference" "D87" (id 0) (at 96.52 139.7 0))
     (property "Value" "RED" (id 1) (at 101.6 139.7 0))
     (property "Footprint" "LED_THT:LED_D5.0mm" (id 2) (at 99.06 139.7 0)
@@
   (symbol (lib_id "8bit-computer-rescue:LED_ALT-Device") (at 114.3 139.7 90) (unit 1)
     (in_bom yes) (on_board yes)
-    (property "Reference" "D52" (id 0) (at 111.76 139.7 0))
+    (property "Reference" "D89" (id 0) (at 111.76 139.7 0))
     (property "Value" "RED" (id 1) (at 116.84 139.7 0))
     (property "Footprint" "LED_THT:LED_D5.0mm" (id 2) (at 114.3 139.7 0)
@@
   (symbol (lib_id "8bit-computer-rescue:LED_ALT-Device") (at 121.92 139.7 90) (unit 1)
     (in_bom yes) (on_board yes)
-    (property "Reference" "D53" (id 0) (at 119.38 139.7 0))
+    (property "Reference" "D90" (id 0) (at 119.38 139.7 0))
     (property "Value" "RED" (id 1) (at 124.46 139.7 0))
     (property "Footprint" "LED_THT:LED_D5.0mm" (id 2) (at 121.92 139.7 0)
@@
   (symbol (lib_id "8bit-computer-rescue:LED_ALT-Device") (at 129.54 139.7 90) (unit 1)
     (in_bom yes) (on_board yes)
-    (property "Reference" "D54" (id 0) (at 127 139.7 0))
+    (property "Reference" "D91" (id 0) (at 127 139.7 0))
     (property "Value" "RED" (id 1) (at 132.08 139.7 0))
     (property "Footprint" "LED_THT:LED_D5.0mm" (id 2) (at 129.54 139.7 0)
@@
   (symbol (lib_id "8bit-computer-rescue:LED_ALT-Device") (at 137.16 139.7 90) (unit 1)
     (in_bom yes) (on_board yes)
-    (property "Reference" "D55" (id 0) (at 134.62 139.7 0))
+    (property "Reference" "D92" (id 0) (at 134.62 139.7 0))
     (property "Value" "RED" (id 1) (at 139.7 139.7 0))
     (property "Footprint" "LED_THT:LED_D5.0mm" (id 2) (at 137.16 139.7 0)
@@
   (symbol (lib_id "8bit-computer-rescue:LED_ALT-Device") (at 144.78 139.7 90) (unit 1)
     (in_bom yes) (on_board yes)
-    (property "Reference" "D56" (id 0) (at 142.24 139.7 0))
+    (property "Reference" "D93" (id 0) (at 142.24 139.7 0))
     (property "Value" "RED" (id 1) (at 147.32 139.7 0))
     (property "Footprint" "LED_THT:LED_D5.0mm" (id 2) (at 144.78 139.7 0)
@@
   (symbol (lib_id "8bit-computer-rescue:LED_ALT-Device") (at 152.4 139.7 90) (unit 1)
     (in_bom yes) (on_board yes)
-    (property "Reference" "D57" (id 0) (at 149.86 139.7 0))
+    (property "Reference" "D94" (id 0) (at 149.86 139.7 0))
     (property "Value" "RED" (id 1) (at 154.94 139.7 0))
     (property "Footprint" "LED_THT:LED_D5.0mm" (id 2) (at 152.4 139.7 0)
@@
   (symbol (lib_id "Device:R") (at 114.3 151.13 0) (unit 1)
     (in_bom yes) (on_board yes)
-    (property "Reference" "R87" (id 0) (at 116.332 151.13 90))
+    (property "Reference" "R98" (id 0) (at 116.332 151.13 90))
     (property "Value" "R" (id 1) (at 114.3 151.13 90))
     (property "Footprint" "Resistor_THT:R_Axial_DIN0207_L6.3mm_D2.5mm_P7.62mm_Horizontal" (id 2) (at 112.522 151.13 90)
@@
   (symbol (lib_id "Device:R") (at 121.92 151.13 0) (unit 1)
     (in_bom yes) (on_board yes)
-    (property "Reference" "R88" (id 0) (at 123.952 151.13 90))
+    (property "Reference" "R99" (id 0) (at 123.952 151.13 90))
     (property "Value" "R" (id 1) (at 121.92 151.13 90))
     (property "Footprint" "Resistor_THT:R_Axial_DIN0207_L6.3mm_D2.5mm_P7.62mm_Horizontal" (id 2) (at 120.142 151.13 90)
@@
   (symbol (lib_id "Device:R") (at 129.54 151.13 0) (unit 1)
     (in_bom yes) (on_board yes)
-    (property "Reference" "R89" (id 0) (at 131.572 151.13 90))
+    (property "Reference" "R100" (id 0) (at 131.572 151.13 90))
     (property "Value" "R" (id 1) (at 129.54 151.13 90))
     (property "Footprint" "Resistor_THT:R_Axial_DIN0207_L6.3mm_D2.5mm_P7.62mm_Horizontal" (id 2) (at 127.762 151.13 90)
@@
   (symbol (lib_id "Device:R") (at 137.16 151.13 0) (unit 1)
     (in_bom yes) (on_board yes)
-    (property "Reference" "R90" (id 0) (at 139.192 151.13 90))
+    (property "Reference" "R101" (id 0) (at 139.192 151.13 90))
     (property "Value" "R" (id 1) (at 137.16 151.13 90))
     (property "Footprint" "Resistor_THT:R_Axial_DIN0207_L6.3mm_D2.5mm_P7.62mm_Horizontal" (id 2) (at 135.382 151.13 90)
@@
   (symbol (lib_id "Device:R") (at 152.4 151.13 0) (unit 1)
     (in_bom yes) (on_board yes)
-    (property "Reference" "R92" (id 0) (at 154.432 151.13 90))
+    (property "Reference" "R103" (id 0) (at 154.432 151.13 90))
     (property "Value" "R" (id 1) (at 152.4 151.13 90))
     (property "Footprint" "Resistor_THT:R_Axial_DIN0207_L6.3mm_D2.5mm_P7.62mm_Horizontal" (id 2) (at 150.622 151.13 90)
@@
   (symbol (lib_id "power:VCC") (at 101.6 83.82 180) (unit 1)
     (in_bom yes) (on_board yes)
-    (property "Reference" "#PWR0121" (id 0) (at 101.6 80.01 0)
+    (property "Reference" "#PWR080" (id 0) (at 101.6 80.01 0)
       (effects (font (size 1.27 1.27)) hide)
     )
@@
   (symbol (lib_id "Device:C") (at 228.6 64.77 0) (unit 1)
     (in_bom yes) (on_board yes)
-    (property "Reference" "C20" (id 0) (at 229.235 62.23 0)
+    (property "Reference" "C19" (id 0) (at 229.235 62.23 0)
       (effects (font (size 1.27 1.27)) (justify left))
     )
@@
   (symbol (lib_id "power:VCC") (at 228.6 58.42 0) (unit 1)
     (in_bom yes) (on_board yes)
-    (property "Reference" "#PWR0124" (id 0) (at 228.6 62.23 0)
+    (property "Reference" "#PWR083" (id 0) (at 228.6 62.23 0)
       (effects (font (size 1.27 1.27)) hide)
     )
@@
   (symbol (lib_id "power:GND") (at 228.6 71.12 0) (unit 1)
     (in_bom yes) (on_board yes)
-    (property "Reference" "#PWR0125" (id 0) (at 228.6 77.47 0)
-      (effects (font (size 1.27 1.27)) hide)
-    )
+    (property "Reference" "#PWR084" (id 0) (at 228.6 77.47 0)
+      (effects (font (size 1.27 1.27)) hide)
+    )
