File: Kicad Files/b-register.kicad_sch (KiCad schematic)
At the start: 20 parts, among them U35 74LS245, U36 74LS173, U37 74LS173

Commit message: tidy up
Parts:
- renumbered C19 to C18, D87 to D71, D88 to D72, D89 to D73, D90 to D74, D91 to D75, D92 to D76, D93 to D77, D94 to D78, R96 to R80, R97 to R81, R98 to R82, R99 to R83, R100 to R84, R101 to R85, R102 to R86, R103 to R87, U35 to U29, U36 to U30, U37 to U31
Changed lines of the file:
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@@
   (symbol (lib_id "8bit-computer-rescue:74LS173-8bit-computer-rescue") (at 186.69 83.82 270) (unit 1)
     (in_bom yes) (on_board yes)
-    (property "Reference" "U37" (id 0) (at 189.23 86.36 0))
+    (property "Reference" "U31" (id 0) (at 189.23 86.36 0))
     (property "Value" "74LS173" (id 1) (at 185.42 86.36 0))
     (property "Footprint" "Package_DIP:DIP-16_W7.62mm" (id 2) (at 186.69 83.82 0)
@@
   (symbol (lib_id "8bit-computer-rescue:74LS245-8bit-computer-rescue") (at 104.14 83.82 90) (unit 1)
     (in_bom yes) (on_board yes)
-    (property "Reference" "U35" (id 0) (at 89.535 81.28 0)
+    (property "Reference" "U29" (id 0) (at 89.535 81.28 0)
       (effects (font (size 1.27 1.27)) (justify left bottom))
     )
@@
   (symbol (lib_id "8bit-computer-rescue:LED_ALT-Device") (at 119.38 157.48 90) (unit 1)
     (in_bom yes) (on_board yes)
-    (property "Reference" "D88" (id 0) (at 116.84 157.48 0))
+    (property "Reference" "D72" (id 0) (at 116.84 157.48 0))
     (property "Value" "RED" (id 1) (at 121.92 157.48 0))
     (property "Footprint" "LED_THT:LED_D5.0mm" (id 2) (at 119.38 157.48 0)
@@
   (symbol (lib_id "Device:R") (at 111.76 168.91 0) (unit 1)
     (in_bom yes) (on_board yes)
-    (property "Reference" "R96" (id 0) (at 113.792 168.91 90))
+    (property "Reference" "R80" (id 0) (at 113.792 168.91 90))
     (property "Value" "R" (id 1) (at 111.76 168.91 90))
     (property "Footprint" "Resistor_THT:R_Axial_DIN0207_L6.3mm_D2.5mm_P7.62mm_Horizontal" (id 2) (at 109.982 168.91 90)
@@
   (symbol (lib_id "Device:R") (at 119.38 168.91 0) (unit 1)
     (in_bom yes) (on_board yes)
-    (property "Reference" "R97" (id 0) (at 121.412 168.91 90))
+    (property "Reference" "R81" (id 0) (at 121.412 168.91 90))
     (property "Value" "R" (id 1) (at 119.38 168.91 90))
     (property "Footprint" "Resistor_THT:R_Axial_DIN0207_L6.3mm_D2.5mm_P7.62mm_Horizontal" (id 2) (at 117.602 168.91 90)
@@
   (symbol (lib_id "Device:R") (at 157.48 168.91 0) (unit 1)
     (in_bom yes) (on_board yes)
-    (property "Reference" "R102" (id 0) (at 159.512 168.91 90))
+    (property "Reference" "R86" (id 0) (at 159.512 168.91 90))
     (property "Value" "R" (id 1) (at 157.48 168.91 90))
     (property "Footprint" "Resistor_THT:R_Axial_DIN0207_L6.3mm_D2.5mm_P7.62mm_Horizontal" (id 2) (at 155.702 168.91 90)
@@
   (symbol (lib_id "power:GND") (at 138.43 181.61 0) (unit 1)
     (in_bom yes) (on_board yes)
-    (property "Reference" "#PWR081" (id 0) (at 138.43 187.96 0)
+    (property "Reference" "#PWR064" (id 0) (at 138.43 187.96 0)
       (effects (font (size 1.27 1.27)) hide)
     )
@@
   (symbol (lib_id "power:GND") (at 208.28 71.12 0) (unit 1)
     (in_bom yes) (on_board yes)
-    (property "Reference" "#PWR082" (id 0) (at 208.28 77.47 0)
+    (property "Reference" "#PWR065" (id 0) (at 208.28 77.47 0)
       (effects (font (size 1.27 1.27)) hide)
     )
@@
   (symbol (lib_id "8bit-computer-rescue:74LS173-8bit-computer-rescue") (at 146.05 83.82 270) (unit 1)
     (in_bom yes) (on_board yes)
-    (property "Reference" "U36" (id 0) (at 148.59 86.36 0))
+    (property "Reference" "U30" (id 0) (at 148.59 86.36 0))
     (property "Value" "74LS173" (id 1) (at 144.78 86.36 0))
     (property "Footprint" "Package_DIP:DIP-16_W7.62mm" (id 2) (at 146.05 83.82 0)
@@
   (symbol (lib_id "8bit-computer-rescue:LED_ALT-Device") (at 111.76 157.48 90) (unit 1)
     (in_bom yes) (on_board yes)
-    (property "Reference" "D87" (id 0) (at 109.22 157.48 0))
+    (property "Reference" "D71" (id 0) (at 109.22 157.48 0))
     (property "Value" "RED" (id 1) (at 114.3 157.48 0))
     (property "Footprint" "LED_THT:LED_D5.0mm" (id 2) (at 111.76 157.48 0)
@@
   (symbol (lib_id "8bit-computer-rescue:LED_ALT-Device") (at 127 157.48 90) (unit 1)
     (in_bom yes) (on_board yes)
-    (property "Reference" "D89" (id 0) (at 124.46 157.48 0))
+    (property "Reference" "D73" (id 0) (at 124.46 157.48 0))
     (property "Value" "RED" (id 1) (at 129.54 157.48 0))
     (property "Footprint" "LED_THT:LED_D5.0mm" (id 2) (at 127 157.48 0)
@@
   (symbol (lib_id "8bit-computer-rescue:LED_ALT-Device") (at 134.62 157.48 90) (unit 1)
     (in_bom yes) (on_board yes)
-    (property "Reference" "D90" (id 0) (at 132.08 157.48 0))
+    (property "Reference" "D74" (id 0) (at 132.08 157.48 0))
     (property "Value" "RED" (id 1) (at 137.16 157.48 0))
     (property "Footprint" "LED_THT:LED_D5.0mm" (id 2) (at 134.62 157.48 0)
@@
   (symbol (lib_id "8bit-computer-rescue:LED_ALT-Device") (at 142.24 157.48 90) (unit 1)
     (in_bom yes) (on_board yes)
-    (property "Reference" "D91" (id 0) (at 139.7 157.48 0))
+    (property "Reference" "D75" (id 0) (at 139.7 157.48 0))
     (property "Value" "RED" (id 1) (at 144.78 157.48 0))
     (property "Footprint" "LED_THT:LED_D5.0mm" (id 2) (at 142.24 157.48 0)
@@
   (symbol (lib_id "8bit-computer-rescue:LED_ALT-Device") (at 149.86 157.48 90) (unit 1)
     (in_bom yes) (on_board yes)
-    (property "Reference" "D92" (id 0) (at 147.32 157.48 0))
+    (property "Reference" "D76" (id 0) (at 147.32 157.48 0))
     (property "Value" "RED" (id 1) (at 152.4 157.48 0))
     (property "Footprint" "LED_THT:LED_D5.0mm" (id 2) (at 149.86 157.48 0)
@@
   (symbol (lib_id "8bit-computer-rescue:LED_ALT-Device") (at 157.48 157.48 90) (unit 1)
     (in_bom yes) (on_board yes)
-    (property "Reference" "D93" (id 0) (at 154.94 157.48 0))
+    (property "Reference" "D77" (id 0) (at 154.94 157.48 0))
     (property "Value" "RED" (id 1) (at 160.02 157.48 0))
     (property "Footprint" "LED_THT:LED_D5.0mm" (id 2) (at 157.48 157.48 0)
@@
   (symbol (lib_id "8bit-computer-rescue:LED_ALT-Device") (at 165.1 157.48 90) (unit 1)
     (in_bom yes) (on_board yes)
-    (property "Reference" "D94" (id 0) (at 162.56 157.48 0))
+    (property "Reference" "D78" (id 0) (at 162.56 157.48 0))
     (property "Value" "RED" (id 1) (at 167.64 157.48 0))
     (property "Footprint" "LED_THT:LED_D5.0mm" (id 2) (at 165.1 157.48 0)
@@
   (symbol (lib_id "Device:R") (at 127 168.91 0) (unit 1)
     (in_bom yes) (on_board yes)
-    (property "Reference" "R98" (id 0) (at 129.032 168.91 90))
+    (property "Reference" "R82" (id 0) (at 129.032 168.91 90))
     (property "Value" "R" (id 1) (at 127 168.91 90))
     (property "Footprint" "Resistor_THT:R_Axial_DIN0207_L6.3mm_D2.5mm_P7.62mm_Horizontal" (id 2) (at 125.222 168.91 90)
@@
   (symbol (lib_id "Device:R") (at 134.62 168.91 0) (unit 1)
     (in_bom yes) (on_board yes)
-    (property "Reference" "R99" (id 0) (at 136.652 168.91 90))
+    (property "Reference" "R83" (id 0) (at 136.652 168.91 90))
     (property "Value" "R" (id 1) (at 134.62 168.91 90))
     (property "Footprint" "Resistor_THT:R_Axial_DIN0207_L6.3mm_D2.5mm_P7.62mm_Horizontal" (id 2) (at 132.842 168.91 90)
@@
   (symbol (lib_id "Device:R") (at 142.24 168.91 0) (unit 1)
     (in_bom yes) (on_board yes)
-    (property "Reference" "R100" (id 0) (at 144.272 168.91 90))
+    (property "Reference" "R84" (id 0) (at 144.272 168.91 90))
     (property "Value" "R" (id 1) (at 142.24 168.91 90))
     (property "Footprint" "Resistor_THT:R_Axial_DIN0207_L6.3mm_D2.5mm_P7.62mm_Horizontal" (id 2) (at 140.462 168.91 90)
@@
   (symbol (lib_id "Device:R") (at 149.86 168.91 0) (unit 1)
     (in_bom yes) (on_board yes)
-    (property "Reference" "R101" (id 0) (at 151.892 168.91 90))
+    (property "Reference" "R85" (id 0) (at 151.892 168.91 90))
     (property "Value" "R" (id 1) (at 149.86 168.91 90))
     (property "Footprint" "Resistor_THT:R_Axial_DIN0207_L6.3mm_D2.5mm_P7.62mm_Horizontal" (id 2) (at 148.082 168.91 90)
@@
   (symbol (lib_id "Device:R") (at 165.1 168.91 0) (unit 1)
     (in_bom yes) (on_board yes)
-    (property "Reference" "R103" (id 0) (at 167.132 168.91 90))
+    (property "Reference" "R87" (id 0) (at 167.132 168.91 90))
     (property "Value" "R" (id 1) (at 165.1 168.91 90))
     (property "Footprint" "Resistor_THT:R_Axial_DIN0207_L6.3mm_D2.5mm_P7.62mm_Horizontal" (id 2) (at 163.322 168.91 90)
@@
   (symbol (lib_id "power:VCC") (at 114.3 101.6 180) (unit 1)
     (in_bom yes) (on_board yes)
-    (property "Reference" "#PWR080" (id 0) (at 114.3 97.79 0)
+    (property "Reference" "#PWR063" (id 0) (at 114.3 97.79 0)
       (effects (font (size 1.27 1.27)) hide)
     )
@@
   (symbol (lib_id "Device:C") (at 241.3 82.55 0) (unit 1)
     (in_bom yes) (on_board yes)
-    (property "Reference" "C19" (id 0) (at 241.935 80.01 0)
+    (property "Reference" "C18" (id 0) (at 241.935 80.01 0)
       (effects (font (size 1.27 1.27)) (justify left))
     )
@@
   (symbol (lib_id "power:VCC") (at 241.3 76.2 0) (unit 1)
     (in_bom yes) (on_board yes)
-    (property "Reference" "#PWR083" (id 0) (at 241.3 80.01 0)
+    (property "Reference" "#PWR066" (id 0) (at 241.3 80.01 0)
       (effects (font (size 1.27 1.27)) hide)
     )
@@
   (symbol (lib_id "power:GND") (at 241.3 88.9 0) (unit 1)
     (in_bom yes) (on_board yes)
-    (property "Reference" "#PWR084" (id 0) (at 241.3 95.25 0)
-      (effects (font (size 1.27 1.27)) hide)
-    )
+    (property "Reference" "#PWR067" (id 0) (at 241.3 95.25 0)
+      (effects (font (size 1.27 1.27)) hide)
+    )

Commit message: updated library
Parts:
- removed D71, D72, D73, D74, D75, D76, D77, D78: RED, LED_THT:LED_D5.0mm, symbol 8bit-computer-rescue:LED_ALT-Device
- removed R80, R81, R82, R83, R84, R85, R86, R87: R, Resistor_THT:R_Axial_DIN0207_L6.3mm_D2.5mm_P7.62mm_Horizontal, symbol Device:R
- removed U29: 74LS245, Package_DIP:DIP-20_W7.62mm, symbol 8bit-computer-rescue:74LS245-8bit-computer-rescue
- removed U30, U31: 74LS173, Package_DIP:DIP-16_W7.62mm, symbol 8bit-computer-rescue:74LS173-8bit-computer-rescue
- added D79, D80, D81, D82, D83, D84, D85, D86: LED, symbol Device:LED
- added R88, R89, R90, R91, R92, R93, R94, R95: R_Small, symbol Device:R_Small
- added U29: 74HC245, symbol 74xx:74HC245
- added U30, U31: 74LS173, symbol 74xx:74LS173
Connections:
- net BUS_0: now also U29.11 (B7), U31.11 (D3)
- net BUS_1: now also U29.12 (B6), U31.12 (D2)
- net BUS_2: now also U29.13 (B5), U31.13 (D1)
- net BUS_3: now also U29.14 (B4), U31.14 (D0)
- net BUS_4: now also U29.15 (B3), U30.11 (D3)
- net BUS_5: now also U29.16 (B2), U30.12 (D2)
- net BUS_6: now also U29.17 (B1), U30.13 (D1)
- net BUS_7: now also U29.18 (B0), U30.14 (D0)
- net B_0: now also D86.2 (A), U29.9 (A7), U31.6 (Q3)
- net B_1: now also D85.2 (A), U29.8 (A6), U31.5 (Q2)
- net B_2: now also D84.2 (A), U29.7 (A5), U31.4 (Q1)
- net B_3: now also D83.2 (A), U29.6 (A4), U31.3 (Q0)
- net B_4: now also D82.2 (A), U29.5 (A3), U30.6 (Q3)
- net B_5: now also D81.2 (A), U29.4 (A2), U30.5 (Q2)
- net B_6: now also D80.2 (A), U29.3 (A1), U30.4 (Q1)
- net B_7: now also D79.2 (A), U29.2 (A0), U30.3 (Q0)
- net CLK: now also U30.7 (Cp), U31.7 (Cp)
- net CLR: now also U30.15 (Mr), U31.15 (Mr)
- net GND: now also R88.2, R89.2, R90.2, R91.2, R92.2, R93.2, R94.2, R95.2, U29.10 (GND), U30.1 (Oe1), U30.16 (VCC), U30.2 (Oe2), U31.1 (Oe1), U31.16 (VCC), U31.2 (Oe2)
- net VCC: now also U29.1 (A->B), U29.20 (VCC), U30.8 (GND), U31.8 (GND)
- net ~{BI}: now also U30.10 (E2), U30.9 (E1), U31.10 (E2), U31.9 (E1)
- net ~{BO}: now also U29.19 (CE)
- new net: D80.1 (K), R89.1
- new net: D81.1 (K), R90.1
- new net: D84.1 (K), R93.1
- new net: D82.1 (K), R91.1
- new net: D79.1 (K), R88.1
- new net: D83.1 (K), R92.1
- new net: D85.1 (K), R94.1
- new net: D86.1 (K), R95.1
Other:
- moved on the sheet: C18

Commit message: im sooo stupiiid
Other:
- moved on the sheet: C18, D79, D80, D81, D82, D83, D84, D85, D86, R88, R89, R90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

Commit message: complete redraw to bus system
Connections:
- net BUS_0 renamed D0
- net BUS_1 renamed D1
- net BUS_2 renamed D2
- net BUS_3 renamed D3
- net BUS_4 renamed D4
- net BUS_5 renamed D5
- net BUS_6 renamed D6
- net BUS_7 renamed D7
Changed lines of the file:
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@@
     (stroke (width 0) (type default) (color 0 0 0 0))
   )
-  (hierarchical_label "BUS_4" (shape bidirectional) (at 60.96 47.625 180)
+  (hierarchical_label "D2" (shape tri_state) (at 60.96 42.545 180)
+    (effects (font (size 1.524 1.524)) (justify right))
+  )
+  (hierarchical_label "D4" (shape tri_state) (at 60.96 47.625 180)
+    (effects (font (size 1.524 1.524)) (justify right))
+  )
+  (hierarchical_label "D1" (shape tri_state) (at 60.96 40.005 180)
     (effects (font (size 1.524 1.524)) (justify right))
   )
   (hierarchical_label "B_5" (shape output) (at 125.476 152.527 0)
     (effects (font (size 1.524 1.524)) (justify left))
-  )
-  (hierarchical_label "BUS_0" (shape bidirectional) (at 60.96 37.465 180)
-    (effects (font (size 1.524 1.524)) (justify right))
   )
   (hierarchical_label "~{BO}" (shape input) (at 245.11 67.945 0)
@@
     (effects (font (size 1.524 1.524)) (justify left))
   )
-  (hierarchical_label "BUS_6" (shape bidirectional) (at 60.96 52.705 180)
-    (effects (font (size 1.524 1.524)) (justify right))
-  )
   (hierarchical_label "B_1" (shape output) (at 125.476 142.367 0)
     (effects (font (size 1.524 1.524)) (justify left))
+  )
+  (hierarchical_label "D0" (shape tri_state) (at 60.96 37.465 180)
+    (effects (font (size 1.524 1.524)) (justify right))
   )
   (hierarchical_label "B_7" (shape output) (at 125.476 157.607 0)
     (effects (font (size 1.524 1.524)) (justify left))
   )
-  (hierarchical_label "BUS_5" (shape bidirectional) (at 60.96 50.165 180)
+  (hierarchical_label "D3" (shape tri_state) (at 60.96 45.085 180)
+    (effects (font (size 1.524 1.524)) (justify right))
+  )
+  (hierarchical_label "D5" (shape tri_state) (at 60.96 50.165 180)
     (effects (font (size 1.524 1.524)) (justify right))
   )
@@
     (effects (font (size 1.524 1.524)) (justify left))
   )
-  (hierarchical_label "BUS_3" (shape bidirectional) (at 60.96 45.085 180)
-    (effects (font (size 1.524 1.524)) (justify right))
-  )
-  (hierarchical_label "BUS_2" (shape bidirectional) (at 60.96 42.545 180)
+  (hierarchical_label "D7" (shape tri_state) (at 60.96 55.245 180)
     (effects (font (size 1.524 1.524)) (justify right))
   )
@@
     (effects (font (size 1.524 1.524)) (justify left))
   )
-  (hierarchical_label "BUS_7" (shape bidirectional) (at 60.96 55.245 180)
+  (hierarchical_label "D6" (shape tri_state) (at 60.96 52.705 180)
     (effects (font (size 1.524 1.524)) (justify right))
   )
-  (hierarchical_label "BUS_1" (shape bidirectional) (at 60.96 40.005 180)
-    (effects (font (size 1.524 1.524)) (justify right))
-  )
