File: Kicad Files/control.kicad_sch (KiCad schematic)
At the start: 61 parts, among them U46 74LS02, U47 74LS161, U48 SST39SF020, U49 SST39SF020, U50 SST39SF020

Commit message: put it allll together
Parts:
- added D? (x8): LED_Small, symbol Device:LED_Small
- added R? (x8): R_Small, symbol Device:R_Small
- added U?: SST39SF020, symbol Memory_Flash:SST39SF020
Connections:
- net CF: now also U?.25 (A11)
- net GND: now also R?.1, R?.1, R?.1, R?.1, R?.1, R?.1, R?.1, R?.1, U?.16 (GND), U?.30 (A17); no longer U48.22 (CE), U48.24 (OE), U49.22 (CE), U49.24 (OE), U50.22 (CE), U50.24 (OE)
- net IR_0: now also U?.12 (A0)
- net IR_1: now also U?.11 (A1)
- net IR_2: now also U?.10 (A2)
- net IR_3: now also U?.9 (A3)
- net IR_4: now also U?.8 (A4)
- net IR_5: now also U?.7 (A5)
- net IR_6: now also U?.6 (A6)
- net IR_7: now also U?.5 (A7)
- net NF: now also U?.26 (A9)
- net OF: now also U?.23 (A10)
- net VCC: now also U?.2 (A16), U?.31 (PGM), U?.32 (VCC)
- net ZF: now also U?.27 (A8)
- net at D69.2 (A), U47.11 (Q3), U48.4 (A12)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: now also U?.4 (A12)
- net at D68.2 (A), U47.12 (Q2), U48.28 (A13)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: now also U?.28 (A13)
- net at D67.2 (A), U47.13 (Q1), U48.29 (A14)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: now also U?.29 (A14)
- net at D66.2 (A), U47.14 (Q0), U48.3 (A15)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: now also U?.3 (A15)
- net at D70.2 (A), U50.21 (D7): no longer U46.3
- net CE: no longer names the net of D81.2 (A)
- net CE: now also U?.18 (D4); no longer U49.18 (D4)
- net HLT: no longer names the net of D77.2 (A), U50.13 (D0)
- net OI: no longer names the net of D78.2 (A)
- net OI: now also U?.21 (D7); no longer U49.21 (D7)
- net RI: no longer names the net of D83.2 (A)
- net RI: now also U?.15 (D2); no longer U49.15 (D2)
- net RO: no longer names the net of D82.2 (A)
- net RO: now also U?.17 (D3); no longer U49.17 (D3)
- net SU: no longer names the net of D86.2 (A)
- net SU: now also U49.21 (D7); no longer U48.21 (D7)
- net ~{AI}: no longer names the net of D93.2 (A)
- net ~{AI}: now also U49.13 (D0); no longer U48.13 (D0)
- net ~{AO}: no longer names the net of D92.2 (A)
- net ~{AO}: now also U49.14 (D1); no longer U48.14 (D1)
- net ~{BI}: no longer names the net of D91.2 (A)
- net ~{BI}: now also U49.15 (D2); no longer U48.15 (D2)
- net ~{BO}: no longer names the net of D90.2 (A)
- net ~{BO}: now also U49.17 (D3); no longer U48.17 (D3)
- net ~{CO}: no longer names the net of D80.2 (A)
- net ~{CO}: now also U?.19 (D5); no longer U49.19 (D5)
- net ~{EO}: no longer names the net of D87.2 (A)
- net ~{EO}: now also U49.20 (D6); no longer U48.20 (D6)
- net ~{FI}: no longer names the net of D85.2 (A)
- net ~{FI}: now also U?.13 (D0); no longer U49.13 (D0)
- net ~{II}: no longer names the net of D89.2 (A)
- net ~{II}: now also U49.18 (D4); no longer U48.18 (D4)
- net ~{IO}: no longer names the net of D88.2 (A)
- net ~{IO}: now also U49.19 (D5); no longer U48.19 (D5)
- net ~{J}: no longer names the net of D79.2 (A)
- net ~{J}: now also U?.20 (D6); no longer U49.20 (D6)
- net ~{MI}: no longer names the net of D84.2 (A)
- net ~{MI}: now also U?.14 (D1); no longer U49.14 (D1)
- new net: D?.1 (K), R?.2 (x8)
- new net: D?.2 (A), U48.13 (D0)
- new net: D?.2 (A), U48.21 (D7)
- new net: D?.2 (A), U48.19 (D5)
- new net: D?.2 (A), U48.15 (D2)
- new net: D?.2 (A), U48.14 (D1)
- new net: D?.2 (A), U48.20 (D6)
- new net: D?.2 (A), U48.17 (D3)
- new net: D?.2 (A), U48.18 (D4)
- new net OVRD: U48.22 (CE), U48.24 (OE), U49.22 (CE), U49.24 (OE), U50.22 (CE), U50.24 (OE), U?.22 (CE), U?.24 (OE)
- no-connect marks 8 -> 9
Other:
- moved on the sheet: D66, D67, D68, D69, D70, D71, D72, D73, D74, D75, D76, D77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

Commit message: finished todo list
Connections:
- net OVRD: no longer U48.22 (CE), U48.24 (OE), U49.22 (CE), U49.24 (OE), U?.22 (CE), U?.24 (OE)
- net VCC: now also U48.22 (CE), U48.24 (OE), U49.22 (CE), U49.24 (OE), U?.22 (CE), U?.24 (OE)
- net ~{RO}: now reaches D76.2 (A), U50.14 (D1)
- net ~{RI}: now reaches D77.2 (A), U50.13 (D0)
- net OI: now reaches D78.2 (A), U?.21 (D7)
- net ~{FI}: now reaches D79.2 (A), U?.20 (D6)
- net ~{IO}: now reaches D80.2 (A), U?.19 (D5)
- net ~{II}: now reaches D81.2 (A), U?.18 (D4)
- net ~{YO}: now reaches D82.2 (A), U?.17 (D3)
- net ~{YI}: now reaches D83.2 (A), U?.15 (D2)
- net ~{XO}: now reaches D84.2 (A), U?.14 (D1)
- net ~{XI}: now reaches D85.2 (A), U?.13 (D0)
- net ~{BO}: now reaches D86.2 (A), U49.21 (D7)
- net ~{BI}: now reaches D87.2 (A), U49.20 (D6)
- net ~{AO}: now reaches D88.2 (A), U49.19 (D5)
- net ~{AI}: now reaches D89.2 (A), U49.18 (D4)
- net SU: now reaches D90.2 (A), U49.17 (D3)
- net ~{ΣO}: now reaches D91.2 (A), U49.15 (D2)
- net ~{MIhb}: now reaches D92.2 (A), U49.14 (D1)
- net ~{MIlb}: now reaches D93.2 (A), U49.13 (D0)
- net ZMS: now reaches U46.3
- net ZMS: now also D?.2 (A), U48.13 (D0)
- net ~{MO}: now reaches D?.2 (A), U48.21 (D7)
- net ~{Jhb}: now reaches D?.2 (A), U48.19 (D5)
- net CO: now reaches D?.2 (A), U48.15 (D2)
- net HLT: now reaches D?.2 (A), U48.14 (D1)
- net ~{Jlb}: now reaches D?.2 (A), U48.20 (D6)
- net CElb: now reaches D?.2 (A), U48.17 (D3)
- net CEhb: now reaches D?.2 (A), U48.18 (D4)
- no-connect marks 9 -> 16

Commit message: fixed erc
Parts:
- gave numbers to parts that had none: 17
- renumbered D66 to D103, D67 to D104, D68 to D105, D69 to D106, D70 to D107, D71 to D108, D72 to D109, D73 to D110, D74 to D111, D75 to D112, D76 to D113, D77 to D114, D78 to D115, D79 to D116, D80 to D117, D81 to D118, D82 to D119, D83 to D120, D84 to D121, D85 to D122, D86 to D123, D87 to D124, D88 to D125, D89 to D126, D90 to D127, D91 to D128, D92 to D129, D93 to D130, R101 to R112, R102 to R113, R103 to R114, R104 to R115, R105 to R116, R106 to R117, R107 to R118, R108 to R119, R109 to R120, R110 to R121, R111 to R122, R112 to R123, R113 to R124, R114 to R125, R115 to R126, R116 to R127, R117 to R128, R118 to R129, R119 to R130, R120 to R131, R121 to R132, R122 to R133, R123 to R134, R124 to R135, R125 to R136, R126 to R137, R127 to R138, R128 to R139, U46 to U41, U47 to U42, U48 to U43, U49 to U44, U50 to U46
