File: Kicad Files/control.kicad_sch (KiCad schematic)
At the start: 78 parts, among them U41 74LS02, U42 74LS161, U43 SST39SF020, U44 SST39SF020, U45 SST39SF020, U46 SST39SF020

Commit message: np3
Changed lines of the file:
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@@
     (effects (font (size 1.524 1.524)) (justify right bottom))
   )
+  (label "~{Jlb}" (at 269.875 222.25 0)
+    (effects (font (size 1.524 1.524)) (justify left bottom))
+  )
+  (label "~{Jhb}" (at 269.875 218.44 0)
+    (effects (font (size 1.524 1.524)) (justify left bottom))
+  )
+  (label "CO" (at 269.875 207.01 0)
+    (effects (font (size 1.524 1.524)) (justify left bottom))
+  )
+  (label "CEhb" (at 269.875 214.63 0)
+    (effects (font (size 1.524 1.524)) (justify left bottom))
+  )
   (label "ZMS" (at 269.875 199.39 0)
+    (effects (font (size 1.524 1.524)) (justify left bottom))
+  )
+  (label "CElb" (at 269.875 210.82 0)
     (effects (font (size 1.524 1.524)) (justify left bottom))
   )
@@
   )
   (hierarchical_label "~{FI}" (shape output) (at 269.875 285.75 0)
-    (effects (font (size 1.524 1.524)) (justify left))
-  )
-  (hierarchical_label "CEhb" (shape output) (at 269.875 214.63 0)
     (effects (font (size 1.524 1.524)) (justify left))
   )
@@
   (hierarchical_label "CF" (shape input) (at 91.44 349.25 270)
     (effects (font (size 1.524 1.524)) (justify right))
-  )
-  (hierarchical_label "~{Jhb}" (shape output) (at 269.875 218.44 0)
-    (effects (font (size 1.524 1.524)) (justify left))
   )
   (hierarchical_label "~{XI}" (shape output) (at 269.875 262.89 0)
@@
     (effects (font (size 1.524 1.524)) (justify left))
   )
-  (hierarchical_label "CO" (shape output) (at 269.875 207.01 0)
-    (effects (font (size 1.524 1.524)) (justify left))
-  )
   (hierarchical_label "IR_2" (shape input) (at 115.57 349.25 270)
     (effects (font (size 1.524 1.524)) (justify right))
@@
   (hierarchical_label "NF" (shape input) (at 96.52 349.25 270)
     (effects (font (size 1.524 1.524)) (justify right))
-  )
-  (hierarchical_label "~{Jlb}" (shape output) (at 269.875 222.25 0)
-    (effects (font (size 1.524 1.524)) (justify left))
   )
   (hierarchical_label "~{YI}" (shape output) (at 269.875 270.51 0)
@@
     (effects (font (size 1.524 1.524)) (justify left))
   )
-  (hierarchical_label "CElb" (shape output) (at 269.875 210.82 0)
-    (effects (font (size 1.524 1.524)) (justify left))
-  )

Commit message: np5
Parts:
- removed U41: 74LS02, symbol 74xx:74LS02
Connections:
- net CLR: now also U42.1 (~{MR})
- net GND: now also U42.3 (D0), U42.4 (D1), U42.5 (D2), U42.6 (D3)
- net VCC: no longer U42.9 (~{PE})
- net ZMS: now also U42.9 (~{PE})
- net OI renamed ZI
- no-connect marks 16 -> 12

Commit message: new control sigs
Parts:
- removed D107, D108, D109, D110, D111, D112, D113, D114, D115, D116, D117, D118, D119, D120, D121, D122, D123, D124, D125, D126, D127, D128, D129, D130, D131, D132, D133, D134, D135, D136, D137, D138: LED_Small, symbol Device:LED_Small
- removed R116, R117, R118, R119, R120, R121, R122, R123, R124, R125, R126, R127, R128, R129, R130, R131, R132, R133, R134, R135, R136, R137, R138, R139, R140, R141, R142, R143, R144, R145, R146, R147: R_Small, symbol Device:R_Small
- added D? (x32): LED, symbol Device:LED
- added R? (x32): R_Small, symbol Device:R_Small
Connections:
- net CEhb is gone; now on net ~{BI}: U43.18 (D4)
- net CElb is gone; now on net ~{BO}: U43.17 (D3)
- net CO is gone; now on net ~{II}: U43.15 (D2)
- net SU is gone; now on net ~{AO}: U44.17 (D3)
- net HLT: now also U45.18 (D4), D?.2 (A); no longer U43.14 (D1)
- net ZI: now also U45.17 (D3), D?.2 (A); no longer U45.21 (D7)
- net ZMS: now also D?.2 (A)
- net ~{AI}: now also D?.2 (A)
- net ~{AO}: now also D?.2 (A); no longer U44.19 (D5)
- net ~{BI}: now also D?.2 (A); no longer U44.20 (D6)
- net ~{BO}: now also D?.2 (A); no longer U44.21 (D7)
- net ~{FI}: now also U44.15 (D2), D?.2 (A); no longer U45.20 (D6)
- net ~{II}: now also D?.2 (A); no longer U45.18 (D4)
- net ~{IO}: now also U43.14 (D1), D?.2 (A); no longer U45.19 (D5)
- net ~{MIhb}: now also U45.20 (D6), D?.2 (A); no longer U44.14 (D1)
- net ~{MIlb}: now also U45.19 (D5), D?.2 (A); no longer U44.13 (D0)
- net ~{MO}: now also U45.21 (D7), D?.2 (A); no longer U43.21 (D7)
- net ~{RI}: now also D?.2 (A)
- net ~{RO}: now also D?.2 (A)
- net ~{XI}: now also D?.2 (A)
- net ~{XO}: now also U44.21 (D7), D?.2 (A); no longer U45.14 (D1)
- net ~{YI}: now also U44.20 (D6), D?.2 (A); no longer U45.15 (D2)
- net ~{YO}: now also U44.19 (D5), D?.2 (A); no longer U45.17 (D3)
- net ~{ΣO}: now also U44.13 (D0), U44.14 (D1), D?.2 (A), D?.2 (A); no longer U44.15 (D2)
- net -1: now reaches U46.20 (D6)
- net -1: now also D?.2 (A)
- net -2: now reaches U46.19 (D5)
- net -2: now also D?.2 (A)
- net -3: now reaches U46.18 (D4)
- net -3: now also D?.2 (A)
- net -4: now reaches U46.17 (D3)
- net -4: now also D?.2 (A)
- net -5: now reaches U46.15 (D2)
- net -5: now also D?.2 (A)
- net -0: now reaches U46.21 (D7)
- net -0: now also D?.2 (A)
- net ~{Jhb} renamed Σ_2
- net Σ_2: now also D?.2 (A)
- net ~{Jlb} renamed Σ_1
- net Σ_1: now also D?.2 (A)
- new net: D?.1 (K), R?.1 (x32)
- new net: R?.2, R?.2, R?.2, R?.2, R?.2, R?.2, R?.2, R?.2 (x4)
- new net -6: D?.2 (A), U45.15 (D2)
- new net -7: D?.2 (A), U45.14 (D1)
- new net Σ_0: D?.2 (A), U43.21 (D7)
- no-connect marks 12 -> 5

Commit message: tidy up
Parts:
- gave numbers to parts that had none: 64
- renumbered D103 to D87, D104 to D88, D105 to D89, D106 to D90, R112 to R96, R113 to R97, R114 to R98, R115 to R99, U42 to U35, U43 to U36, U44 to U37, U45 to U38, U46 to U39

Commit message: updated library
Parts:
- renumbered D92 to D100, D93 to D101, D94 to D102, D95 to D103, D96 to D104, D97 to D105, D98 to D106, D99 to D107, D100 to D108, D101 to D109, D102 to D110, D103 to D111, D104 to D112, D105 to D113, D106 to D114, D107 to D115, D108 to D116, D109 to D117, D110 to D118, D111 to D119, D112 to D120, D113 to D121, D114 to D122, D115 to D123, D116 to D124, D117 to D125, D118 to D126, D119 to D127, D120 to D128, D121 to D129, D122 to D130, D87 to D95, D88 to D96, D89 to D97, D90 to D98, D91 to D99, R96 to R104, R97 to R105, R98 to R106, R99 to R107, R100 to R108, R101 to R109, R102 to R110, R103 to R111, R104 to R112, R105 to R113, R106 to R114, R107 to R115, R108 to R116, R109 to R117, R110 to R118, R111 to R119, R112 to R120, R113 to R121, R114 to R122, R115 to R123, R116 to R124, R117 to R125, R118 to R126, R119 to R127, R120 to R128, R121 to R129, R122 to R130, R123 to R131, R124 to R132, R125 to R133, R126 to R134, R127 to R135, R128 to R136, R129 to R137, R130 to R138, R131 to R139
Connections:
- net -5: now also D118.2 (A), U38.17 (D3); no longer D125.2 (A), U39.15 (D2)
- net HLT: now also D123.2 (A), U39.13 (D0); no longer D119.2 (A), U38.18 (D4)
- net ZI: now also D119.2 (A), U38.18 (D4); no longer D118.2 (A), U38.17 (D3)
- net ~{RI}: now also D124.2 (A), U39.14 (D1); no longer D123.2 (A), U39.13 (D0)
- net ~{RO}: now also D125.2 (A), U39.15 (D2); no longer D124.2 (A), U39.14 (D1)

Commit message: im sooo stupiiid
Connections:
- net OF is gone; now on net CF: U36.23 (A10), U37.23 (A10), U38.23 (A10), U39.23 (A10)
- net -5: now also D125.2 (A), U38.21 (D7); no longer D118.2 (A), U38.17 (D3)
- net -6: now also D124.2 (A), U38.20 (D6); no longer D117.2 (A), U38.15 (D2)
- net CF: no longer U36.25 (A11), U37.25 (A11), U38.25 (A11), U39.25 (A11)
- net GND: now also R108.2, R109.2, R110.2, R111.2, R112.2, R113.2, R114.2, R115.2, R116.2, R117.2, R118.2, R119.2, R120.2, R121.2, R122.2, R123.2, R124.2, R125.2, R126.2, R127.2, R128.2, R129.2, R130.2, R131.2, R132.2, R133.2, R134.2, R135.2, R136.2, R137.2, R138.2, R139.2
- net HLT: now also D115.2 (A); no longer D123.2 (A)
- net ZI: now also D100.2 (A), U36.14 (D1); no longer D119.2 (A), U38.18 (D4)
- net ~{AI}: now also D114.2 (A), U37.21 (D7); no longer D111.2 (A), U37.18 (D4)
- net ~{AO}: now also D113.2 (A), U37.20 (D6); no longer D110.2 (A), U37.17 (D3)
- net ~{BI}: now also D112.2 (A), U37.19 (D5); no longer D103.2 (A), U36.18 (D4)
- net ~{BO}: now also D111.2 (A), U37.18 (D4); no longer D102.2 (A), U36.17 (D3)
- net ~{FI}: now also D110.2 (A), U37.17 (D3); no longer D109.2 (A), U37.15 (D2)
- net ~{II}: now also D121.2 (A), U38.17 (D3); no longer D101.2 (A), U36.15 (D2)
- net ~{IO}: now also D122.2 (A), U38.18 (D4); no longer D100.2 (A), U36.14 (D1)
- net ~{MO}: now also D118.2 (A), U38.15 (D2); no longer D122.2 (A), U38.21 (D7)
- net ~{XI}: now also D104.2 (A), U36.19 (D5); no longer D115.2 (A), U38.13 (D0)
- net ~{XO}: now also D103.2 (A), U36.18 (D4); no longer D114.2 (A), U37.21 (D7)
- net ~{YI}: now also D102.2 (A), U36.17 (D3); no longer D113.2 (A), U37.20 (D6)
- net ~{YO}: now also D101.2 (A), U36.15 (D2); no longer D112.2 (A), U37.19 (D5)
- net ~{ΣO}: no longer D107.2 (A), U37.13 (D0)
- net Σ_0: now also D107.2 (A), U37.13 (D0); no longer D106.2 (A), U36.21 (D7)
- net Σ_1: now also D106.2 (A), U36.21 (D7); no longer D105.2 (A), U36.20 (D6)
- net Σ_2: now also D105.2 (A), U36.20 (D6); no longer D104.2 (A), U36.19 (D5)
- net -7 renamed ~{HI}
- net ~{HI}: now also D117.2 (A); no longer D116.2 (A)
- net ZMS renamed ~{ZO}
- net ~{ZO}: no longer U35.9 (~{PE})
- removed net ~{MIhb}: D121.2 (A), U38.20 (D6)
- net ~{MIlb} renamed MS0
- net MS0: now also D123.2 (A), U35.9 (~{PE}); no longer D120.2 (A)
- net ~{RI} renamed ~{W}
- net ~{W}: now also D119.2 (A); no longer D124.2 (A)
- net ~{RO} renamed ~{R}
- net ~{R}: now also D120.2 (A); no longer D125.2 (A)
- new net BF: U36.25 (A11), U37.25 (A11), U38.25 (A11), U39.25 (A11)
- new net ~{FO}: D109.2 (A), U37.15 (D2)
- new net ~{LI}: D116.2 (A), U38.13 (D0)
Other:
- moved on the sheet: D100, D101, D102, D103, D104, D105, D106, D107, D108, D109, D110, D111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
