File: Kicad Files/inst-register.kicad_sch (KiCad schematic)
At the start: 20 parts, among them U43 74LS245, U44 74LS173, U45 74LS173

Commit message: fixed erc
Parts:
- renumbered C21 to C20, D63 to D100, D64 to D101, D65 to D102, D58 to D95, D59 to D96, D60 to D97, D61 to D98, D62 to D99, R93 to R104, R94 to R105, R95 to R106, R96 to R107, R97 to R108, R98 to R109, R99 to R110, R100 to R111, U43 to U38, U44 to U39, U45 to U40
Changed lines of the file:
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@@
   (symbol (lib_id "8bit-computer-rescue:LED_ALT-Device") (at 139.7 154.94 90) (unit 1)
     (in_bom yes) (on_board yes)
-    (property "Reference" "D62" (id 0) (at 137.16 154.94 0))
+    (property "Reference" "D99" (id 0) (at 137.16 154.94 0))
     (property "Value" "YELLOW" (id 1) (at 142.24 154.94 0))
     (property "Footprint" "LED_THT:LED_D5.0mm" (id 2) (at 139.7 154.94 0)
@@
   (symbol (lib_id "8bit-computer-rescue:LED_ALT-Device") (at 147.32 154.94 90) (unit 1)
     (in_bom yes) (on_board yes)
-    (property "Reference" "D63" (id 0) (at 144.78 154.94 0))
+    (property "Reference" "D100" (id 0) (at 144.78 154.94 0))
     (property "Value" "YELLOW" (id 1) (at 149.86 154.94 0))
     (property "Footprint" "LED_THT:LED_D5.0mm" (id 2) (at 147.32 154.94 0)
@@
   (symbol (lib_id "Device:R") (at 139.7 162.56 0) (unit 1)
     (in_bom yes) (on_board yes)
-    (property "Reference" "R97" (id 0) (at 141.732 162.56 90))
+    (property "Reference" "R108" (id 0) (at 141.732 162.56 90))
     (property "Value" "R" (id 1) (at 139.7 162.56 90))
     (property "Footprint" "Resistor_THT:R_Axial_DIN0207_L6.3mm_D2.5mm_P7.62mm_Horizontal" (id 2) (at 137.922 162.56 90)
@@
   (symbol (lib_id "power:GND") (at 91.44 107.95 0) (unit 1)
     (in_bom yes) (on_board yes)
-    (property "Reference" "#PWR0128" (id 0) (at 91.44 114.3 0)
+    (property "Reference" "#PWR087" (id 0) (at 91.44 114.3 0)
       (effects (font (size 1.27 1.27)) hide)
     )
@@
   (symbol (lib_id "8bit-computer-rescue:74LS173-8bit-computer-rescue") (at 143.51 81.28 270) (unit 1)
     (in_bom yes) (on_board yes)
-    (property "Reference" "U44" (id 0) (at 146.05 83.82 0))
+    (property "Reference" "U39" (id 0) (at 146.05 83.82 0))
     (property "Value" "74LS173" (id 1) (at 142.24 83.82 0))
     (property "Footprint" "Package_DIP:DIP-16_W7.62mm" (id 2) (at 143.51 81.28 0)
@@
   (symbol (lib_id "8bit-computer-rescue:74LS173-8bit-computer-rescue") (at 184.15 81.28 270) (unit 1)
     (in_bom yes) (on_board yes)
-    (property "Reference" "U45" (id 0) (at 186.69 83.82 0))
+    (property "Reference" "U40" (id 0) (at 186.69 83.82 0))
     (property "Value" "74LS173" (id 1) (at 182.88 83.82 0))
     (property "Footprint" "Package_DIP:DIP-16_W7.62mm" (id 2) (at 184.15 81.28 0)
@@
   (symbol (lib_id "8bit-computer-rescue:74LS245-8bit-computer-rescue") (at 101.6 81.28 90) (unit 1)
     (in_bom yes) (on_board yes)
-    (property "Reference" "U43" (id 0) (at 86.995 78.74 0)
+    (property "Reference" "U38" (id 0) (at 86.995 78.74 0)
       (effects (font (size 1.27 1.27)) (justify left bottom))
     )
@@
   (symbol (lib_id "8bit-computer-rescue:LED_ALT-Device") (at 154.94 154.94 90) (unit 1)
     (in_bom yes) (on_board yes)
-    (property "Reference" "D64" (id 0) (at 152.4 154.94 0))
+    (property "Reference" "D101" (id 0) (at 152.4 154.94 0))
     (property "Value" "YELLOW" (id 1) (at 157.48 154.94 0))
     (property "Footprint" "LED_THT:LED_D5.0mm" (id 2) (at 154.94 154.94 0)
@@
   (symbol (lib_id "8bit-computer-rescue:LED_ALT-Device") (at 162.56 154.94 90) (unit 1)
     (in_bom yes) (on_board yes)
-    (property "Reference" "D65" (id 0) (at 160.02 154.94 0))
+    (property "Reference" "D102" (id 0) (at 160.02 154.94 0))
     (property "Value" "YELLOW" (id 1) (at 165.1 154.94 0))
     (property "Footprint" "LED_THT:LED_D5.0mm" (id 2) (at 162.56 154.94 0)
@@
   (symbol (lib_id "Device:R") (at 109.22 162.56 0) (unit 1)
     (in_bom yes) (on_board yes)
-    (property "Reference" "R93" (id 0) (at 111.252 162.56 90))
+    (property "Reference" "R104" (id 0) (at 111.252 162.56 90))
     (property "Value" "R" (id 1) (at 109.22 162.56 90))
     (property "Footprint" "Resistor_THT:R_Axial_DIN0207_L6.3mm_D2.5mm_P7.62mm_Horizontal" (id 2) (at 107.442 162.56 90)
@@
   (symbol (lib_id "Device:R") (at 116.84 162.56 0) (unit 1)
     (in_bom yes) (on_board yes)
-    (property "Reference" "R94" (id 0) (at 118.872 162.56 90))
+    (property "Reference" "R105" (id 0) (at 118.872 162.56 90))
     (property "Value" "R" (id 1) (at 116.84 162.56 90))
     (property "Footprint" "Resistor_THT:R_Axial_DIN0207_L6.3mm_D2.5mm_P7.62mm_Horizontal" (id 2) (at 115.062 162.56 90)
@@
   (symbol (lib_id "Device:R") (at 124.46 162.56 0) (unit 1)
     (in_bom yes) (on_board yes)
-    (property "Reference" "R95" (id 0) (at 126.492 162.56 90))
+    (property "Reference" "R106" (id 0) (at 126.492 162.56 90))
     (property "Value" "R" (id 1) (at 124.46 162.56 90))
     (property "Footprint" "Resistor_THT:R_Axial_DIN0207_L6.3mm_D2.5mm_P7.62mm_Horizontal" (id 2) (at 122.682 162.56 90)
@@
   (symbol (lib_id "Device:R") (at 132.08 162.56 0) (unit 1)
     (in_bom yes) (on_board yes)
-    (property "Reference" "R96" (id 0) (at 134.112 162.56 90))
+    (property "Reference" "R107" (id 0) (at 134.112 162.56 90))
     (property "Value" "R" (id 1) (at 132.08 162.56 90))
     (property "Footprint" "Resistor_THT:R_Axial_DIN0207_L6.3mm_D2.5mm_P7.62mm_Horizontal" (id 2) (at 130.302 162.56 90)
@@
   (symbol (lib_id "Device:R") (at 147.32 162.56 0) (unit 1)
     (in_bom yes) (on_board yes)
-    (property "Reference" "R98" (id 0) (at 149.352 162.56 90))
+    (property "Reference" "R109" (id 0) (at 149.352 162.56 90))
     (property "Value" "R" (id 1) (at 147.32 162.56 90))
     (property "Footprint" "Resistor_THT:R_Axial_DIN0207_L6.3mm_D2.5mm_P7.62mm_Horizontal" (id 2) (at 145.542 162.56 90)
@@
   (symbol (lib_id "Device:R") (at 154.94 162.56 0) (unit 1)
     (in_bom yes) (on_board yes)
-    (property "Reference" "R99" (id 0) (at 156.972 162.56 90))
+    (property "Reference" "R110" (id 0) (at 156.972 162.56 90))
     (property "Value" "R" (id 1) (at 154.94 162.56 90))
     (property "Footprint" "Resistor_THT:R_Axial_DIN0207_L6.3mm_D2.5mm_P7.62mm_Horizontal" (id 2) (at 153.162 162.56 90)
@@
   (symbol (lib_id "Device:R") (at 162.56 162.56 0) (unit 1)
     (in_bom yes) (on_board yes)
-    (property "Reference" "R100" (id 0) (at 164.592 162.56 90))
+    (property "Reference" "R111" (id 0) (at 164.592 162.56 90))
     (property "Value" "R" (id 1) (at 162.56 162.56 90))
     (property "Footprint" "Resistor_THT:R_Axial_DIN0207_L6.3mm_D2.5mm_P7.62mm_Horizontal" (id 2) (at 160.782 162.56 90)
@@
   (symbol (lib_id "power:GND") (at 135.89 166.37 0) (unit 1)
     (in_bom yes) (on_board yes)
-    (property "Reference" "#PWR0130" (id 0) (at 135.89 172.72 0)
+    (property "Reference" "#PWR089" (id 0) (at 135.89 172.72 0)
       (effects (font (size 1.27 1.27)) hide)
     )
@@
   (symbol (lib_id "power:VCC") (at 111.76 99.06 180) (unit 1)
     (in_bom yes) (on_board yes)
-    (property "Reference" "#PWR0129" (id 0) (at 111.76 95.25 0)
+    (property "Reference" "#PWR088" (id 0) (at 111.76 95.25 0)
       (effects (font (size 1.27 1.27)) hide)
     )
@@
   (symbol (lib_id "power:GND") (at 205.74 68.58 0) (unit 1)
     (in_bom yes) (on_board yes)
-    (property "Reference" "#PWR0131" (id 0) (at 205.74 74.93 0)
+    (property "Reference" "#PWR090" (id 0) (at 205.74 74.93 0)
       (effects (font (size 1.27 1.27)) hide)
     )
@@
   (symbol (lib_id "Device:C") (at 64.77 88.9 0) (unit 1)
     (in_bom yes) (on_board yes)
-    (property "Reference" "C21" (id 0) (at 65.405 86.36 0)
+    (property "Reference" "C20" (id 0) (at 65.405 86.36 0)
       (effects (font (size 1.27 1.27)) (justify left))
     )
@@
   (symbol (lib_id "power:GND") (at 64.77 95.25 0) (unit 1)
     (in_bom yes) (on_board yes)
-    (property "Reference" "#PWR0127" (id 0) (at 64.77 101.6 0)
+    (property "Reference" "#PWR086" (id 0) (at 64.77 101.6 0)
       (effects (font (size 1.27 1.27)) hide)
     )
@@
   (symbol (lib_id "power:VCC") (at 64.77 82.55 0) (unit 1)
     (in_bom yes) (on_board yes)
-    (property "Reference" "#PWR0126" (id 0) (at 64.77 86.36 0)
+    (property "Reference" "#PWR085" (id 0) (at 64.77 86.36 0)
       (effects (font (size 1.27 1.27)) hide)
     )
@@
   (symbol (lib_id "8bit-computer-rescue:LED_ALT-Device") (at 109.22 154.94 90) (unit 1)
     (in_bom yes) (on_board yes)
-    (property "Reference" "D58" (id 0) (at 106.68 154.94 0))
+    (property "Reference" "D95" (id 0) (at 106.68 154.94 0))
     (property "Value" "YELLOW" (id 1) (at 111.76 154.94 0))
     (property "Footprint" "LED_THT:LED_D5.0mm" (id 2) (at 109.22 154.94 0)
@@
   (symbol (lib_id "8bit-computer-rescue:LED_ALT-Device") (at 116.84 154.94 90) (unit 1)
     (in_bom yes) (on_board yes)
-    (property "Reference" "D59" (id 0) (at 114.3 154.94 0))
+    (property "Reference" "D96" (id 0) (at 114.3 154.94 0))
     (property "Value" "YELLOW" (id 1) (at 119.38 154.94 0))
     (property "Footprint" "LED_THT:LED_D5.0mm" (id 2) (at 116.84 154.94 0)
@@
   (symbol (lib_id "8bit-computer-rescue:LED_ALT-Device") (at 124.46 154.94 90) (unit 1)
     (in_bom yes) (on_board yes)
-    (property "Reference" "D60" (id 0) (at 121.92 154.94 0))
+    (property "Reference" "D97" (id 0) (at 121.92 154.94 0))
     (property "Value" "YELLOW" (id 1) (at 127 154.94 0))
     (property "Footprint" "LED_THT:LED_D5.0mm" (id 2) (at 124.46 154.94 0)
@@
   (symbol (lib_id "8bit-computer-rescue:LED_ALT-Device") (at 132.08 154.94 90) (unit 1)
     (in_bom yes) (on_board yes)
-    (property "Reference" "D61" (id 0) (at 129.54 154.94 0))
+    (property "Reference" "D98" (id 0) (at 129.54 154.94 0))
     (property "Value" "YELLOW" (id 1) (at 134.62 154.94 0))
     (property "Footprint" "LED_THT:LED_D5.0mm" (id 2) (at 132.08 154.94 0)
