File: Kicad Files/x-register.kicad_sch (KiCad schematic)
At the start: 20 parts

Commit message: finished todo list
Changed lines of the file:
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@@
     (stroke (width 0) (type default) (color 0 0 0 0))
   )
-  (wire (pts (xy 204.47 50.8) (xy 217.17 50.8))
+  (wire (pts (xy 168.91 55.88) (xy 217.17 55.88))
     (stroke (width 0) (type default) (color 0 0 0 0))
   )
@@
     (stroke (width 0) (type default) (color 0 0 0 0))
   )
+  (wire (pts (xy 217.17 60.96) (xy 207.645 60.96))
+    (stroke (width 0) (type default) (color 0 0 0 0))
+  )
   (wire (pts (xy 107.95 158.75) (xy 107.95 162.56))
     (stroke (width 0) (type default) (color 0 0 0 0))
@@
     (stroke (width 0) (type default) (color 0 0 0 0))
   )
-  (wire (pts (xy 168.91 55.88) (xy 204.47 55.88))
-    (stroke (width 0) (type default) (color 0 0 0 0))
-  )
   (wire (pts (xy 153.67 170.18) (xy 153.67 173.99))
     (stroke (width 0) (type default) (color 0 0 0 0))
@@
     (stroke (width 0) (type default) (color 0 0 0 0))
   )
-  (wire (pts (xy 113.03 106.68) (xy 217.17 106.68))
+  (wire (pts (xy 113.03 106.68) (xy 207.645 106.68))
     (stroke (width 0) (type default) (color 0 0 0 0))
   )
@@
     (stroke (width 0) (type default) (color 0 0 0 0))
   )
-  (wire (pts (xy 204.47 55.88) (xy 204.47 50.8))
-    (stroke (width 0) (type default) (color 0 0 0 0))
-  )
   (wire (pts (xy 138.43 58.42) (xy 176.53 58.42))
     (stroke (width 0) (type default) (color 0 0 0 0))
@@
   )
   (wire (pts (xy 46.99 48.26) (xy 87.63 48.26))
+    (stroke (width 0) (type default) (color 0 0 0 0))
+  )
+  (wire (pts (xy 207.645 60.96) (xy 207.645 106.68))
     (stroke (width 0) (type default) (color 0 0 0 0))
   )
@@
     (effects (font (size 1.524 1.524)) (justify left))
   )
-  (hierarchical_label "~{XO}" (shape input) (at 217.17 106.68 0)
+  (hierarchical_label "~{XO}" (shape input) (at 217.17 60.96 0)
     (effects (font (size 1.524 1.524)) (justify left))
   )
@@
     (effects (font (size 1.524 1.524)) (justify right))
   )
-  (hierarchical_label "CLR" (shape input) (at 217.17 50.8 0)
+  (hierarchical_label "CLR" (shape input) (at 217.17 55.88 0)
     (effects (font (size 1.524 1.524)) (justify left))
   )

Commit message: fixed erc
Parts:
- removed C?: C, Capacitor_THT:C_Disc_D4.3mm_W1.9mm_P5.00mm, symbol Device:C
- removed D? (x8): RED, LED_THT:LED_D5.0mm, symbol 8bit-computer-rescue:LED_ALT-Device
- removed R? (x8): R, Resistor_THT:R_Axial_DIN0207_L6.3mm_D2.5mm_P7.62mm_Horizontal, symbol Device:R
- removed U? (x2): 74LS173, Package_DIP:DIP-16_W7.62mm, symbol 8bit-computer-rescue:74LS173-8bit-computer-rescue
- removed U?: 74LS245, Package_DIP:DIP-20_W7.62mm, symbol 8bit-computer-rescue:74LS245-8bit-computer-rescue
- added C23: C, Capacitor_THT:C_Disc_D4.3mm_W1.9mm_P5.00mm, symbol Device:C
- added D153, D154, D155, D156, D157, D158, D159, D160: RED, LED_THT:LED_D5.0mm, symbol 8bit-computer-rescue:LED_ALT-Device
- added R162, R163, R164, R165, R166, R167, R168, R169: R, Resistor_THT:R_Axial_DIN0207_L6.3mm_D2.5mm_P7.62mm_Horizontal, symbol Device:R
- added U64: 74LS245, Package_DIP:DIP-20_W7.62mm, symbol 8bit-computer-rescue:74LS245-8bit-computer-rescue
- added U65, U66: 74LS173, Package_DIP:DIP-16_W7.62mm, symbol 8bit-computer-rescue:74LS173-8bit-computer-rescue
Connections:
- net BUS_0: now also U64.11 (B7), U66.11 (D3)
- net BUS_1: now also U64.12 (B6), U66.12 (D2)
- net BUS_2: now also U64.13 (B5), U66.13 (D1)
- net BUS_3: now also U64.14 (B4), U66.14 (D0)
- net BUS_4: now also U64.15 (B3), U65.11 (D3)
- net BUS_5: now also U64.16 (B2), U65.12 (D2)
- net BUS_6: now also U64.17 (B1), U65.13 (D1)
- net BUS_7: now also U64.18 (B0), U65.14 (D0)
- net CLK: now also U65.7 (Cp), U66.7 (Cp)
- net CLR: now also U65.15 (Mr), U66.15 (Mr)
- net GND: now also C23.2, R162.2, R163.2, R164.2, R165.2, R166.2, R167.2, R168.2, R169.2, U64.10 (GND), U65.1 (Oe1), U65.2 (Oe2), U65.8 (GND), U66.1 (Oe1), U66.2 (Oe2), U66.8 (GND)
- net VCC: now also C23.1, U64.1 (A->B), U64.20 (VCC), U65.16 (VCC), U66.16 (VCC)
- net ~{XI}: now also U65.10 (E2), U65.9 (E1), U66.10 (E2), U66.9 (E1)
- net ~{XO}: now also U64.19 (CE)
- new net: D160.1 (K), R169.1
- new net: D160.2 (A), U64.9 (A7), U66.6 (Q3)
- new net: D153.1 (K), R162.1
- new net: D158.1 (K), R167.1
- new net: D153.2 (A), U64.2 (A0), U65.3 (Q0)
- new net: D154.2 (A), U64.3 (A1), U65.4 (Q1)
- new net: D155.2 (A), U64.4 (A2), U65.5 (Q2)
- new net: D156.2 (A), U64.5 (A3), U65.6 (Q3)
- new net: D157.2 (A), U64.6 (A4), U66.3 (Q0)
- new net: D158.2 (A), U64.7 (A5), U66.4 (Q1)
- new net: D159.2 (A), U64.8 (A6), U66.5 (Q2)
- new net: D154.1 (K), R163.1
- new net: D157.1 (K), R166.1
- new net: D156.1 (K), R165.1
- new net: D155.1 (K), R164.1
- new net: D159.1 (K), R168.1
