File: Kicad Files/x-register.kicad_sch (KiCad schematic)
At the start: 20 parts, among them U64 74LS245, U65 74LS173, U66 74LS173

Commit message: tidy up
Parts:
- renumbered C23 to C20, D153 to D135, D154 to D136, D155 to D137, D156 to D138, D157 to D139, D158 to D140, D159 to D141, D160 to D142, R162 to R144, R163 to R145, R164 to R146, R165 to R147, R166 to R148, R167 to R149, R168 to R150, R169 to R151, U64 to U43, U65 to U44, U66 to U45
Changed lines of the file:
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@@
   (symbol (lib_id "8bit-computer-rescue:LED_ALT-Device") (at 161.29 154.94 90) (unit 1)
     (in_bom yes) (on_board yes)
-    (property "Reference" "D160" (id 0) (at 158.75 154.94 0))
+    (property "Reference" "D142" (id 0) (at 158.75 154.94 0))
     (property "Value" "RED" (id 1) (at 163.83 154.94 0))
     (property "Footprint" "LED_THT:LED_D5.0mm" (id 2) (at 161.29 154.94 0)
@@
   (symbol (lib_id "Device:R") (at 107.95 166.37 0) (unit 1)
     (in_bom yes) (on_board yes)
-    (property "Reference" "R162" (id 0) (at 109.982 166.37 90))
+    (property "Reference" "R144" (id 0) (at 109.982 166.37 90))
     (property "Value" "R" (id 1) (at 107.95 166.37 90))
     (property "Footprint" "Resistor_THT:R_Axial_DIN0207_L6.3mm_D2.5mm_P7.62mm_Horizontal" (id 2) (at 106.172 166.37 90)
@@
   (symbol (lib_id "power:VCC") (at 110.49 99.06 180) (unit 1)
     (in_bom yes) (on_board yes)
-    (property "Reference" "#PWR0127" (id 0) (at 110.49 95.25 0)
+    (property "Reference" "#PWR0109" (id 0) (at 110.49 95.25 0)
       (effects (font (size 1.27 1.27)) hide)
     )
@@
   (symbol (lib_id "Device:C") (at 240.03 80.01 0) (unit 1)
     (in_bom yes) (on_board yes)
-    (property "Reference" "C23" (id 0) (at 240.665 77.47 0)
+    (property "Reference" "C20" (id 0) (at 240.665 77.47 0)
       (effects (font (size 1.27 1.27)) (justify left))
     )
@@
   (symbol (lib_id "Device:R") (at 146.05 166.37 0) (unit 1)
     (in_bom yes) (on_board yes)
-    (property "Reference" "R167" (id 0) (at 148.082 166.37 90))
+    (property "Reference" "R149" (id 0) (at 148.082 166.37 90))
     (property "Value" "R" (id 1) (at 146.05 166.37 90))
     (property "Footprint" "Resistor_THT:R_Axial_DIN0207_L6.3mm_D2.5mm_P7.62mm_Horizontal" (id 2) (at 144.272 166.37 90)
@@
   (symbol (lib_id "8bit-computer-rescue:74LS245-8bit-computer-rescue") (at 100.33 81.28 90) (unit 1)
     (in_bom yes) (on_board yes)
-    (property "Reference" "U64" (id 0) (at 85.725 78.74 0)
+    (property "Reference" "U43" (id 0) (at 85.725 78.74 0)
       (effects (font (size 1.27 1.27)) (justify left bottom))
     )
@@
   (symbol (lib_id "power:VCC") (at 240.03 73.66 0) (unit 1)
     (in_bom yes) (on_board yes)
-    (property "Reference" "#PWR0130" (id 0) (at 240.03 77.47 0)
+    (property "Reference" "#PWR0112" (id 0) (at 240.03 77.47 0)
       (effects (font (size 1.27 1.27)) hide)
     )
@@
   (symbol (lib_id "power:GND") (at 240.03 86.36 0) (unit 1)
     (in_bom yes) (on_board yes)
-    (property "Reference" "#PWR0131" (id 0) (at 240.03 92.71 0)
+    (property "Reference" "#PWR0113" (id 0) (at 240.03 92.71 0)
       (effects (font (size 1.27 1.27)) hide)
     )
@@
   (symbol (lib_id "Device:R") (at 115.57 166.37 0) (unit 1)
     (in_bom yes) (on_board yes)
-    (property "Reference" "R163" (id 0) (at 117.602 166.37 90))
+    (property "Reference" "R145" (id 0) (at 117.602 166.37 90))
     (property "Value" "R" (id 1) (at 115.57 166.37 90))
     (property "Footprint" "Resistor_THT:R_Axial_DIN0207_L6.3mm_D2.5mm_P7.62mm_Horizontal" (id 2) (at 113.792 166.37 90)
@@
   (symbol (lib_id "power:GND") (at 204.47 68.58 0) (unit 1)
     (in_bom yes) (on_board yes)
-    (property "Reference" "#PWR0129" (id 0) (at 204.47 74.93 0)
+    (property "Reference" "#PWR0111" (id 0) (at 204.47 74.93 0)
       (effects (font (size 1.27 1.27)) hide)
     )
@@
   (symbol (lib_id "8bit-computer-rescue:74LS173-8bit-computer-rescue") (at 182.88 81.28 270) (unit 1)
     (in_bom yes) (on_board yes)
-    (property "Reference" "U66" (id 0) (at 185.42 83.82 0))
+    (property "Reference" "U45" (id 0) (at 185.42 83.82 0))
     (property "Value" "74LS173" (id 1) (at 181.61 83.82 0))
     (property "Footprint" "Package_DIP:DIP-16_W7.62mm" (id 2) (at 182.88 81.28 0)
@@
   (symbol (lib_id "8bit-computer-rescue:LED_ALT-Device") (at 146.05 154.94 90) (unit 1)
     (in_bom yes) (on_board yes)
-    (property "Reference" "D158" (id 0) (at 143.51 154.94 0))
+    (property "Reference" "D140" (id 0) (at 143.51 154.94 0))
     (property "Value" "RED" (id 1) (at 148.59 154.94 0))
     (property "Footprint" "LED_THT:LED_D5.0mm" (id 2) (at 146.05 154.94 0)
@@
   (symbol (lib_id "8bit-computer-rescue:LED_ALT-Device") (at 115.57 154.94 90) (unit 1)
     (in_bom yes) (on_board yes)
-    (property "Reference" "D154" (id 0) (at 113.03 154.94 0))
+    (property "Reference" "D136" (id 0) (at 113.03 154.94 0))
     (property "Value" "RED" (id 1) (at 118.11 154.94 0))
     (property "Footprint" "LED_THT:LED_D5.0mm" (id 2) (at 115.57 154.94 0)
@@
   (symbol (lib_id "Device:R") (at 161.29 166.37 0) (unit 1)
     (in_bom yes) (on_board yes)
-    (property "Reference" "R169" (id 0) (at 163.322 166.37 90))
+    (property "Reference" "R151" (id 0) (at 163.322 166.37 90))
     (property "Value" "R" (id 1) (at 161.29 166.37 90))
     (property "Footprint" "Resistor_THT:R_Axial_DIN0207_L6.3mm_D2.5mm_P7.62mm_Horizontal" (id 2) (at 159.512 166.37 90)
@@
   (symbol (lib_id "Device:R") (at 138.43 166.37 0) (unit 1)
     (in_bom yes) (on_board yes)
-    (property "Reference" "R166" (id 0) (at 140.462 166.37 90))
+    (property "Reference" "R148" (id 0) (at 140.462 166.37 90))
     (property "Value" "R" (id 1) (at 138.43 166.37 90))
     (property "Footprint" "Resistor_THT:R_Axial_DIN0207_L6.3mm_D2.5mm_P7.62mm_Horizontal" (id 2) (at 136.652 166.37 90)
@@
   (symbol (lib_id "8bit-computer-rescue:LED_ALT-Device") (at 130.81 154.94 90) (unit 1)
     (in_bom yes) (on_board yes)
-    (property "Reference" "D156" (id 0) (at 128.27 154.94 0))
+    (property "Reference" "D138" (id 0) (at 128.27 154.94 0))
     (property "Value" "RED" (id 1) (at 133.35 154.94 0))
     (property "Footprint" "LED_THT:LED_D5.0mm" (id 2) (at 130.81 154.94 0)
@@
   (symbol (lib_id "8bit-computer-rescue:LED_ALT-Device") (at 123.19 154.94 90) (unit 1)
     (in_bom yes) (on_board yes)
-    (property "Reference" "D155" (id 0) (at 120.65 154.94 0))
+    (property "Reference" "D137" (id 0) (at 120.65 154.94 0))
     (property "Value" "RED" (id 1) (at 125.73 154.94 0))
     (property "Footprint" "LED_THT:LED_D5.0mm" (id 2) (at 123.19 154.94 0)
@@
   (symbol (lib_id "8bit-computer-rescue:LED_ALT-Device") (at 107.95 154.94 90) (unit 1)
     (in_bom yes) (on_board yes)
-    (property "Reference" "D153" (id 0) (at 105.41 154.94 0))
+    (property "Reference" "D135" (id 0) (at 105.41 154.94 0))
     (property "Value" "RED" (id 1) (at 110.49 154.94 0))
     (property "Footprint" "LED_THT:LED_D5.0mm" (id 2) (at 107.95 154.94 0)
@@
   (symbol (lib_id "power:GND") (at 134.62 179.07 0) (unit 1)
     (in_bom yes) (on_board yes)
-    (property "Reference" "#PWR0128" (id 0) (at 134.62 185.42 0)
+    (property "Reference" "#PWR0110" (id 0) (at 134.62 185.42 0)
       (effects (font (size 1.27 1.27)) hide)
     )
@@
   (symbol (lib_id "Device:R") (at 153.67 166.37 0) (unit 1)
     (in_bom yes) (on_board yes)
-    (property "Reference" "R168" (id 0) (at 155.702 166.37 90))
+    (property "Reference" "R150" (id 0) (at 155.702 166.37 90))
     (property "Value" "R" (id 1) (at 153.67 166.37 90))
     (property "Footprint" "Resistor_THT:R_Axial_DIN0207_L6.3mm_D2.5mm_P7.62mm_Horizontal" (id 2) (at 151.892 166.37 90)
@@
   (symbol (lib_id "8bit-computer-rescue:74LS173-8bit-computer-rescue") (at 142.24 81.28 270) (unit 1)
     (in_bom yes) (on_board yes)
-    (property "Reference" "U65" (id 0) (at 144.78 83.82 0))
+    (property "Reference" "U44" (id 0) (at 144.78 83.82 0))
     (property "Value" "74LS173" (id 1) (at 140.97 83.82 0))
     (property "Footprint" "Package_DIP:DIP-16_W7.62mm" (id 2) (at 142.24 81.28 0)
@@
   (symbol (lib_id "8bit-computer-rescue:LED_ALT-Device") (at 153.67 154.94 90) (unit 1)
     (in_bom yes) (on_board yes)
-    (property "Reference" "D159" (id 0) (at 151.13 154.94 0))
+    (property "Reference" "D141" (id 0) (at 151.13 154.94 0))
     (property "Value" "RED" (id 1) (at 156.21 154.94 0))
     (property "Footprint" "LED_THT:LED_D5.0mm" (id 2) (at 153.67 154.94 0)
@@
   (symbol (lib_id "Device:R") (at 130.81 166.37 0) (unit 1)
     (in_bom yes) (on_board yes)
-    (property "Reference" "R165" (id 0) (at 132.842 166.37 90))
+    (property "Reference" "R147" (id 0) (at 132.842 166.37 90))
     (property "Value" "R" (id 1) (at 130.81 166.37 90))
     (property "Footprint" "Resistor_THT:R_Axial_DIN0207_L6.3mm_D2.5mm_P7.62mm_Horizontal" (id 2) (at 129.032 166.37 90)
@@
   (symbol (lib_id "8bit-computer-rescue:LED_ALT-Device") (at 138.43 154.94 90) (unit 1)
     (in_bom yes) (on_board yes)
-    (property "Reference" "D157" (id 0) (at 135.89 154.94 0))
+    (property "Reference" "D139" (id 0) (at 135.89 154.94 0))
     (property "Value" "RED" (id 1) (at 140.97 154.94 0))
     (property "Footprint" "LED_THT:LED_D5.0mm" (id 2) (at 138.43 154.94 0)
@@
   (symbol (lib_id "Device:R") (at 123.19 166.37 0) (unit 1)
     (in_bom yes) (on_board yes)
-    (property "Reference" "R164" (id 0) (at 125.222 166.37 90))
+    (property "Reference" "R146" (id 0) (at 125.222 166.37 90))
     (property "Value" "R" (id 1) (at 123.19 166.37 90))
     (property "Footprint" "Resistor_THT:R_Axial_DIN0207_L6.3mm_D2.5mm_P7.62mm_Horizontal" (id 2) (at 121.412 166.37 90)

Commit message: updated library
Parts:
- removed D135, D136, D137, D138, D139, D140, D141, D142: RED, LED_THT:LED_D5.0mm, symbol 8bit-computer-rescue:LED_ALT-Device
- removed R144, R145, R146, R147, R148, R149, R150, R151: R, Resistor_THT:R_Axial_DIN0207_L6.3mm_D2.5mm_P7.62mm_Horizontal, symbol Device:R
- removed U43: 74LS245, Package_DIP:DIP-20_W7.62mm, symbol 8bit-computer-rescue:74LS245-8bit-computer-rescue
- removed U44, U45: 74LS173, Package_DIP:DIP-16_W7.62mm, symbol 8bit-computer-rescue:74LS173-8bit-computer-rescue
- added D143, D144, D145, D146, D147, D148, D149, D150: LED, symbol Device:LED
- added R152, R153, R154, R155, R156, R157, R158, R159: R_Small, symbol Device:R_Small
- added U43: 74HC245, symbol 74xx:74HC245
- added U44, U45: 74LS173, symbol 74xx:74LS173
Connections:
- net BUS_0: now also U43.11 (B7), U45.11 (D3)
- net BUS_1: now also U43.12 (B6), U45.12 (D2)
- net BUS_2: now also U43.13 (B5), U45.13 (D1)
- net BUS_3: now also U43.14 (B4), U45.14 (D0)
- net BUS_4: now also U43.15 (B3), U44.11 (D3)
- net BUS_5: now also U43.16 (B2), U44.12 (D2)
- net BUS_6: now also U43.17 (B1), U44.13 (D1)
- net BUS_7: now also U43.18 (B0), U44.14 (D0)
- net CLK: now also U44.7 (Cp), U45.7 (Cp)
- net CLR: now also U44.15 (Mr), U45.15 (Mr)
- net GND: now also R152.2, R153.2, R154.2, R155.2, R156.2, R157.2, R158.2, R159.2, U43.10 (GND), U44.1 (Oe1), U44.16 (VCC), U44.2 (Oe2), U45.1 (Oe1), U45.16 (VCC), U45.2 (Oe2)
- net VCC: now also U43.1 (A->B), U43.20 (VCC), U44.8 (GND), U45.8 (GND)
- net ~{XI}: now also U44.10 (E2), U44.9 (E1), U45.10 (E2), U45.9 (E1)
- net ~{XO}: now also U43.19 (CE)
- new net: D149.1 (K), R158.1
- new net: D147.1 (K), R156.1
- new net: D144.1 (K), R153.1
- new net: D144.2 (A), U43.3 (A1), U44.4 (Q1)
- new net: D147.2 (A), U43.6 (A4), U45.3 (Q0)
- new net: D148.2 (A), U43.7 (A5), U45.4 (Q1)
- new net: D149.2 (A), U43.8 (A6), U45.5 (Q2)
- new net: D150.2 (A), U43.9 (A7), U45.6 (Q3)
- new net: D150.1 (K), R159.1
- new net: D146.1 (K), R155.1
- new net: D146.2 (A), U43.5 (A3), U44.6 (Q3)
- new net: D143.1 (K), R152.1
- new net: D143.2 (A), U43.2 (A0), U44.3 (Q0)
- new net: D145.1 (K), R154.1
- new net: D145.2 (A), U43.4 (A2), U44.5 (Q2)
- new net: D148.1 (K), R157.1
Other:
- moved on the sheet: C20

Commit message: im sooo stupiiid
Parts:
- renumbered U43 to U45, U44 to U46, U45 to U47
Changed lines of the file:
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@@
   (symbol (lib_id "power:GND") (at 218.44 86.36 0) (unit 1)
     (in_bom yes) (on_board yes) (fields_autoplaced)
-    (property "Reference" "#PWR0148" (id 0) (at 218.44 92.71 0)
+    (property "Reference" "#PWR0174" (id 0) (at 218.44 92.71 0)
       (effects (font (size 1.27 1.27)) hide)
     )
@@
   (symbol (lib_id "power:VCC") (at 110.49 99.06 180) (unit 1)
     (in_bom yes) (on_board yes)
-    (property "Reference" "#PWR0141" (id 0) (at 110.49 95.25 0)
+    (property "Reference" "#PWR0167" (id 0) (at 110.49 95.25 0)
       (effects (font (size 1.27 1.27)) hide)
     )
@@
   (symbol (lib_id "power:GND") (at 105.41 144.78 0) (unit 1)
     (in_bom yes) (on_board yes)
-    (property "Reference" "#PWR0140" (id 0) (at 105.41 151.13 0)
+    (property "Reference" "#PWR0166" (id 0) (at 105.41 151.13 0)
       (effects (font (size 1.27 1.27)) hide)
     )
@@
   (symbol (lib_id "power:VCC") (at 172.72 86.36 0) (unit 1)
     (in_bom yes) (on_board yes) (fields_autoplaced)
-    (property "Reference" "#PWR0146" (id 0) (at 172.72 90.17 0)
+    (property "Reference" "#PWR0172" (id 0) (at 172.72 90.17 0)
       (effects (font (size 1.27 1.27)) hide)
     )
@@
   (symbol (lib_id "74xx:74LS173") (at 195.58 86.36 270) (unit 1)
     (in_bom yes) (on_board yes)
-    (property "Reference" "U45" (id 0) (at 189.865 92.71 90))
+    (property "Reference" "U47" (id 0) (at 189.865 92.71 90))
     (property "Value" "74LS173" (id 1) (at 182.88 92.71 90))
     (property "Footprint" "" (id 2) (at 195.58 86.36 0)
@@
   (symbol (lib_id "power:VCC") (at 80.01 86.36 0) (unit 1)
     (in_bom yes) (on_board yes) (fields_autoplaced)
-    (property "Reference" "#PWR0139" (id 0) (at 80.01 90.17 0)
+    (property "Reference" "#PWR0165" (id 0) (at 80.01 90.17 0)
       (effects (font (size 1.27 1.27)) hide)
     )
@@
   (symbol (lib_id "power:VCC") (at 263.525 20.955 0) (unit 1)
     (in_bom yes) (on_board yes)
-    (property "Reference" "#PWR0149" (id 0) (at 263.525 24.765 0)
+    (property "Reference" "#PWR0175" (id 0) (at 263.525 24.765 0)
       (effects (font (size 1.27 1.27)) hide)
     )
@@
   (symbol (lib_id "power:GND") (at 169.545 86.36 0) (unit 1)
     (in_bom yes) (on_board yes) (fields_autoplaced)
-    (property "Reference" "#PWR0145" (id 0) (at 169.545 92.71 0)
+    (property "Reference" "#PWR0171" (id 0) (at 169.545 92.71 0)
       (effects (font (size 1.27 1.27)) hide)
     )
@@
   (symbol (lib_id "74xx:74HC245") (at 100.33 86.36 90) (unit 1)
     (in_bom yes) (on_board yes)
-    (property "Reference" "U43" (id 0) (at 108.585 75.565 90))
+    (property "Reference" "U45" (id 0) (at 108.585 75.565 90))
     (property "Value" "74HC245" (id 1) (at 111.76 77.47 90))
     (property "Footprint" "" (id 2) (at 100.33 86.36 0)
@@
   (symbol (lib_id "power:GND") (at 263.525 33.655 0) (unit 1)
     (in_bom yes) (on_board yes)
-    (property "Reference" "#PWR0150" (id 0) (at 263.525 40.005 0)
+    (property "Reference" "#PWR0176" (id 0) (at 263.525 40.005 0)
       (effects (font (size 1.27 1.27)) hide)
     )
@@
   (symbol (lib_id "power:GND") (at 198.12 73.66 180) (unit 1)
     (in_bom yes) (on_board yes)
-    (property "Reference" "#PWR0147" (id 0) (at 198.12 67.31 0)
+    (property "Reference" "#PWR0173" (id 0) (at 198.12 67.31 0)
       (effects (font (size 1.27 1.27)) hide)
     )
@@
   (symbol (lib_id "power:GND") (at 149.225 73.66 180) (unit 1)
     (in_bom yes) (on_board yes)
-    (property "Reference" "#PWR0144" (id 0) (at 149.225 67.31 0)
+    (property "Reference" "#PWR0170" (id 0) (at 149.225 67.31 0)
       (effects (font (size 1.27 1.27)) hide)
     )
@@
   (symbol (lib_id "74xx:74LS173") (at 146.685 86.36 270) (unit 1)
     (in_bom yes) (on_board yes)
-    (property "Reference" "U44" (id 0) (at 140.97 92.71 90))
+    (property "Reference" "U46" (id 0) (at 140.97 92.71 90))
     (property "Value" "74LS173" (id 1) (at 133.985 92.71 90))
     (property "Footprint" "" (id 2) (at 146.685 86.36 0)
@@
   )
   (symbol (lib_id "power:VCC") (at 123.825 86.36 0) (unit 1)
-    (in_bom yes) (on_board yes) (fields_autoplaced)
-    (property "Reference" "#PWR0143" (id 0) (at 123.825 90.17 0)
+    (in_bom yes) (on_board yes)
+    (property "Reference" "#PWR0169" (id 0) (at 123.825 90.17 0)
       (effects (font (size 1.27 1.27)) hide)
     )
@@
   (symbol (lib_id "power:GND") (at 120.65 86.36 0) (unit 1)
     (in_bom yes) (on_board yes) (fields_autoplaced)
-    (property "Reference" "#PWR0142" (id 0) (at 120.65 92.71 0)
-      (effects (font (size 1.27 1.27)) hide)
-    )
+    (property "Reference" "#PWR0168" (id 0) (at 120.65 92.71 0)
+      (effects (font (size 1.27 1.27)) hide)
+    )

Commit message: complete redraw to bus system
Connections:
- net BUS_0 renamed D0
- net BUS_1 renamed D1
- net BUS_2 renamed D2
- net BUS_3 renamed D3
- net BUS_4 renamed D4
- net BUS_5 renamed D5
- net BUS_6 renamed D6
- net BUS_7 renamed D7
Changed lines of the file:
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@@
     (stroke (width 0) (type default) (color 0 0 0 0))
   )
-  (hierarchical_label "BUS_3" (shape bidirectional) (at 46.99 38.1 180)
-    (effects (font (size 1.524 1.524)) (justify right))
-  )
-  (hierarchical_label "BUS_7" (shape bidirectional) (at 46.99 48.26 180)
+  (hierarchical_label "D6" (shape tri_state) (at 46.99 45.72 180)
     (effects (font (size 1.524 1.524)) (justify right))
   )
@@
     (effects (font (size 1.524 1.524)) (justify left))
   )
-  (hierarchical_label "BUS_5" (shape bidirectional) (at 46.99 43.18 180)
+  (hierarchical_label "D4" (shape tri_state) (at 46.99 40.64 180)
     (effects (font (size 1.524 1.524)) (justify right))
   )
-  (hierarchical_label "BUS_4" (shape bidirectional) (at 46.99 40.64 180)
+  (hierarchical_label "D1" (shape tri_state) (at 46.99 33.02 180)
     (effects (font (size 1.524 1.524)) (justify right))
   )
-  (hierarchical_label "BUS_1" (shape bidirectional) (at 46.99 33.02 180)
+  (hierarchical_label "D3" (shape tri_state) (at 46.99 38.1 180)
     (effects (font (size 1.524 1.524)) (justify right))
   )
-  (hierarchical_label "BUS_0" (shape bidirectional) (at 46.99 30.48 180)
+  (hierarchical_label "D7" (shape tri_state) (at 46.99 48.26 180)
     (effects (font (size 1.524 1.524)) (justify right))
   )
-  (hierarchical_label "BUS_2" (shape bidirectional) (at 46.99 35.56 180)
+  (hierarchical_label "D0" (shape tri_state) (at 46.99 30.48 180)
     (effects (font (size 1.524 1.524)) (justify right))
   )
-  (hierarchical_label "BUS_6" (shape bidirectional) (at 46.99 45.72 180)
+  (hierarchical_label "D2" (shape tri_state) (at 46.99 35.56 180)
     (effects (font (size 1.524 1.524)) (justify right))
   )
+  (hierarchical_label "D5" (shape tri_state) (at 46.99 43.18 180)
+    (effects (font (size 1.524 1.524)) (justify right))
+  )
