File: Kicad Files/y-register.kicad_sch (KiCad schematic)
At the start: 20 parts

Commit message: finished todo list
Changed lines of the file:
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@@
     (stroke (width 0) (type default) (color 0 0 0 0))
   )
-  (wire (pts (xy 204.47 50.8) (xy 217.17 50.8))
+  (wire (pts (xy 168.91 55.88) (xy 217.17 55.88))
     (stroke (width 0) (type default) (color 0 0 0 0))
   )
@@
     (stroke (width 0) (type default) (color 0 0 0 0))
   )
+  (wire (pts (xy 208.28 60.96) (xy 208.28 106.68))
+    (stroke (width 0) (type default) (color 0 0 0 0))
+  )
   (wire (pts (xy 189.23 30.48) (xy 189.23 63.5))
     (stroke (width 0) (type default) (color 0 0 0 0))
@@
     (stroke (width 0) (type default) (color 0 0 0 0))
   )
-  (wire (pts (xy 168.91 55.88) (xy 204.47 55.88))
-    (stroke (width 0) (type default) (color 0 0 0 0))
-  )
   (wire (pts (xy 153.67 170.18) (xy 153.67 173.99))
     (stroke (width 0) (type default) (color 0 0 0 0))
@@
     (stroke (width 0) (type default) (color 0 0 0 0))
   )
-  (wire (pts (xy 113.03 106.68) (xy 217.17 106.68))
+  (wire (pts (xy 113.03 106.68) (xy 208.28 106.68))
     (stroke (width 0) (type default) (color 0 0 0 0))
   )
@@
     (stroke (width 0) (type default) (color 0 0 0 0))
   )
-  (wire (pts (xy 204.47 55.88) (xy 204.47 50.8))
-    (stroke (width 0) (type default) (color 0 0 0 0))
-  )
   (wire (pts (xy 138.43 58.42) (xy 176.53 58.42))
     (stroke (width 0) (type default) (color 0 0 0 0))
@@
   )
   (wire (pts (xy 102.87 33.02) (xy 102.87 63.5))
+    (stroke (width 0) (type default) (color 0 0 0 0))
+  )
+  (wire (pts (xy 217.17 60.96) (xy 208.28 60.96))
     (stroke (width 0) (type default) (color 0 0 0 0))
   )
@@
     (effects (font (size 1.524 1.524)) (justify left))
   )
-  (hierarchical_label "~{YO}" (shape input) (at 217.17 106.68 0)
+  (hierarchical_label "~{YO}" (shape input) (at 217.17 60.96 0)
     (effects (font (size 1.524 1.524)) (justify left))
   )
@@
     (effects (font (size 1.524 1.524)) (justify right))
   )
-  (hierarchical_label "CLR" (shape input) (at 217.17 50.8 0)
+  (hierarchical_label "CLR" (shape input) (at 217.17 55.88 0)
     (effects (font (size 1.524 1.524)) (justify left))
   )

Commit message: fixed erc
Parts:
- gave numbers to parts that had none: 20
Changed lines of the file:
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@@
   (symbol (lib_id "8bit-computer-rescue:74LS173-8bit-computer-rescue") (at 182.88 81.28 270) (unit 1)
     (in_bom yes) (on_board yes)
-    (property "Reference" "U?" (id 0) (at 185.42 83.82 0))
+    (property "Reference" "U3" (id 0) (at 185.42 83.82 0))
     (property "Value" "74LS173" (id 1) (at 181.61 83.82 0))
     (property "Footprint" "Package_DIP:DIP-16_W7.62mm" (id 2) (at 182.88 81.28 0)
@@
   (symbol (lib_id "8bit-computer-rescue:LED_ALT-Device") (at 115.57 154.94 90) (unit 1)
     (in_bom yes) (on_board yes)
-    (property "Reference" "D?" (id 0) (at 113.03 154.94 0))
+    (property "Reference" "D26" (id 0) (at 113.03 154.94 0))
     (property "Value" "RED" (id 1) (at 118.11 154.94 0))
     (property "Footprint" "LED_THT:LED_D5.0mm" (id 2) (at 115.57 154.94 0)
@@
   (symbol (lib_id "Device:R") (at 123.19 166.37 0) (unit 1)
     (in_bom yes) (on_board yes)
-    (property "Reference" "R?" (id 0) (at 125.222 166.37 90))
+    (property "Reference" "R27" (id 0) (at 125.222 166.37 90))
     (property "Value" "R" (id 1) (at 123.19 166.37 90))
     (property "Footprint" "Resistor_THT:R_Axial_DIN0207_L6.3mm_D2.5mm_P7.62mm_Horizontal" (id 2) (at 121.412 166.37 90)
@@
   (symbol (lib_id "Device:C") (at 240.03 80.01 0) (unit 1)
     (in_bom yes) (on_board yes)
-    (property "Reference" "C?" (id 0) (at 240.665 77.47 0)
+    (property "Reference" "C2" (id 0) (at 240.665 77.47 0)
       (effects (font (size 1.27 1.27)) (justify left))
     )
@@
   (symbol (lib_id "8bit-computer-rescue:LED_ALT-Device") (at 153.67 154.94 90) (unit 1)
     (in_bom yes) (on_board yes)
-    (property "Reference" "D?" (id 0) (at 151.13 154.94 0))
+    (property "Reference" "D31" (id 0) (at 151.13 154.94 0))
     (property "Value" "RED" (id 1) (at 156.21 154.94 0))
     (property "Footprint" "LED_THT:LED_D5.0mm" (id 2) (at 153.67 154.94 0)
@@
   (symbol (lib_id "8bit-computer-rescue:LED_ALT-Device") (at 107.95 154.94 90) (unit 1)
     (in_bom yes) (on_board yes)
-    (property "Reference" "D?" (id 0) (at 105.41 154.94 0))
+    (property "Reference" "D25" (id 0) (at 105.41 154.94 0))
     (property "Value" "RED" (id 1) (at 110.49 154.94 0))
     (property "Footprint" "LED_THT:LED_D5.0mm" (id 2) (at 107.95 154.94 0)
@@
   (symbol (lib_id "8bit-computer-rescue:74LS173-8bit-computer-rescue") (at 142.24 81.28 270) (unit 1)
     (in_bom yes) (on_board yes)
-    (property "Reference" "U?" (id 0) (at 144.78 83.82 0))
+    (property "Reference" "U2" (id 0) (at 144.78 83.82 0))
     (property "Value" "74LS173" (id 1) (at 140.97 83.82 0))
     (property "Footprint" "Package_DIP:DIP-16_W7.62mm" (id 2) (at 142.24 81.28 0)
@@
   (symbol (lib_id "8bit-computer-rescue:LED_ALT-Device") (at 146.05 154.94 90) (unit 1)
     (in_bom yes) (on_board yes)
-    (property "Reference" "D?" (id 0) (at 143.51 154.94 0))
+    (property "Reference" "D30" (id 0) (at 143.51 154.94 0))
     (property "Value" "RED" (id 1) (at 148.59 154.94 0))
     (property "Footprint" "LED_THT:LED_D5.0mm" (id 2) (at 146.05 154.94 0)
@@
   (symbol (lib_id "power:GND") (at 134.62 179.07 0) (unit 1)
     (in_bom yes) (on_board yes)
-    (property "Reference" "#PWR?" (id 0) (at 134.62 185.42 0)
+    (property "Reference" "#PWR05" (id 0) (at 134.62 185.42 0)
       (effects (font (size 1.27 1.27)) hide)
     )
@@
   (symbol (lib_id "power:VCC") (at 110.49 99.06 180) (unit 1)
     (in_bom yes) (on_board yes)
-    (property "Reference" "#PWR?" (id 0) (at 110.49 95.25 0)
+    (property "Reference" "#PWR04" (id 0) (at 110.49 95.25 0)
       (effects (font (size 1.27 1.27)) hide)
     )
@@
   (symbol (lib_id "8bit-computer-rescue:LED_ALT-Device") (at 138.43 154.94 90) (unit 1)
     (in_bom yes) (on_board yes)
-    (property "Reference" "D?" (id 0) (at 135.89 154.94 0))
+    (property "Reference" "D29" (id 0) (at 135.89 154.94 0))
     (property "Value" "RED" (id 1) (at 140.97 154.94 0))
     (property "Footprint" "LED_THT:LED_D5.0mm" (id 2) (at 138.43 154.94 0)
@@
   (symbol (lib_id "8bit-computer-rescue:LED_ALT-Device") (at 161.29 154.94 90) (unit 1)
     (in_bom yes) (on_board yes)
-    (property "Reference" "D?" (id 0) (at 158.75 154.94 0))
+    (property "Reference" "D32" (id 0) (at 158.75 154.94 0))
     (property "Value" "RED" (id 1) (at 163.83 154.94 0))
     (property "Footprint" "LED_THT:LED_D5.0mm" (id 2) (at 161.29 154.94 0)
@@
   (symbol (lib_id "8bit-computer-rescue:LED_ALT-Device") (at 123.19 154.94 90) (unit 1)
     (in_bom yes) (on_board yes)
-    (property "Reference" "D?" (id 0) (at 120.65 154.94 0))
+    (property "Reference" "D27" (id 0) (at 120.65 154.94 0))
     (property "Value" "RED" (id 1) (at 125.73 154.94 0))
     (property "Footprint" "LED_THT:LED_D5.0mm" (id 2) (at 123.19 154.94 0)
@@
   (symbol (lib_id "8bit-computer-rescue:LED_ALT-Device") (at 130.81 154.94 90) (unit 1)
     (in_bom yes) (on_board yes)
-    (property "Reference" "D?" (id 0) (at 128.27 154.94 0))
+    (property "Reference" "D28" (id 0) (at 128.27 154.94 0))
     (property "Value" "RED" (id 1) (at 133.35 154.94 0))
     (property "Footprint" "LED_THT:LED_D5.0mm" (id 2) (at 130.81 154.94 0)
@@
   (symbol (lib_id "Device:R") (at 161.29 166.37 0) (unit 1)
     (in_bom yes) (on_board yes)
-    (property "Reference" "R?" (id 0) (at 163.322 166.37 90))
+    (property "Reference" "R32" (id 0) (at 163.322 166.37 90))
     (property "Value" "R" (id 1) (at 161.29 166.37 90))
     (property "Footprint" "Resistor_THT:R_Axial_DIN0207_L6.3mm_D2.5mm_P7.62mm_Horizontal" (id 2) (at 159.512 166.37 90)
@@
   (symbol (lib_id "8bit-computer-rescue:74LS245-8bit-computer-rescue") (at 100.33 81.28 90) (unit 1)
     (in_bom yes) (on_board yes)
-    (property "Reference" "U?" (id 0) (at 85.725 78.74 0)
+    (property "Reference" "U1" (id 0) (at 85.725 78.74 0)
       (effects (font (size 1.27 1.27)) (justify left bottom))
     )
@@
   (symbol (lib_id "Device:R") (at 146.05 166.37 0) (unit 1)
     (in_bom yes) (on_board yes)
-    (property "Reference" "R?" (id 0) (at 148.082 166.37 90))
+    (property "Reference" "R30" (id 0) (at 148.082 166.37 90))
     (property "Value" "R" (id 1) (at 146.05 166.37 90))
     (property "Footprint" "Resistor_THT:R_Axial_DIN0207_L6.3mm_D2.5mm_P7.62mm_Horizontal" (id 2) (at 144.272 166.37 90)
@@
   (symbol (lib_id "power:VCC") (at 240.03 73.66 0) (unit 1)
     (in_bom yes) (on_board yes)
-    (property "Reference" "#PWR?" (id 0) (at 240.03 77.47 0)
+    (property "Reference" "#PWR07" (id 0) (at 240.03 77.47 0)
       (effects (font (size 1.27 1.27)) hide)
     )
@@
   (symbol (lib_id "power:GND") (at 204.47 68.58 0) (unit 1)
     (in_bom yes) (on_board yes)
-    (property "Reference" "#PWR?" (id 0) (at 204.47 74.93 0)
+    (property "Reference" "#PWR06" (id 0) (at 204.47 74.93 0)
       (effects (font (size 1.27 1.27)) hide)
     )
@@
   (symbol (lib_id "Device:R") (at 138.43 166.37 0) (unit 1)
     (in_bom yes) (on_board yes)
-    (property "Reference" "R?" (id 0) (at 140.462 166.37 90))
+    (property "Reference" "R29" (id 0) (at 140.462 166.37 90))
     (property "Value" "R" (id 1) (at 138.43 166.37 90))
     (property "Footprint" "Resistor_THT:R_Axial_DIN0207_L6.3mm_D2.5mm_P7.62mm_Horizontal" (id 2) (at 136.652 166.37 90)
@@
   (symbol (lib_id "Device:R") (at 153.67 166.37 0) (unit 1)
     (in_bom yes) (on_board yes)
-    (property "Reference" "R?" (id 0) (at 155.702 166.37 90))
+    (property "Reference" "R31" (id 0) (at 155.702 166.37 90))
     (property "Value" "R" (id 1) (at 153.67 166.37 90))
     (property "Footprint" "Resistor_THT:R_Axial_DIN0207_L6.3mm_D2.5mm_P7.62mm_Horizontal" (id 2) (at 151.892 166.37 90)
@@
   (symbol (lib_id "Device:R") (at 130.81 166.37 0) (unit 1)
     (in_bom yes) (on_board yes)
-    (property "Reference" "R?" (id 0) (at 132.842 166.37 90))
+    (property "Reference" "R28" (id 0) (at 132.842 166.37 90))
     (property "Value" "R" (id 1) (at 130.81 166.37 90))
     (property "Footprint" "Resistor_THT:R_Axial_DIN0207_L6.3mm_D2.5mm_P7.62mm_Horizontal" (id 2) (at 129.032 166.37 90)
@@
   (symbol (lib_id "power:GND") (at 240.03 86.36 0) (unit 1)
     (in_bom yes) (on_board yes)
-    (property "Reference" "#PWR?" (id 0) (at 240.03 92.71 0)
+    (property "Reference" "#PWR08" (id 0) (at 240.03 92.71 0)
       (effects (font (size 1.27 1.27)) hide)
     )
@@
   (symbol (lib_id "Device:R") (at 107.95 166.37 0) (unit 1)
     (in_bom yes) (on_board yes)
-    (property "Reference" "R?" (id 0) (at 109.982 166.37 90))
+    (property "Reference" "R25" (id 0) (at 109.982 166.37 90))
     (property "Value" "R" (id 1) (at 107.95 166.37 90))
     (property "Footprint" "Resistor_THT:R_Axial_DIN0207_L6.3mm_D2.5mm_P7.62mm_Horizontal" (id 2) (at 106.172 166.37 90)
@@
   (symbol (lib_id "Device:R") (at 115.57 166.37 0) (unit 1)
     (in_bom yes) (on_board yes)
-    (property "Reference" "R?" (id 0) (at 117.602 166.37 90))
+    (property "Reference" "R26" (id 0) (at 117.602 166.37 90))
     (property "Value" "R" (id 1) (at 115.57 166.37 90))
     (property "Footprint" "Resistor_THT:R_Axial_DIN0207_L6.3mm_D2.5mm_P7.62mm_Horizontal" (id 2) (at 113.792 166.37 90)
