File: Kicad Files/program-counter.kicad_sch (KiCad schematic)
At the start: 20 parts

Commit message: started tidy up in control
Parts:
- gave numbers to parts that had none: 20
Changed lines of the file:
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@@
   (symbol (lib_id "Device:C") (at 223.52 58.42 0) (unit 1)
     (in_bom yes) (on_board yes)
-    (property "Reference" "" (id 0) (at 224.155 55.88 0)
+    (property "Reference" "C10" (id 0) (at 224.155 55.88 0)
       (effects (font (size 1.27 1.27)) (justify left))
     )
@@
   (symbol (lib_id "8bit-computer-rescue:LED_ALT-Device") (at 160.02 109.22 90) (unit 1)
     (in_bom yes) (on_board yes)
-    (property "Reference" "" (id 0) (at 157.48 109.22 0))
+    (property "Reference" "D72" (id 0) (at 157.48 109.22 0))
     (property "Value" "GREEN" (id 1) (at 162.56 109.22 0))
     (property "Footprint" "LED_THT:LED_D5.0mm" (id 2) (at 160.02 109.22 0)
@@
   (symbol (lib_id "8bit-computer-rescue:LED_ALT-Device") (at 154.94 109.22 90) (unit 1)
     (in_bom yes) (on_board yes)
-    (property "Reference" "" (id 0) (at 152.4 109.22 0))
+    (property "Reference" "D71" (id 0) (at 152.4 109.22 0))
     (property "Value" "GREEN" (id 1) (at 157.48 109.22 0))
     (property "Footprint" "LED_THT:LED_D5.0mm" (id 2) (at 154.94 109.22 0)
@@
   (symbol (lib_id "8bit-computer-rescue:LED_ALT-Device") (at 149.86 109.22 90) (unit 1)
     (in_bom yes) (on_board yes)
-    (property "Reference" "" (id 0) (at 147.32 109.22 0))
+    (property "Reference" "D70" (id 0) (at 147.32 109.22 0))
     (property "Value" "GREEN" (id 1) (at 152.4 109.22 0))
     (property "Footprint" "LED_THT:LED_D5.0mm" (id 2) (at 149.86 109.22 0)
@@
   (symbol (lib_id "8bit-computer-rescue:LED_ALT-Device") (at 144.78 109.22 90) (unit 1)
     (in_bom yes) (on_board yes)
-    (property "Reference" "" (id 0) (at 142.24 109.22 0))
+    (property "Reference" "D69" (id 0) (at 142.24 109.22 0))
     (property "Value" "GREEN" (id 1) (at 147.32 109.22 0))
     (property "Footprint" "LED_THT:LED_D5.0mm" (id 2) (at 144.78 109.22 0)
@@
   (symbol (lib_id "Device:R") (at 160.02 119.38 180) (unit 1)
     (in_bom yes) (on_board yes)
-    (property "Reference" "" (id 0) (at 157.988 119.38 90))
+    (property "Reference" "R84" (id 0) (at 157.988 119.38 90))
     (property "Value" "220" (id 1) (at 160.02 119.38 90))
     (property "Footprint" "Resistor_THT:R_Axial_DIN0207_L6.3mm_D2.5mm_P7.62mm_Horizontal" (id 2) (at 161.798 119.38 90)
@@
   (symbol (lib_id "Device:R") (at 154.94 119.38 180) (unit 1)
     (in_bom yes) (on_board yes)
-    (property "Reference" "" (id 0) (at 152.908 119.38 90))
+    (property "Reference" "R83" (id 0) (at 152.908 119.38 90))
     (property "Value" "220" (id 1) (at 154.94 119.38 90))
     (property "Footprint" "Resistor_THT:R_Axial_DIN0207_L6.3mm_D2.5mm_P7.62mm_Horizontal" (id 2) (at 156.718 119.38 90)
@@
   (symbol (lib_id "Device:R") (at 149.86 119.38 180) (unit 1)
     (in_bom yes) (on_board yes)
-    (property "Reference" "" (id 0) (at 147.828 119.38 90))
+    (property "Reference" "R82" (id 0) (at 147.828 119.38 90))
     (property "Value" "220" (id 1) (at 149.86 119.38 90))
     (property "Footprint" "Resistor_THT:R_Axial_DIN0207_L6.3mm_D2.5mm_P7.62mm_Horizontal" (id 2) (at 151.638 119.38 90)
@@
   (symbol (lib_id "Device:R") (at 144.78 119.38 180) (unit 1)
     (in_bom yes) (on_board yes)
-    (property "Reference" "" (id 0) (at 142.748 119.38 90))
+    (property "Reference" "R81" (id 0) (at 142.748 119.38 90))
     (property "Value" "220" (id 1) (at 144.78 119.38 90))
     (property "Footprint" "Resistor_THT:R_Axial_DIN0207_L6.3mm_D2.5mm_P7.62mm_Horizontal" (id 2) (at 146.558 119.38 90)
@@
   (symbol (lib_id "74xx:74LS245") (at 203.2 90.17 0) (unit 1)
     (in_bom yes) (on_board yes)
-    (property "Reference" "" (id 0) (at 203.2 85.09 0))
+    (property "Reference" "U39" (id 0) (at 203.2 85.09 0))
     (property "Value" "74LS245" (id 1) (at 209.55 100.33 90))
     (property "Footprint" "" (id 2) (at 203.2 90.17 0)
@@
   (symbol (lib_id "74xx:74LS161") (at 114.3 64.77 0) (unit 1)
     (in_bom yes) (on_board yes)
-    (property "Reference" "" (id 0) (at 120.65 68.58 90))
+    (property "Reference" "U38" (id 0) (at 120.65 68.58 90))
     (property "Value" "74LS161" (id 1) (at 120.65 74.93 90))
     (property "Footprint" "" (id 2) (at 114.3 64.77 0)
@@
   (symbol (lib_id "74xx:74LS161") (at 114.3 107.95 0) (unit 1)
     (in_bom yes) (on_board yes)
-    (property "Reference" "" (id 0) (at 120.65 111.76 90))
+    (property "Reference" "U40" (id 0) (at 120.65 111.76 90))
     (property "Value" "74LS161" (id 1) (at 120.65 118.11 90))
     (property "Footprint" "" (id 2) (at 114.3 107.95 0)
@@
   (symbol (lib_id "8bit-computer-rescue:LED_ALT-Device") (at 180.34 109.22 90) (unit 1)
     (in_bom yes) (on_board yes)
-    (property "Reference" "" (id 0) (at 177.8 109.22 0))
+    (property "Reference" "D76" (id 0) (at 177.8 109.22 0))
     (property "Value" "GREEN" (id 1) (at 182.88 109.22 0))
     (property "Footprint" "LED_THT:LED_D5.0mm" (id 2) (at 180.34 109.22 0)
@@
   (symbol (lib_id "8bit-computer-rescue:LED_ALT-Device") (at 175.26 109.22 90) (unit 1)
     (in_bom yes) (on_board yes)
-    (property "Reference" "" (id 0) (at 172.72 109.22 0))
+    (property "Reference" "D75" (id 0) (at 172.72 109.22 0))
     (property "Value" "GREEN" (id 1) (at 177.8 109.22 0))
     (property "Footprint" "LED_THT:LED_D5.0mm" (id 2) (at 175.26 109.22 0)
@@
   (symbol (lib_id "8bit-computer-rescue:LED_ALT-Device") (at 170.18 109.22 90) (unit 1)
     (in_bom yes) (on_board yes)
-    (property "Reference" "" (id 0) (at 167.64 109.22 0))
+    (property "Reference" "D74" (id 0) (at 167.64 109.22 0))
     (property "Value" "GREEN" (id 1) (at 172.72 109.22 0))
     (property "Footprint" "LED_THT:LED_D5.0mm" (id 2) (at 170.18 109.22 0)
@@
   (symbol (lib_id "8bit-computer-rescue:LED_ALT-Device") (at 165.1 109.22 90) (unit 1)
     (in_bom yes) (on_board yes)
-    (property "Reference" "" (id 0) (at 162.56 109.22 0))
+    (property "Reference" "D73" (id 0) (at 162.56 109.22 0))
     (property "Value" "GREEN" (id 1) (at 167.64 109.22 0))
     (property "Footprint" "LED_THT:LED_D5.0mm" (id 2) (at 165.1 109.22 0)
@@
   (symbol (lib_id "Device:R") (at 180.34 119.38 180) (unit 1)
     (in_bom yes) (on_board yes)
-    (property "Reference" "" (id 0) (at 178.308 119.38 90))
+    (property "Reference" "R88" (id 0) (at 178.308 119.38 90))
     (property "Value" "220" (id 1) (at 180.34 119.38 90))
     (property "Footprint" "Resistor_THT:R_Axial_DIN0207_L6.3mm_D2.5mm_P7.62mm_Horizontal" (id 2) (at 182.118 119.38 90)
@@
   (symbol (lib_id "Device:R") (at 175.26 119.38 180) (unit 1)
     (in_bom yes) (on_board yes)
-    (property "Reference" "" (id 0) (at 173.228 119.38 90))
+    (property "Reference" "R87" (id 0) (at 173.228 119.38 90))
     (property "Value" "220" (id 1) (at 175.26 119.38 90))
     (property "Footprint" "Resistor_THT:R_Axial_DIN0207_L6.3mm_D2.5mm_P7.62mm_Horizontal" (id 2) (at 177.038 119.38 90)
@@
   (symbol (lib_id "Device:R") (at 170.18 119.38 180) (unit 1)
     (in_bom yes) (on_board yes)
-    (property "Reference" "" (id 0) (at 168.148 119.38 90))
+    (property "Reference" "R86" (id 0) (at 168.148 119.38 90))
     (property "Value" "220" (id 1) (at 170.18 119.38 90))
     (property "Footprint" "Resistor_THT:R_Axial_DIN0207_L6.3mm_D2.5mm_P7.62mm_Horizontal" (id 2) (at 171.958 119.38 90)
@@
   (symbol (lib_id "Device:R") (at 165.1 119.38 180) (unit 1)
     (in_bom yes) (on_board yes)
-    (property "Reference" "" (id 0) (at 163.068 119.38 90))
+    (property "Reference" "R85" (id 0) (at 163.068 119.38 90))
     (property "Value" "220" (id 1) (at 165.1 119.38 90))
     (property "Footprint" "Resistor_THT:R_Axial_DIN0207_L6.3mm_D2.5mm_P7.62mm_Horizontal" (id 2) (at 166.878 119.38 90)

Commit message: work on cl
Parts:
- C14: renamed from C10; value 0.1µF -> C
- R63: renamed from R81; value 220 -> R
- R64: renamed from R82; value 220 -> R
- R65: renamed from R83; value 220 -> R
- R66: renamed from R84; value 220 -> R
- R67: renamed from R85; value 220 -> R
- R68: renamed from R86; value 220 -> R
- R69: renamed from R87; value 220 -> R
- R70: renamed from R88; value 220 -> R
- renumbered D69 to D32, D70 to D33, D71 to D34, D72 to D35, D73 to D36, D74 to D37, D75 to D38, D76 to D39, U38 to U23, U40 to U24, U39 to U25

Commit message: w2
Parts:
- removed D32, D33, D34, D35, D36, D37, D38, D39: GREEN, LED_THT:LED_D5.0mm, symbol 8bit-computer-rescue:LED_ALT-Device
- removed R63, R64, R65, R66, R67, R68, R69, R70: R, Resistor_THT:R_Axial_DIN0207_L6.3mm_D2.5mm_P7.62mm_Horizontal, symbol Device:R
- added U? (x2): 74LS161, symbol 74xx:74LS161
- added U?: 74LS245, symbol 74xx:74LS245
Connections:
- net BUS_0: now also U?.18 (B0), U?.3 (D0)
- net BUS_1: now also U?.17 (B1), U?.4 (D1)
- net BUS_2: now also U?.16 (B2), U?.5 (D2)
- net BUS_3: now also U?.15 (B3), U?.6 (D3)
- net BUS_4: now also U?.14 (B4), U?.3 (D0)
- net BUS_5: now also U?.13 (B5), U?.4 (D1)
- net BUS_6: now also U?.12 (B6), U?.5 (D2)
- net BUS_7: now also U?.11 (B7), U?.6 (D3)
- net CE: now also U?.10 (CET), U?.7 (CEP), U?.7 (CEP); no longer U23.10 (CET)
- net CLK: now also U?.2 (CP), U?.2 (CP)
- net GND: now also U?.10 (GND), U?.8 (GND), U?.8 (GND)
- net VCC: now also U?.1 (A->B), U?.16 (VCC), U?.16 (VCC), U?.20 (VCC)
- net ~{CLR}: now also U?.1 (~{MR}), U?.1 (~{MR})
- net ~{CO}: now also U?.19 (CE)
- net ~{J}: now also U?.9 (~{PE}), U?.9 (~{PE})
- new net: U23.10 (CET), U?.15 (TC)
- new net: U?.10 (CET), U?.15 (TC)
- new net: U?.11 (Q3), U?.9 (A7)
- new net: U?.12 (Q2), U?.8 (A6)
- new net: U?.13 (Q1), U?.7 (A5)
- new net: U?.14 (Q0), U?.6 (A4)
- new net: U?.11 (Q3), U?.5 (A3)
- new net: U?.12 (Q2), U?.4 (A2)
- new net: U?.13 (Q1), U?.3 (A1)
- new net: U?.14 (Q0), U?.2 (A0)
Other:
- moved on the sheet: C14, U23, U24, U25

Commit message: work on PC
Connections:
- net ~{CO} renamed ~{COhB}
- net ~{COhB}: no longer U25.19 (CE)
- net ~{J} renamed ~{JhB}
- net ~{JhB}: no longer U23.9 (~{PE}), U24.9 (~{PE})
- new net ~{COlB}: U25.19 (CE)
- new net ~{JlB}: U23.9 (~{PE}), U24.9 (~{PE})
Changed lines of the file:
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@@
   (junction (at 55.88 152.4) (diameter 0) (color 0 0 0 0)
   )
+  (junction (at 50.8 142.24) (diameter 0) (color 0 0 0 0)
+  )
+  (junction (at 172.72 160.02) (diameter 0) (color 0 0 0 0)
+  )
+  (junction (at 162.56 170.18) (diameter 0) (color 0 0 0 0)
+  )
+  (junction (at 30.48 129.54) (diameter 0) (color 0 0 0 0)
+  )
+  (junction (at 53.34 53.34) (diameter 0) (color 0 0 0 0)
+  )
+  (junction (at 58.42 147.32) (diameter 0) (color 0 0 0 0)
+  )
+  (junction (at 58.42 104.14) (diameter 0) (color 0 0 0 0)
+  )
+  (junction (at 55.88 109.22) (diameter 0) (color 0 0 0 0)
+  )
+  (junction (at 38.1 170.18) (diameter 0) (color 0 0 0 0)
+  )
+  (junction (at 157.48 175.26) (diameter 0) (color 0 0 0 0)
+  )
+  (junction (at 160.02 172.72) (diameter 0) (color 0 0 0 0)
+  )
   (junction (at 53.34 139.7) (diameter 0) (color 0 0 0 0)
-  )
-  (junction (at 50.8 142.24) (diameter 0) (color 0 0 0 0)
-  )
-  (junction (at 172.72 160.02) (diameter 0) (color 0 0 0 0)
-  )
-  (junction (at 162.56 170.18) (diameter 0) (color 0 0 0 0)
-  )
-  (junction (at 30.48 129.54) (diameter 0) (color 0 0 0 0)
-  )
-  (junction (at 53.34 53.34) (diameter 0) (color 0 0 0 0)
-  )
-  (junction (at 53.34 96.52) (diameter 0) (color 0 0 0 0)
-  )
-  (junction (at 58.42 147.32) (diameter 0) (color 0 0 0 0)
-  )
-  (junction (at 58.42 104.14) (diameter 0) (color 0 0 0 0)
-  )
-  (junction (at 55.88 109.22) (diameter 0) (color 0 0 0 0)
-  )
-  (junction (at 38.1 170.18) (diameter 0) (color 0 0 0 0)
-  )
-  (junction (at 157.48 175.26) (diameter 0) (color 0 0 0 0)
-  )
-  (junction (at 160.02 172.72) (diameter 0) (color 0 0 0 0)
-  )
-  (junction (at 124.46 99.06) (diameter 0) (color 0 0 0 0)
   )
   (junction (at 27.94 127) (diameter 0) (color 0 0 0 0)
@@
     (stroke (width 0) (type default) (color 0 0 0 0))
   )
-  (wire (pts (xy 53.34 96.52) (xy 53.34 139.7))
-    (stroke (width 0) (type default) (color 0 0 0 0))
-  )
   (wire (pts (xy 62.23 96.52) (xy 53.34 96.52))
     (stroke (width 0) (type default) (color 0 0 0 0))
   )
+  (wire (pts (xy 53.34 101.6) (xy 48.26 101.6))
+    (stroke (width 0) (type default) (color 0 0 0 0))
+  )
   (wire (pts (xy 60.96 74.93) (xy 60.96 101.6))
     (stroke (width 0) (type default) (color 0 0 0 0))
@@
     (stroke (width 0) (type default) (color 0 0 0 0))
   )
+  (wire (pts (xy 53.34 139.7) (xy 53.34 101.6))
+    (stroke (width 0) (type default) (color 0 0 0 0))
+  )
   (wire (pts (xy 30.48 129.54) (xy 30.48 43.18))
     (stroke (width 0) (type default) (color 0 0 0 0))
@@
     (stroke (width 0) (type default) (color 0 0 0 0))
   )
+  (wire (pts (xy 29.21 26.67) (xy 121.92 26.67))
+    (stroke (width 0) (type default) (color 0 0 0 0))
+  )
   (wire (pts (xy 87.63 170.18) (xy 127 170.18))
     (stroke (width 0) (type default) (color 0 0 0 0))
@@
     (stroke (width 0) (type default) (color 0 0 0 0))
   )
-  (wire (pts (xy 127 185.42) (xy 124.46 185.42))
+  (wire (pts (xy 121.92 185.42) (xy 127 185.42))
     (stroke (width 0) (type default) (color 0 0 0 0))
   )
@@
     (stroke (width 0) (type default) (color 0 0 0 0))
   )
-  (wire (pts (xy 124.46 99.06) (xy 124.46 185.42))
-    (stroke (width 0) (type default) (color 0 0 0 0))
-  )
   (wire (pts (xy 113.665 165.1) (xy 127 165.1))
     (stroke (width 0) (type default) (color 0 0 0 0))
@@
     (stroke (width 0) (type default) (color 0 0 0 0))
   )
-  (wire (pts (xy 29.21 26.67) (xy 53.34 26.67))
+  (wire (pts (xy 29.21 29.21) (xy 53.34 29.21))
     (stroke (width 0) (type default) (color 0 0 0 0))
   )
@@
     (stroke (width 0) (type default) (color 0 0 0 0))
   )
+  (wire (pts (xy 29.21 31.75) (xy 48.26 31.75))
+    (stroke (width 0) (type default) (color 0 0 0 0))
+  )
   (wire (pts (xy 62.23 190.5) (xy 58.42 190.5))
     (stroke (width 0) (type default) (color 0 0 0 0))
@@
     (stroke (width 0) (type default) (color 0 0 0 0))
   )
+  (wire (pts (xy 121.92 26.67) (xy 121.92 185.42))
+    (stroke (width 0) (type default) (color 0 0 0 0))
+  )
   (wire (pts (xy 165.1 226.06) (xy 165.1 167.64))
     (stroke (width 0) (type default) (color 0 0 0 0))
@@
     (stroke (width 0) (type default) (color 0 0 0 0))
   )
+  (wire (pts (xy 48.26 101.6) (xy 48.26 31.75))
+    (stroke (width 0) (type default) (color 0 0 0 0))
+  )
   (wire (pts (xy 113.665 132.08) (xy 113.665 165.1))
     (stroke (width 0) (type default) (color 0 0 0 0))
@@
     (stroke (width 0) (type default) (color 0 0 0 0))
   )
-  (wire (pts (xy 53.34 26.67) (xy 53.34 53.34))
+  (wire (pts (xy 53.34 29.21) (xy 53.34 53.34))
     (stroke (width 0) (type default) (color 0 0 0 0))
   )
@@
     (effects (font (size 1.524 1.524)) (justify left))
   )
+  (hierarchical_label "~{JlB}" (shape input) (at 29.21 31.75 180)
+    (effects (font (size 1.524 1.524)) (justify right))
+  )
   (hierarchical_label "BUS_6" (shape bidirectional) (at 179.07 175.26 0)
     (effects (font (size 1.524 1.524)) (justify left))
@@
   (hierarchical_label "BUS_1" (shape bidirectional) (at 179.07 162.56 0)
     (effects (font (size 1.524 1.524)) (justify left))
+  )
+  (hierarchical_label "~{COlB}" (shape input) (at 29.21 26.67 180)
+    (effects (font (size 1.524 1.524)) (justify right))
   )
   (hierarchical_label "CE" (shape input) (at 29.21 21.59 180)
@@
     (effects (font (size 1.524 1.524)) (justify left))
   )
-  (hierarchical_label "~{J}" (shape input) (at 29.21 26.67 180)
+  (hierarchical_label "~{JhB}" (shape input) (at 29.21 29.21 180)
     (effects (font (size 1.524 1.524)) (justify right))
   )
@@
     (effects (font (size 1.524 1.524)) (justify left))
   )
-  (hierarchical_label "~{CO}" (shape input) (at 29.21 24.13 180)
+  (hierarchical_label "~{COhB}" (shape input) (at 29.21 24.13 180)
     (effects (font (size 1.524 1.524)) (justify right))
   )

Commit message: work on pc2
Parts:
- removed U23, U24, U? (x2): 74LS161, symbol 74xx:74LS161
- removed U25, U?: 74LS245, symbol 74xx:74LS245
- added D? (x16): LED, symbol Device:LED
- added R? (x16): R_Small, symbol Device:R_Small
- added U? (x2): 74HC245, symbol 74xx:74HC245
- added U? (x4): 74LS161, symbol 74xx:74LS161
Connections:
- net BUS_0: now also U?.14 (Q0), U?.14 (Q0)
- net BUS_1: now also U?.13 (Q1), U?.13 (Q1)
- net BUS_2: now also U?.12 (Q2), U?.12 (Q2)
- net BUS_3: now also U?.11 (Q3), U?.11 (Q3)
- net BUS_4: now also U?.14 (Q0), U?.14 (Q0)
- net BUS_5: now also U?.13 (Q1), U?.13 (Q1)
- net BUS_6: now also U?.12 (Q2), U?.12 (Q2)
- net BUS_7: now also U?.11 (Q3), U?.11 (Q3)
- net CLK: now also U?.1 (~{MR}), U?.1 (~{MR}), U?.1 (~{MR}), U?.1 (~{MR})
- net GND: now also R?.2, R?.2, R?.2, R?.2, R?.2, R?.2, R?.2, R?.2, R?.2, R?.2, R?.2, R?.2, R?.2, R?.2, R?.2, R?.2, U?.8 (GND), U?.8 (GND), U?.8 (GND), U?.8 (GND)
- net VCC: now also U?.16 (VCC), U?.16 (VCC), U?.16 (VCC), U?.16 (VCC)
- net ~{CLR}: now also U?.2 (CP), U?.2 (CP), U?.2 (CP), U?.2 (CP)
- new net: D?.1 (K), R?.1 (x16)
- new net: D?.2 (A), U?.15 (B3), U?.6 (D3)
- new net: D?.2 (A), U?.5 (D2) (x2)
- new net: D?.2 (A), U?.18 (B0), U?.3 (D0)
- new net: D?.2 (A), U?.6 (D3) (x2)
- new net: D?.2 (A), U?.12 (B6), U?.5 (D2)
- new net: D?.2 (A), U?.3 (D0) (x2)
- new net: D?.2 (A), U?.17 (B1), U?.4 (D1)
- new net: U?.10 (CET), U?.15 (TC) (x3)
- new net: D?.2 (A), U?.4 (D1) (x2)
- new net: D?.2 (A), U?.14 (B4), U?.3 (D0)
- new net: D?.2 (A), U?.13 (B5), U?.4 (D1)
- new net: D?.2 (A), U?.11 (B7), U?.6 (D3)
- new net: D?.2 (A), U?.16 (B2), U?.5 (D2)
- new net ABUS_00: U?.2 (A0)
- new net ABUS_01: U?.3 (A1)
- new net ABUS_02: U?.4 (A2)
- new net ABUS_03: U?.5 (A3)
- new net ABUS_04: U?.6 (A4)
- new net ABUS_05: U?.7 (A5)
- new net ABUS_06: U?.8 (A6)
- new net ABUS_07: U?.9 (A7)
- new net ABUS_08: U?.2 (A0)
- new net ABUS_09: U?.3 (A1)
- new net ABUS_10: U?.4 (A2)
- new net ABUS_11: U?.5 (A3)
- new net ABUS_12: U?.6 (A4)
- new net ABUS_13: U?.7 (A5)
- new net ABUS_14: U?.8 (A6)
- new net ABUS_15: U?.9 (A7)
- new net CEhb: U?.10 (CET), U?.7 (CEP), U?.7 (CEP)
- new net CElb: U?.7 (CEP), U?.7 (CEP)
- new net ~{Jhb}: U?.9 (~{PE}), U?.9 (~{PE})
- new net ~{Jlb}: U?.9 (~{PE}), U?.9 (~{PE})
Other:
- moved on the sheet: C14

Commit message: put it allll together
Connections:
- net CO: now also U?.19 (CE), U?.19 (CE)
- net GND: now also U?.1 (A->B), U?.1 (A->B), U?.10 (GND), U?.10 (GND)
- net VCC: now also U?.20 (VCC), U?.20 (VCC)
- net at D?.2 (A), U?.5 (D2): now also U?.12 (B6)
- net at U?.11 (B7): now also D?.2 (A), U?.6 (D3)
- net at U?.13 (B5): now also D?.2 (A), U?.4 (D1)
- net at U?.14 (B4): now also D?.2 (A), U?.3 (D0)
- net at U?.15 (B3): now also D?.2 (A), U?.6 (D3)
- net at U?.16 (B2): now also D?.2 (A), U?.5 (D2)
- net at U?.17 (B1): now also D?.2 (A), U?.4 (D1)
- net at U?.18 (B0): now also D?.2 (A), U?.3 (D0)
Other:
- moved on the sheet: C14, D?, R?, U?

Commit message: fixed erc
Parts:
- gave numbers to parts that had none: 38
- renumbered C14 to C13

Commit message: np2
Parts:
- removed D61, D62, D63, D64, D65, D66, D67, D68, D69, D70, D71, D72, D73, D74, D75, D76: LED, symbol Device:LED
- removed R66, R67, R68, R69, R70, R71, R72, R73, R74, R75, R76, R77, R78, R79, R80, R81: R_Small, symbol Device:R_Small
- added D? (x16): LED, symbol Device:LED
- added R? (x16): R_Small, symbol Device:R_Small
Connections:
- net BUS_0: now also U18.11 (Q3), U20.11 (Q3); no longer U17.14 (Q0), U19.14 (Q0)
- net BUS_1: now also U18.12 (Q2), U20.12 (Q2); no longer U17.13 (Q1), U19.13 (Q1)
- net BUS_2: now also U18.13 (Q1), U20.13 (Q1); no longer U17.12 (Q2), U19.12 (Q2)
- net BUS_3: now also U18.14 (Q0), U20.14 (Q0); no longer U17.11 (Q3), U19.11 (Q3)
- net BUS_4: now also U17.11 (Q3), U19.11 (Q3); no longer U18.14 (Q0), U20.14 (Q0)
- net BUS_5: now also U17.12 (Q2), U19.12 (Q2); no longer U18.13 (Q1), U20.13 (Q1)
- net BUS_6: now also U17.13 (Q1), U19.13 (Q1); no longer U18.12 (Q2), U20.12 (Q2)
- net BUS_7: now also U17.14 (Q0), U19.14 (Q0); no longer U18.11 (Q3), U20.11 (Q3)
- net CLK: no longer U17.1 (~{MR}), U18.1 (~{MR}), U19.1 (~{MR}), U20.1 (~{MR})
- net CO: no longer U15.19 (CE), U16.19 (CE)
- net GND: now also R?.2, R?.2, R?.2, R?.2, R?.2, R?.2, R?.2, R?.2, R?.2, R?.2, R?.2, R?.2, R?.2, R?.2, R?.2, R?.2
- net ~{CLR}: no longer U17.2 (CP), U18.2 (CP), U19.2 (CP), U20.2 (CP)
- net at U15.15 (B3), U17.6 (D3): now also D?.2 (A)
- net at U16.12 (B6), U20.5 (D2): now also D?.2 (A)
- net at U15.18 (B0), U17.3 (D0): now also D?.2 (A)
- net at U16.11 (B7), U20.6 (D3): now also D?.2 (A)
- net at U16.13 (B5), U20.4 (D1): now also D?.2 (A)
- net at U16.14 (B4), U20.3 (D0): now also D?.2 (A)
- net at U16.15 (B3), U19.6 (D3): now also D?.2 (A)
- net at U16.16 (B2), U19.5 (D2): now also D?.2 (A)
- net at U16.17 (B1), U19.4 (D1): now also D?.2 (A)
- net at U16.18 (B0), U19.3 (D0): now also D?.2 (A)
- net at U15.12 (B6), U18.5 (D2): now also D?.2 (A)
- net at U15.17 (B1), U17.4 (D1): now also D?.2 (A)
- net at U15.14 (B4), U18.3 (D0): now also D?.2 (A)
- net at U15.13 (B5), U18.4 (D1): now also D?.2 (A)
- net at U15.11 (B7), U18.6 (D3): now also D?.2 (A)
- net at U15.16 (B2), U17.5 (D2): now also D?.2 (A)
- new net: D?.1 (K), R?.1 (x16)
- new net: U17.1 (~{MR}), U18.1 (~{MR}), U19.1 (~{MR}), U20.1 (~{MR})
- new net: U17.2 (CP), U18.2 (CP), U19.2 (CP), U20.2 (CP)
Other:
- moved on the sheet: C13, U15, U16, U17, U18, U19, U20
