File: Kicad Files/program-counter.kicad_sch (KiCad schematic)
At the start: 39 parts, among them U15 74HC245, U16 74HC245, U17 74LS161, U18 74LS161, U19 74LS161, U20 74LS161

Commit message: np3
Connections:
- net CLK: now also U17.2 (CP), U18.2 (CP), U19.2 (CP), U20.2 (CP)
- net CO: now also U15.19 (CE), U16.19 (CE)
- net ~{CLR}: now also U17.1 (~{MR}), U18.1 (~{MR}), U19.1 (~{MR}), U20.1 (~{MR})
Changed lines of the file:
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@@
   (junction (at 96.52 106.68) (diameter 0) (color 0 0 0 0)
+  )
+  (junction (at 41.275 124.46) (diameter 0) (color 0 0 0 0)
   )
   (junction (at 99.06 179.705) (diameter 0) (color 0 0 0 0)
@@
     (stroke (width 0) (type default) (color 0 0 0 0))
   )
-  (wire (pts (xy 47.625 168.275) (xy 60.325 168.275))
+  (wire (pts (xy 41.275 168.275) (xy 60.325 168.275))
     (stroke (width 0) (type default) (color 0 0 0 0))
   )
@@
     (stroke (width 0) (type default) (color 0 0 0 0))
   )
+  (wire (pts (xy 41.275 124.46) (xy 60.325 124.46))
+    (stroke (width 0) (type default) (color 0 0 0 0))
+  )
   (wire (pts (xy 226.06 17.78) (xy 229.235 17.78))
     (stroke (width 0) (type default) (color 0 0 0 0))
@@
     (stroke (width 0) (type default) (color 0 0 0 0))
   )
-  (wire (pts (xy 60.325 124.46) (xy 47.625 124.46))
-    (stroke (width 0) (type default) (color 0 0 0 0))
-  )
   (wire (pts (xy 177.8 33.02) (xy 177.8 44.45))
     (stroke (width 0) (type default) (color 0 0 0 0))
@@
     (stroke (width 0) (type default) (color 0 0 0 0))
   )
+  (wire (pts (xy 41.275 89.535) (xy 29.21 89.535))
+    (stroke (width 0) (type default) (color 0 0 0 0))
+  )
   (wire (pts (xy 134.62 22.86) (xy 220.98 22.86))
     (stroke (width 0) (type default) (color 0 0 0 0))
@@
     (stroke (width 0) (type default) (color 0 0 0 0))
   )
+  (wire (pts (xy 41.275 124.46) (xy 41.275 89.535))
+    (stroke (width 0) (type default) (color 0 0 0 0))
+  )
   (wire (pts (xy 238.76 74.295) (xy 195.58 74.295))
     (stroke (width 0) (type default) (color 0 0 0 0))
@@
   )
   (wire (pts (xy 236.22 71.755) (xy 209.55 71.755))
+    (stroke (width 0) (type default) (color 0 0 0 0))
+  )
+  (wire (pts (xy 41.275 124.46) (xy 41.275 168.275))
     (stroke (width 0) (type default) (color 0 0 0 0))
   )
@@
     (effects (font (size 1.524 1.524)) (justify right))
   )
-  (hierarchical_label "CLK" (shape input) (at 250.825 77.47 0)
+  (hierarchical_label "CLK" (shape input) (at 260.35 74.295 0)
     (effects (font (size 1.524 1.524)) (justify left))
   )
@@
     (effects (font (size 1.524 1.524)) (justify right))
   )
-  (hierarchical_label "~{CLR}" (shape input) (at 250.825 80.01 0)
+  (hierarchical_label "~{CLR}" (shape input) (at 260.35 76.835 0)
     (effects (font (size 1.524 1.524)) (justify left))
   )
