File: Kicad Files/mar.kicad_sch (KiCad schematic)
At the start: 37 parts, among them U14 74LS173, U16 74LS173

Commit message: finished todo list
Changed lines of the file:
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@@
+    (stroke (width 0) (type default) (color 0 0 0 0))
+  )
+  (wire (pts (xy 39.37 128.27) (xy 165.1 128.27))
     (stroke (width 0) (type default) (color 0 0 0 0))
   )
@@
     (stroke (width 0) (type default) (color 0 0 0 0))
   )
-  (wire (pts (xy 40.64 125.73) (xy 68.58 125.73))
+  (wire (pts (xy 39.37 125.73) (xy 68.58 125.73))
     (stroke (width 0) (type default) (color 0 0 0 0))
   )
@@
   )
   (wire (pts (xy 50.8 133.35) (xy 147.32 133.35))
-    (stroke (width 0) (type default) (color 0 0 0 0))
-  )
-  (wire (pts (xy 40.64 128.27) (xy 165.1 128.27))
     (stroke (width 0) (type default) (color 0 0 0 0))
   )
@@
     (effects (font (size 1.524 1.524)) (justify right))
   )
-  (hierarchical_label "~{MIlb}" (shape input) (at 40.64 125.73 180)
+  (hierarchical_label "~{MIlb}" (shape input) (at 39.37 125.73 180)
     (effects (font (size 1.524 1.524)) (justify right))
   )
@@
     (effects (font (size 1.524 1.524)) (justify right))
   )
-  (hierarchical_label "~{MIhb}" (shape input) (at 40.64 128.27 180)
+  (hierarchical_label "~{MIhb}" (shape input) (at 39.37 128.27 180)
     (effects (font (size 1.524 1.524)) (justify right))
   )

Commit message: fixed erc
Parts:
- gave numbers to parts that had none: 34
- renumbered U14 to U11, U16 to U12

Commit message: updated library
Parts:
- renumbered D37 to D45, D38 to D46, D39 to D47, D40 to D48, D41 to D49, D42 to D50, D43 to D51, D44 to D52, D45 to D53, D46 to D54, D47 to D55, D48 to D56, D49 to D57, D50 to D58, D51 to D59, D52 to D60, R42 to R50, R43 to R51, R44 to R52, R45 to R53, R46 to R54, R47 to R55, R48 to R56, R49 to R57, R50 to R58, R51 to R59, R52 to R60, R53 to R61, R54 to R62, R55 to R63, R56 to R64, R57 to R65
