File: Kicad Files/Z register.kicad_sch (KiCad schematic)
At the start: 24 parts, among them SW3 SW_DIP_x02, U21 74LS00, U22 LM555xN, U23 74LS273, U24 74LS112, U25 74LS112, U26 28C256, U27 7SEGMENT_CC, U28 74LS139, U29 7SEGMENT_CC, U30 7SEGMENT_CC, U31 7SEGMENT_CC

Commit message: new control sigs
Connections:
- net OI renamed ZI
Changed lines of the file:
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@@
     (effects (font (size 1.524 1.524)) (justify right))
   )
-  (hierarchical_label "OI" (shape input) (at 25.4 121.92 180)
+  (hierarchical_label "ZI" (shape input) (at 25.4 121.92 180)
     (effects (font (size 1.524 1.524)) (justify right))
   )

Commit message: tidy up
Parts:
- renumbered C14 to C13, C15 to C14, C16 to C15, C17 to C16, D77 to D61, D78 to D62, R82 to R66, R83 to R67, R84 to R68, R85 to R69, R86 to R70, R87 to R71, U21 to U15, U22 to U16, U23 to U17, U24 to U18, U25 to U19, U26 to U20, U27 to U21, U28 to U22, U29 to U23, U30 to U24, U31 to U25

Commit message: updated library
Parts:
- removed U17: 74LS273, Package_DIP:DIP-20_W7.62mm, symbol 8bit-computer-rescue:74LS273-8bit-computer-rescue
- removed U21, U23, U24, U25: 7SEGMENT_CC, Display_7Segment:7SegmentLED_LTS6760_LTS6780, symbol 8bit-computer-rescue:7SEGMENT_CC-8bit-computer-rescue
- removed U22: 74LS139, Package_DIP:DIP-16_W7.62mm, symbol 8bit-computer-rescue:74LS139-8bit-computer-rescue
- added U17: 74LS273, symbol 74xx:74LS273
- added U21: 74LS139, symbol 74xx:74LS139
- added U22, U23, U24, U25: HDSP-7403, Display_7Segment:HDSP-7401, symbol Display_Character:HDSP-7403
- renumbered D61 to D69, D62 to D70, R66 to R74, R67 to R75, R68 to R76, R69 to R77, R70 to R78, R71 to R79
Connections:
- net BUS_0: now also U17.3 (D0)
- net BUS_1: now also U17.4 (D1)
- net BUS_2: now also U17.7 (D2)
- net BUS_3: now also U17.8 (D3)
- net BUS_4: now also U17.13 (D4)
- net BUS_5: now also U17.14 (D5)
- net BUS_6: now also U17.17 (D6)
- net BUS_7: now also U17.18 (D7)
- net GND: now also U17.10 (GND), U21.1 (E)
- net VCC: now also U17.20 (VCC)
- net at U20.13 (D2): now also U22.4 (E), U23.4 (E), U24.4 (E), U25.4 (E)
- net at U20.11 (D0): now also U22.3 (G), U23.3 (G), U24.3 (G), U25.3 (G)
- net at U20.15 (D3): now also U22.5 (D), U23.5 (D), U24.5 (D), U25.5 (D)
- net at U20.16 (D4): now also U22.8 (C), U23.8 (C), U24.8 (C), U25.8 (C)
- net at U20.19 (D7): now also U22.7 (DP), U23.7 (DP), U24.7 (DP), U25.7 (DP)
- net at U20.17 (D5): now also U22.9 (B), U23.9 (B), U24.9 (B), U25.9 (B)
- net at U20.18 (D6): now also U22.10 (A), U23.10 (A), U24.10 (A), U25.10 (A)
- net at U20.12 (D1): now also U22.2 (F), U23.2 (F), U24.2 (F), U25.2 (F)
- net at U18.6 (~{Q}), U19.1 (C), U20.24 (A9): now also U21.2 (A0)
- net at U19.6 (~{Q}), U20.25 (A8): now also U21.3 (A1)
- net at U15.8: now also U17.1 (~{Mr})
- net at U15.6: now also U17.11 (Cp)
- net at U20.6 (A4): now also U17.12 (Q4)
- net at U20.5 (A5): now also U17.15 (Q5)
- net at U20.4 (A6): now also U17.16 (Q6)
- net at U20.3 (A7): now also U17.19 (Q7)
- net at U20.10 (A0): now also U17.2 (Q0)
- net at U20.9 (A1): now also U17.5 (Q1)
- net at U20.8 (A2): now also U17.6 (Q2)
- net at U20.7 (A3): now also U17.9 (Q3)
- new net: U21.4 (O0), U25.1 (CC), U25.6 (CC)
- new net: U21.5 (O1), U24.1 (CC), U24.6 (CC)
- new net: U21.6 (O2), U23.1 (CC), U23.6 (CC)
- new net: U21.7 (O3), U22.1 (CC), U22.6 (CC)

Commit message: im sooo stupiiid
Parts:
- added U?: 74HC245, symbol 74xx:74HC245
Connections:
- net BUS_0: now also U?.2 (A0)
- net BUS_1: now also U?.3 (A1)
- net BUS_2: now also U?.4 (A2)
- net BUS_3: now also U?.5 (A3)
- net BUS_4: now also U?.6 (A4)
- net BUS_5: now also U?.7 (A5)
- net BUS_6: now also U?.8 (A6)
- net BUS_7: now also U?.9 (A7)
- net GND: now also U?.1 (A->B), U?.10 (GND)
- net VCC: now also U16.3 (Q), U18.1 (C), U18.6 (~{Q}), U19.1 (C), U20.24 (A9), U21.2 (A0)
- net at U17.12 (Q4), U20.6 (A4): now also U?.14 (B4)
- net at U17.15 (Q5), U20.5 (A5): now also U?.13 (B5)
- net at U17.16 (Q6), U20.4 (A6): now also U?.12 (B6)
- net at U17.19 (Q7), U20.3 (A7): now also U?.11 (B7)
- net at U17.2 (Q0), U20.10 (A0): now also U?.18 (B0)
- net at U17.5 (Q1), U20.9 (A1): now also U?.17 (B1)
- net at U17.6 (Q2), U20.8 (A2): now also U?.16 (B2)
- net at U17.9 (Q3), U20.7 (A3): now also U?.15 (B3)
- new net ~{ZO}: U?.19 (CE)
Other:
- moved on the sheet: C13, C14, D69, D70, R74, R75, R76, R77, R78, R79, SW3, U15A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

Commit message: complete redraw to bus system
Connections:
- net BUS_0 renamed D0
- net BUS_1 renamed D1
- net BUS_2 renamed D2
- net BUS_3 renamed D3
- net BUS_4 renamed D4
- net BUS_5 renamed D5
- net BUS_6 renamed D6
- net BUS_7 renamed D7
Changed lines of the file:
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@@
     (effects (font (size 1.524 1.524)) (justify left bottom))
+  )
+  (hierarchical_label "D7" (shape input) (at 35.56 66.04 180)
+    (effects (font (size 1.524 1.524)) (justify right))
+  )
+  (hierarchical_label "D2" (shape input) (at 35.56 53.34 180)
+    (effects (font (size 1.524 1.524)) (justify right))
   )
   (hierarchical_label "CLR" (shape input) (at 25.4 149.86 180)
@@
     (effects (font (size 1.524 1.524)) (justify right))
   )
-  (hierarchical_label "BUS_0" (shape input) (at 35.56 48.26 180)
+  (hierarchical_label "D6" (shape input) (at 35.56 63.5 180)
     (effects (font (size 1.524 1.524)) (justify right))
   )
-  (hierarchical_label "BUS_5" (shape input) (at 35.56 60.96 180)
+  (hierarchical_label "D1" (shape input) (at 35.56 50.8 180)
     (effects (font (size 1.524 1.524)) (justify right))
   )
-  (hierarchical_label "BUS_7" (shape input) (at 35.56 66.04 180)
+  (hierarchical_label "D4" (shape input) (at 35.56 58.42 180)
     (effects (font (size 1.524 1.524)) (justify right))
   )
-  (hierarchical_label "BUS_2" (shape input) (at 35.56 53.34 180)
+  (hierarchical_label "D3" (shape input) (at 35.56 55.88 180)
     (effects (font (size 1.524 1.524)) (justify right))
   )
-  (hierarchical_label "BUS_3" (shape input) (at 35.56 55.88 180)
-    (effects (font (size 1.524 1.524)) (justify right))
-  )
-  (hierarchical_label "BUS_6" (shape input) (at 35.56 63.5 180)
-    (effects (font (size 1.524 1.524)) (justify right))
-  )
-  (hierarchical_label "BUS_1" (shape input) (at 35.56 50.8 180)
-    (effects (font (size 1.524 1.524)) (justify right))
-  )
-  (hierarchical_label "BUS_4" (shape input) (at 35.56 58.42 180)
+  (hierarchical_label "D5" (shape input) (at 35.56 60.96 180)
     (effects (font (size 1.524 1.524)) (justify right))
   )
@@
     (effects (font (size 1.524 1.524)) (justify right))
   )
+  (hierarchical_label "D0" (shape input) (at 35.56 48.26 180)
+    (effects (font (size 1.524 1.524)) (justify right))
+  )
