File: Kicad Files/addrdec.kicad_sch (KiCad schematic)
At the start: 9 parts, among them U21 74LS139, U32 SST39SF010, U55 HDSP-A151, U56 HDSP-A151, U57 SST39SF020, U58 HDSP-A151, U59 HDSP-A151, U60 MAX7375AXR105, U62 74LS161

Commit message: rethink alu
Parts:
- added J1: Conn_01x02_Pin, symbol Connector:Conn_01x02_Pin
- added J2: Conn_01x02_Socket, symbol Connector:Conn_01x02_Socket
Connections:
- net R/~{W}: now also J1.2 (Pin_2), J2.1 (Pin_1)
- net ~{R}/W: now also J1.1 (Pin_1), J2.2 (Pin_2)
Changed lines of the file:
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@@
+    (stroke (width 0) (type default))
+  )
+  (wire (pts (xy 95.885 61.595) (xy 99.06 61.595))
     (stroke (width 0) (type default))
   )
@@
     (stroke (width 0) (type default))
   )
+  (wire (pts (xy 95.885 61.595) (xy 95.885 73.025))
+    (stroke (width 0) (type default))
+  )
   (wire (pts (xy 197.485 51.435) (xy 207.645 51.435))
     (stroke (width 0) (type default))
@@
     (stroke (width 0) (type default))
   )
+  (wire (pts (xy 97.155 70.485) (xy 116.84 70.485))
+    (stroke (width 0) (type default))
+  )
   (wire (pts (xy 210.185 74.295) (xy 210.185 99.695))
     (stroke (width 0) (type default))
@@
     (stroke (width 0) (type default))
   )
+  (wire (pts (xy 116.84 73.025) (xy 95.885 73.025))
+    (stroke (width 0) (type default))
+  )
+  (wire (pts (xy 97.155 64.135) (xy 97.155 70.485))
+    (stroke (width 0) (type default))
+  )
   (wire (pts (xy 225.425 94.615) (xy 215.265 94.615))
     (stroke (width 0) (type default))
@@
     (stroke (width 0) (type default))
   )
+  (wire (pts (xy 99.06 64.135) (xy 97.155 64.135))
+    (stroke (width 0) (type default))
+  )
   (wire (pts (xy 205.105 104.775) (xy 205.105 130.175))
     (stroke (width 0) (type default))
@@
     (effects (font (size 1.524 1.524)) (justify right))
   )
-  (hierarchical_label "~{R}{slash}W" (shape output) (at 81.28 139.7 0) (fields_autoplaced)
+  (hierarchical_label "~{R}{slash}W" (shape output) (at 99.06 61.595 0) (fields_autoplaced)
     (effects (font (size 1.524 1.524)) (justify left))
   )
@@
   (hierarchical_label "a11" (shape input) (at 68.58 69.215 180) (fields_autoplaced)
     (effects (font (size 1.524 1.524)) (justify right))
+  )
+  (hierarchical_label "~{R}{slash}W" (shape input) (at 127 70.485 0) (fields_autoplaced)
+    (effects (font (size 1.524 1.524)) (justify left))
   )
   (hierarchical_label "~{CS}_{4}" (shape output) (at 99.06 51.435 0) (fields_autoplaced)
@@
     (effects (font (size 1.524 1.524)) (justify right))
   )
-  (hierarchical_label "R{slash}~{W}" (shape input) (at 66.04 139.7 180) (fields_autoplaced)
-    (effects (font (size 1.524 1.524)) (justify right))
+  (hierarchical_label "R{slash}~{W}" (shape output) (at 99.06 64.135 0) (fields_autoplaced)
+    (effects (font (size 1.524 1.524)) (justify left))
   )
   (hierarchical_label "~{CS}_{ROM}" (shape output) (at 99.06 41.275 0) (fields_autoplaced)
+    (effects (font (size 1.524 1.524)) (justify left))
+  )
+  (hierarchical_label "R{slash}~{W}" (shape input) (at 127 73.025 0) (fields_autoplaced)
     (effects (font (size 1.524 1.524)) (justify left))
   )
@@
     )
   )
+  (symbol (lib_id "Connector:Conn_01x02_Pin") (at 121.92 70.485 0) (unit 1)
+    (in_bom yes) (on_board yes) (dnp no)
+    (property "Reference" "J1" (at 122.555 66.04 0)
+      (effects (font (size 1.27 1.27)))
+    )
+    (property "Value" "Conn_01x02_Pin" (at 121.92 75.565 0)
+      (effects (font (size 1.27 1.27)))
+    )
+    (property "Footprint" "" (at 121.92 70.485 0)
+      (effects (font (size 1.27 1.27)) hide)
+    )
+    (property "Datasheet" "~" (at 121.92 70.485 0)
+      (effects (font (size 1.27 1.27)) hide)
+    )
+    (pin "1")
+    (pin "2")
+    (instances
+      (project "8bit-computer"
+        (path "/191de3e9-4a12-4a8c-98d6-fd12e8e1e7d7/4d1ce46d-22a2-4504-8697-c06d99bb8de0"
+          (reference "J1") (unit 1)
+        )
+      )
+    )
+  )
   (symbol (lib_id "Display_Character:HDSP-A151") (at 233.045 122.555 0) (unit 1)
     (in_bom yes) (on_board yes) (dnp no)
@@
         )
       )
+    )
+  )
+  (symbol (lib_id "Connector:Conn_01x02_Socket") (at 121.92 70.485 0) (unit 1)
+    (in_bom yes) (on_board yes) (dnp no)
+    (property "Reference" "J2" (at 123.825 71.12 0)
+      (effects (font (size 1.27 1.27)) (justify left))
+    )
+    (property "Value" "Conn_01x02_Socket" (at 112.395 77.47 0)
+      (effects (font (size 1.27 1.27)) (justify left))
+    )
+    (property "Footprint" "" (at 121.92 70.485 0)
+      (effects (font (size 1.27 1.27)) hide)
+    )
+    (property "Datasheet" "~" (at 121.92 70.485 0)
+      (effects (font (size 1.27 1.27)) hide)
+    )
+    (pin "1")
+    (pin "2")
+    (instances
+      (project "8bit-computer"
+        (path "/191de3e9-4a12-4a8c-98d6-fd12e8e1e7d7/4d1ce46d-22a2-4504-8697-c06d99bb8de0"
+          (reference "J2") (unit 1)
+        )
+      )
