File: Kicad Files/areg.kicad_sch (KiCad schematic)
At the start: 23 parts, among them U42 74HC245, U44 74LS173, U54 74LS173

Commit message: c30
Parts:
- added U42: 74HC245, symbol 74xx:74HC245
Connections:
- net GND: now also U42.10 (GND)
- net VCC: now also U42.1 (A->B), U42.20 (VCC)
- net d_{i}0: now also U42.11 (B7)
- net d_{i}1: now also U42.12 (B6)
- net d_{i}2: now also U42.13 (B5)
- net d_{i}3: now also U42.14 (B4)
- net d_{i}4: now also U42.15 (B3)
- net d_{i}5: now also U42.16 (B2)
- net d_{i}6: now also U42.17 (B1)
- net d_{i}7: now also U42.18 (B0)
