File: Kicad Files/id.kicad_sch (KiCad schematic)
At the start: 80 parts, among them SW1 SW_Push, U16 74HC00, U27 74HC00, U60 74LS161, U61 SST39SF040, U62 SST39SF040, U63 SST39SF040, U64 SST39SF040, U74 74HC00

Commit message: c30
Parts:
- removed D41 (x4), D42 (x4), D44 (x4), D55 (x4), D56 (x4), D57 (x4), D58 (x4), D59 (x4): LED_Small, symbol Device:LED_Small
- removed R42 (x4), R45 (x4), R49 (x4), R60 (x4), R61 (x4), R62 (x4), R63 (x4), R64 (x4): R_Small, symbol Device:R_Small
- removed unit 3 of U27
- removed U64: SST39SF040, symbol Memory_Flash:SST39SF040
- added D1 (x4), D2 (x4), D3 (x4), D4 (x3), D41 (x4), D42 (x4), D44 (x4), D5 (x3), D55 (x4), D56 (x4), D57 (x4), D58 (x4), D59 (x4), D6 (x3), D7 (x3), D8 (x3): LED_Small, symbol Device:LED_Small
- added R1 (x4), R2 (x4), R3 (x4), R4 (x3), R42 (x4), R45 (x4), R49 (x4), R5 (x3), R6 (x3), R60 (x4), R61 (x4), R62 (x4), R63 (x4), R64 (x4), R7 (x3), R8 (x3): R_Small, symbol Device:R_Small
- added R172: R, symbol Device:R
- added SW1: SW_Push, symbol Switch:SW_Push
- added U102, U104, U106, U107: SST39SF040, symbol Memory_Flash:SST39SF040
- added U79, U84, U96: 74HC00, symbol 74xx:74HC00
- added U97: 74LS161, symbol 74xx:74LS161
Connections:
- net CLK: now also U84.4, U84.5
- net CLR: now also R172.1, SW1.2, U96.1, U96.2
- net F_4: now also U102.4 (A12), U104.4 (A12), U106.4 (A12), U107.4 (A12)
- net F_5: now also U102.28 (A13), U104.28 (A13), U106.28 (A13), U107.28 (A13)
- net F_6: now also U102.29 (A14), U104.29 (A14), U106.29 (A14), U107.29 (A14)
- net F_7: now also U102.3 (A15), U104.3 (A15), U106.3 (A15), U107.3 (A15)
- net F_C: now also U102.27 (A8), U104.27 (A8), U106.27 (A8), U107.27 (A8)
- net F_N: now also U102.23 (A10), U104.23 (A10), U106.23 (A10), U107.23 (A10)
- net F_V: now also U102.25 (A11), U104.25 (A11), U106.25 (A11), U107.25 (A11)
- net F_Z: now also U102.26 (A9), U104.26 (A9), U106.26 (A9), U107.26 (A9)
- net GND: now also R1.2, R1.2, R1.2, R1.2, R172.2, R2.2, R2.2, R2.2, R2.2, R3.2, R3.2, R3.2, R3.2, R4.2, R4.2, R4.2, R42.2, R42.2, R42.2, R42.2, R45.2, R45.2, R45.2, R45.2, R49.2, R49.2, R49.2, R49.2, R5.2, R5.2, R5.2, R6.2, R6.2, R6.2, R60.2, R60.2, R60.2, R60.2, R61.2, R61.2, R61.2, R61.2, R62.2, R62.2, R62.2, R62.2, R63.2, R63.2, R63.2, R63.2, R64.2, R64.2, R64.2, R64.2, R7.2, R7.2, R7.2, R8.2, R8.2, R8.2, U102.16 (GND), U104.16 (GND), U106.16 (GND), U107.16 (GND), U79.7 (GND), U97.3 (D0), U97.4 (D1), U97.5 (D2), U97.6 (D3), U97.8 (GND)
- net HLT: now also U63.18 (D4), D5.2 (A)
- net H/~{L}: now also U63.17 (D3), D4.2 (A); no longer U61.15 (D2)
- net I_0: now also U102.12 (A0), U104.12 (A0), U106.12 (A0), U107.12 (A0)
- net I_1: now also U102.11 (A1), U104.11 (A1), U106.11 (A1), U107.11 (A1)
- net I_2: now also U102.10 (A2), U104.10 (A2), U106.10 (A2), U107.10 (A2)
- net I_3: now also U102.9 (A3), U104.9 (A3), U106.9 (A3), U107.9 (A3)
- net I_4: now also U102.8 (A4), U104.8 (A4), U106.8 (A4), U107.8 (A4)
- net I_5: now also U102.7 (A5), U104.7 (A5), U106.7 (A5), U107.7 (A5)
- net I_6: now also U102.6 (A6), U104.6 (A6), U106.6 (A6), U107.6 (A6)
- net I_7: now also U102.5 (A7), U104.5 (A7), U106.5 (A7), U107.5 (A7)
- net R/~{W}: now also U63.15 (D2), D3.2 (A); no longer U61.14 (D1)
- net VCC: now also SW1.1, U102.22 (CE), U102.24 (OE), U102.31 (PGM), U102.32 (VCC), U104.22 (CE), U104.24 (OE), U104.31 (PGM), U104.32 (VCC), U106.22 (CE), U106.24 (OE), U106.31 (PGM), U106.32 (VCC), U107.22 (CE), U107.24 (OE), U107.31 (PGM), U107.32 (VCC), U79.14 (VCC), U84.12, U84.13, U97.10 (CET), U97.16 (VCC), U97.7 (CEP)
- net Z_{I}: now also D44.2 (A), U106.15 (D2); no longer U63.15 (D2)
- net ~{A}_{I}: now also D56.2 (A), U106.18 (D4); no longer U63.18 (D4)
- net ~{A}_{O}: now also D55.2 (A), U106.17 (D3); no longer U63.17 (D3)
- net ~{D_{O}}: now also D56.2 (A), U107.18 (D4)
- net ~{F}: now also D57.2 (A), U106.19 (D5); no longer U63.19 (D5)
- net ~{I}_{I}: now also D59.2 (A), U107.21 (D7)
- net ~{I}_{O}: now also D58.2 (A), U107.20 (D6)
- net ~{M_{I}}: now also D41.2 (A), U106.13 (D0); no longer U63.13 (D0)
- net ~{M_{O}}: now also D59.2 (A), U104.21 (D7); no longer U62.21 (D7)
- net ~{PC_{I}}: now also D58.2 (A), U104.20 (D6); no longer U62.20 (D6)
- net ~{PC_{Oa}}: now also D56.2 (A), U104.18 (D4); no longer U62.18 (D4)
- net ~{PC_{Od}}: now also D57.2 (A), U104.19 (D5); no longer U62.19 (D5)
- net ~{P}_{I}: now also D55.2 (A), U107.17 (D3)
- net ~{P}_{O}: now also D44.2 (A), U107.15 (D2)
- net ~{RMS}: now also U63.13 (D0), D1.2 (A), D41.2 (A), U102.13 (D0), U97.9 (~{PE}); no longer U61.13 (D0)
- net ~{R}/W: now also U63.14 (D1), D2.2 (A)
- net ~{SP_{I}}: now also D55.2 (A), U104.17 (D3); no longer U62.17 (D3)
- net ~{SP_{Oa}}: now also D42.2 (A), U104.14 (D1); no longer U62.14 (D1)
- net ~{SP_{Od}}: now also D44.2 (A), U104.15 (D2); no longer U62.15 (D2)
- net ~{X_{I}}: now also D41.2 (A), U104.13 (D0); no longer U62.13 (D0)
- net ~{X_{Oa}}: now also D58.2 (A), U102.20 (D6); no longer U61.20 (D6)
- net ~{X_{Od}}: now also D59.2 (A), U102.21 (D7); no longer U61.21 (D7)
- net ~{Y_{I}}: now also D57.2 (A), U102.19 (D5); no longer U61.19 (D5)
- net ~{Y_{Oa}}: now also D55.2 (A), U102.17 (D3); no longer U61.17 (D3)
- net ~{Y_{Od}}: now also D56.2 (A), U102.18 (D4); no longer U61.18 (D4)
- net ~{Z}_{O}: now also D42.2 (A), U106.14 (D1); no longer U63.14 (D1)
- net ~{Σ}_{O}: now also D42.2 (A), U107.14 (D1)
- net Σ_0: now also D41.2 (A), U107.13 (D0)
- net Σ_1: now also D59.2 (A), U106.21 (D7); no longer U63.21 (D7)
- net Σ_2: now also D58.2 (A), U106.20 (D6); no longer U63.20 (D6)
- new net: D42.1 (K), R45.1 (x4)
- new net: D1.1 (K), R2.1
- new net: D1.2 (A), U102.1 (A18), U104.1 (A18), U106.1 (A18), U107.1 (A18), U97.14 (Q0)
- new net: D56.1 (K), R61.1 (x4)
- new net: D4.1 (K), R4.1 (x3)
- new net: D58.1 (K), R63.1 (x4)
- new net: D5.1 (K), R5.1 (x3)
- new net: D7.1 (K), R7.1 (x3)
- new net: D59.1 (K), R64.1 (x4)
- new net: D41.1 (K), R42.1 (x4)
- new net: D57.1 (K), R62.1 (x4)
- new net: D2.1 (K), R2.1 (x3)
- new net: D55.1 (K), R60.1 (x4)
- new net: D6.1 (K), R6.1 (x3)
- new net: D8.1 (K), R8.1 (x3)
- new net: D2.1 (K), R1.1
- new net: D2.2 (A), U102.30 (A17), U104.30 (A17), U106.30 (A17), U107.30 (A17), U97.13 (Q1)
- new net: D6.2 (A), U63.19 (D5)
- new net: D7.2 (A), U63.20 (D6)
- new net: D44.1 (K), R49.1 (x4)
- new net: D3.2 (A), U102.2 (A16), U104.2 (A16), U106.2 (A16), U107.2 (A16), U97.12 (Q2)
- new net: D1.1 (K), R1.1 (x3)
- new net: D3.1 (K), R3.1 (x4)
- new net: D57.2 (A), U107.19 (D5)
- new net: U96.3, U97.1 (~{MR})
- new net: D42.2 (A), U102.14 (D1), U84.10, U84.9
- new net: D44.2 (A), U102.15 (D2)
- new net: D8.2 (A), U63.21 (D7)
- new net: U84.6, U97.2 (CP)
- new net CA_{M}0: D1.2 (A), U61.13 (D0)
- new net CA_{M}1: D2.2 (A), U61.14 (D1)
- new net CA_{M}2: D3.2 (A), U61.15 (D2)
- new net CA_{M}3: D4.2 (A), U61.17 (D3)
- new net CA_{S}0: D5.2 (A), U61.18 (D4)
- new net CA_{S}1: D6.2 (A), U61.19 (D5)
- new net CA_{S}2: D7.2 (A), U61.20 (D6)
- new net CA_{S}3: D8.2 (A), U61.21 (D7)
- new net CO_{M}0: D1.2 (A), U62.13 (D0)
- new net CO_{M}1: D2.2 (A), U62.14 (D1)
- new net CO_{M}2: D3.2 (A), U62.15 (D2)
- new net CO_{M}3: D4.2 (A), U62.17 (D3)
- new net CO_{S}0: D5.2 (A), U62.18 (D4)
- new net CO_{S}1: D6.2 (A), U62.19 (D5)
- new net CO_{S}2: D7.2 (A), U62.20 (D6)
- new net CO_{S}3: D8.2 (A), U62.21 (D7)
- no-connect marks 2 -> 4
Other:
- moved on the sheet: D1, D2, D3, R1, R156, R2, R3, SW1, U16E, U27B, U27D, U60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
