File: Kicad Files/sp.kicad_sch (KiCad schematic)
At the start: 27 parts, among them U45 74HC245, U46 74LS173, U47 74LS173

Commit message: rethink alu
Other:
- note added: "Stack address"
Changed lines of the file:
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@@
     (stroke (width 0) (type default))
+  )
+  (text "Stack address" (at 212.725 138.43 90)
+    (effects (font (size 1.524 1.524)) (justify right bottom))
   )
   (hierarchical_label "d_{i}4" (shape tri_state) (at 20.955 26.67 180) (fields_autoplaced)

Commit message: updated stuff
Other:
- note added: "Stack Limited to 256 Bytes Not bottom open Might need rework Top 8 Adr Bits are Hardwired!"
Changed lines of the file:
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@@
     (stroke (width 0) (type default))
+  )
+  (text "Stack Limited to 256 Bytes\n	Not bottom open\n	Might need rework\n	Top 8 Adr Bits are Hardwired!\n"
+    (at 113.03 129.54 0)
+    (effects (font (size 1.524 1.524)) (justify left bottom))
   )
   (text "Stack address" (at 212.725 138.43 90)
